File: V0/Design/HW.ACIM-DBG/HW.ACIM-DBG.kicad_sch (KiCad schematic)
At the start: 0 parts

Commit message: V0.1 production files
Parts:
- added SH1, SH2, SH3, SH4, SH5: SCREW HOLDER, SAMPI:SCREWHOLE-2.5M, symbol SAMPI:SCREWHOLDER
Other:
- added sheet AC-DC Adapter (ACDCAdapter.kicad_sch)
