File: V0/Design/HW.ACIM-DBG/USB_HUB.kicad_sch (KiCad schematic)
At the start: 82 parts, among them J1 INV DEBUG, J2 Micro USB, J3 PSU DEBUG, J4 USB, Q1 20V/1A, Q2 20V/1A, U1 LDO 3.3V/300mA, U2 USB HUB 2.0 4-CH, U3 ISO USB 2.0, U4 24MHz (3225)

Commit message: V0.1 production files
Parts:
- removed FT12: 120R@100MHz, SAMPI:FT0603, symbol SAMPI:FerriteBead
- removed MD1: DC-DC, SAMPI:B0505MT-1WR4, symbol SAMPI:DC-DC_B05xxMT-1WR4
- removed Q1: 20V/1A, SAMPI:SOT23, symbol SAMPI:FET_P-CH
- removed Q2: 20V/1A, SAMPI:SOT23, symbol SAMPI:FET_N-CH
- removed R3: 10K, SAMPI:RES0603, symbol SAMPI:RES
- added C54, C55: 220uF/6.3V, SAMPI:CAP1411, symbol SAMPI:ELECCAP
- added MD1: DUAL 5V-5V/2W, SAMPI:B0505S-2WR2-DUAL, symbol SAMPI:DC-DC
- added U9: LOAD SWITCHER, SAMPI:SOT363, symbol SAMPI:MIC94090YC6
- C18: now not fitted; now left out of the parts list
- D1: MFT Nexperia -> Nexperia
- FT11: now fitted; now in the parts list
Connections:
- net +3V3: no longer R10.2
- net +5V: now also C54.+, MD1.6 (DC+), U9.4 (VIN)
- net +5V_ISO: now also MD1.1 (VI+)
- net GND: now also R10.2, C54.-, MD1.4 (DC-), MD1.5 (NC), U9.2 (GND), U9.5 (GND)
- net GND_ISO: now also C55.-, MD1.2 (VI-)
- net PRG_VBUS: now also U9.6 (EN)
- net USB6_N: now also FT11.1; no longer FT11.4
- net USB6_P: now also FT11.4; no longer FT11.1
- net at C3.2, D1.4 (CH3), FT1.2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: now also C55.+
- net at C10.2, C9.2, J2.1 (VCC): now also U9.1 (VOUT)
Other:
- moved on the sheet: C10, C11, C2, C3, C53, C7, C8, C9, J1, J2, J3, MD2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
