File: V0/Design/HW.ACIM-DBG/VCP.kicad_sch (KiCad schematic)
At the start: 62 parts, among them U5 FT4232H, U6 SPI EEPROM, U7 SHIFT REG 8BIT, U8 12MHz (3225)

Commit message: V0.1 production files
Parts:
- removed U8: 12MHz (3225), SAMPI:CDFN3225-4LD-PL-1, symbol SAMPI:OSC
- added D7: VCP, SAMPI:LED0603, symbol SAMPI:RLED
- added R3: 1.1K, SAMPI:RES0603, symbol SAMPI:RES
- added U8: 12MHz, SAMPI:CDFN2520-ABM10, symbol SAMPI:XTAL-4P
- C33: value 100nF -> 22pF; MFT Samsung -> Walsin; MNP CL10B104KB8NNNC -> 0603N220J500CT; Unit Price 0.0146 -> 0.012
- D2, D3, D4, D5: MFT Harvatek -> Harvatek
- R15: value 0R -> 1.1K; MNP RC0603JR-070RL -> AC0603FR-071K1L; Unit Price 0.015 -> 0.021; now not fitted; now left out of the parts list
Connections:
- net +3V3: now also R15.1; no longer C33.2
- net GND: now also R3.2, U8.2 (GND1), U8.4 (X2)
- net at U5.30 (~{SUSPEND}): now also D7.A
- net OSCO: now reaches U5.4 (OSCO)
- net OSCO: now also C33.2, U8.3 (GND2)
- net at R15.2: now also D7.K, R3.1
- net SYS_CLK renamed OSCI
- net OSCI: now also U8.1 (X1); no longer R15.1
- no-connect marks 24 -> 21
Other:
- moved on the sheet: C32
