File: V1/Design/HW.ACIM-DBG/ISOLATOR.kicad_sch (KiCad schematic)
At the start: 23 parts, among them J1 EXT INV DEBUG, J2 Micro USB, J3 PSU DEBUG, J5 INV DEBUG, U1 LOAD SWITCHER, U3 ISO USB 2.0

Commit message: V1 schematic update 1
Parts:
- removed C1, C12: 100nF, SAMPI:CAP0603, symbol SAMPI:CERCAP
- removed C10, C9: 100pF/2kV, SAMPI:CAP1206, symbol SAMPI:CERCAP
- removed C11, C6: 10uF, SAMPI:CAP0603, symbol SAMPI:CERCAP
- removed C2, C4: 220uF/6.3V, SAMPI:CAP1411, symbol SAMPI:ELECCAP
- removed D9: PWR, SAMPI:LED0603, symbol SAMPI:WLED
- removed FT11, FT3: 2x 120R@100MHz, SAMPI:IND1210_4P, symbol SAMPI:IND1210_4P
- removed J1: EXT INV DEBUG, SAMPI:HDM1x8x2.54_TH_RA, symbol SAMPI:SIL08
- removed J3: PSU DEBUG, SAMPI:HDF1x10x2.54_TH_RA, symbol SAMPI:SIL10
- removed J5: INV DEBUG, SAMPI:HDF1x10x2.54_TH_RA, symbol SAMPI:SIL10
- removed R4: 10K, SAMPI:RES0603, symbol SAMPI:RES
- removed R55: 1.1K, SAMPI:RES0603, symbol SAMPI:RES
- removed U3: ISO USB 2.0, SAMPI:SOIC16_7.5_AN, symbol SAMPI:ADUM3160
- added C26, C27, C28, C29: 10uF, SAMPI:CAP0603, symbol SAMPI:CERCAP
- added J3: SIL08, symbol SAMPI:SIL08
- added J5: MCDBG, SAMPI:IDC-2x5x2MM-TH, symbol SAMPI:MCDBG
- added OP1, OP2: OPTO-BJT-1CH, SAMPI:OPTO_SO4_7.6MM, symbol SAMPI:OPTO-BJT-1CH
- added Q2, Q3: MFET P, symbol SAMPI:FET_P-CH
- added R21, R22: 100R, Liem:RES0402, symbol SAMPI:RES
- added R23, R26, R29: 1K, Liem:RES0402, symbol SAMPI:RES
- added R24, R28: 47K, Liem:RES0402, symbol SAMPI:RES
- added R25: 10K, Liem:RES0402, symbol SAMPI:RES
- added R27: 5.1K, Liem:RES0402, symbol SAMPI:RES
- added RL1: RELAY2-NL, SAMPI:EA2-5NU, symbol SAMPI:RELAY2-NL
- added U6, U7: ISO6740, SAMPI:SOIC16-W, symbol SAMPI:ISO6740
Connections:
- net +3V3: now also C27.2, C28.2, Q2.3 (D), Q3.2 (S), R24.2, R28.1, U6.10 (EN2), U6.16 (VCC2), U7.1 (VCC1)
- net GND: now also C27.1, C28.1, J3.3, OP1.3 (E), OP2.2 (K), R25.2, U6.15 (GND2), U6.9 (GND2), U7.2 (GND1), U7.8 (GND1)
- net GND_ISO: now also C26.1, C29.1, J5.6 (GND), OP1.2 (K), OP2.3 (E), U6.2 (GND1), U6.8 (GND1), U7.15 (GND2), U7.9 (GND2)
- net USB6_N renamed PRG_USB_N
- net USB6_P renamed PRG_USB_P
- new net: R21.1, U7.11 (OUTD)
- new net: OP1.4 (C), Q2.1 (G), R24.1
- new net: J3.8, RL1.7 (NO2)
- new net: J3.4, RL1.9 (NC2)
- new net: OP1.1 (A), R23.1
- new net: R22.2, U6.14 (OUTA)
- new net: OP2.1 (A), R26.1
- new net: Q3.3 (D), R26.2
- new net: Q3.1 (G), R28.2, R29.2
- new net +3V3_ISO: C26.2, C29.2, J5.4 (VDD), R23.2, R27.2, U6.1 (VCC1), U7.10 (EN2), U7.16 (VCC2)
- new net DB_TXD: U6.11 (OUTD)
- new net DV_CTS: U7.4 (INB)
- new net DV_RTS: U6.12 (OUTC)
- new net DV_RXD: U7.3 (INA)
- new net DV_TXD: U6.13 (OUTB)
- new net ISO_DB_TXD: J5.9 (DB_TXD), U6.6 (IND)
- new net ISO_DV_CTS: J5.7 (DV_CTS), U7.13 (OUTB)
- new net ISO_DV_RTS: J5.5 (DV_RTS), U6.5 (INC)
- new net ISO_DV_RXD: J5.3 (DV_RXD), U7.14 (OUTA)
- new net ISO_DV_TXD: J5.1 (DV_TXD), U6.4 (INB)
- new net ISO_PGC: J5.10 (PGC/SWIO), U7.12 (OUTC)
- new net ISO_PGD: J5.8 (PGD/SWCK), R21.2, U6.3 (INA)
- new net PGC: J3.5, U7.5 (INC)
- new net PGD: R22.1, RL1.8 (COM2), U7.6 (IND)
- new net VDD_SEN: J3.2, Q2.2 (S), R25.1
- new net ~{ISO_MCLR}: J5.2 (~{RESET}), OP2.4 (C), R27.1
- new net ~{MCLR}: J3.1, R29.1
- no-connect marks 1 -> 3
Other:
- note added: "ISOLATED POWER - DANGER-ZONE"
- moved on the sheet: C5, C7, C8, J2, MD1, U1

Commit message: V1 schematic update 2
Parts:
- removed C5: 10uF, SAMPI:CAP0603, symbol SAMPI:CERCAP
- removed RL1: RELAY2-NL, SAMPI:EA2-5NU, symbol SAMPI:RELAY2-NL
- added C4: 220uF, Liem:CAP2312-6032, symbol SAMPI:ELECCAP
- added D4: PIC, Liem:LED0603, symbol Liem:RLED
- added D5: ARM, Liem:LED0603, symbol Liem:RLED
- added R15, R16: 1K, Liem:RES0402, symbol SAMPI:RES
- added R17, R18: 100K, Liem:RES0402, symbol SAMPI:RES
- added SW1: PRG SEL, SAMPI:SW_PUSH_2DPDT, symbol SAMPI:SW_DPDT
- C7: Checked OK -> (none); Unit Price 0.079 -> (none)
- C8: Checked OK -> (none); Unit Price 0.0146 -> (none)
- J2: value Micro USB -> MICRO USB; Checked OK -> (none)
- J3: value SIL08 -> SNAP PINOUT; footprint (none) -> SAMPI:HDF1x8x2.54_TH_RA; MFT (none) -> Sullins Connector Solutions; MNP (none) -> PPTC081LGBN-RC
- J5: value MCDBG -> MCLS
- MD1: Checked OK -> (none)
- Q2, Q3: value MFET P -> 20V/2.3A; MFT (none) -> Vishay; MNP (none) -> SI2301DS
- R24, R28: value 47K -> 10K
Connections:
- net GND: now also R26.1, C4.-, D4.K, D5.K, R17.1, R18.1; no longer OP2.2 (K)
- net PGD: now also SW1.2 (COM1)
- net at C7.2, J2.1 (VCC), U1.1 (VOUT): now also C4.+, SW1.5 (COM2)
- net at J3.8: now also SW1.3 (NO1)
- net at J3.4: now also SW1.1 (NC1)
- net at OP2.1 (A): now also Q3.3 (D); no longer R26.1
- net at R26.2: now also OP2.2 (K); no longer Q3.3 (D)
- net DV_CTS renamed HS_CTS
- net DV_RXD renamed HS_RXD
- new net: R15.2, R17.2, SW1.4 (NC2)
- new net: D4.A, R15.1
- new net: R16.2, R18.2, SW1.6 (NO2)
- new net: D5.A, R16.1
Other:
- moved on the sheet: C26, C27, C28, C29, C7, C8, J2, J3, J5, MD1, OP1, OP2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

Commit message: V1 schematic update 3
Parts:
- added Q1: 20V/2.9A, SAMPI:SOT23, symbol SAMPI:FET_N-CH
- C4: footprint Liem:CAP2312-6032 -> SAMPI:CAP1411
- D4, D5: footprint Liem:LED0603 -> SAMPI:LED0603; MFT Rohm Semiconductor -> Harvatek; MNP SML-D12V8WT86P -> B1911USD-20D000114U1930
- Q2, Q3: footprint (none) -> SAMPI:SOT23
- R15, R16, R23, R26, R29: footprint Liem:RES0402 -> SAMPI:RES0603; MFT Rohm Semiconductor -> YAGEO; MNP MCR01MZPJ102 -> RC0603FR-071KL
- R17, R18: footprint Liem:RES0402 -> SAMPI:RES0603; MFT Rohm Semiconductor -> YAGEO; MNP MCR01MRTJ104 -> RC0603FR-07100KL
- R21, R22: footprint Liem:RES0402 -> SAMPI:RES0603; MFT Rohm Semiconductor -> YAGEO; MNP MCR01MZPJ102 -> RC0603FR-07100RL
- R24: footprint Liem:RES0402 -> SAMPI:RES0603; MFT Rohm Semiconductor -> YAGEO; MNP MCR01MZPJ473 -> RC0603FR-0710KL
- R25, R28: footprint Liem:RES0402 -> SAMPI:RES0603; MFT Rohm Semiconductor -> YAGEO; MNP MCR01MZPJ102 -> RC0603FR-0710KL
- R27: footprint Liem:RES0402 -> SAMPI:RES0603; MNP RC0402FR-075K1L -> RC0603FR-075K1L
Connections:
- net +3V3: now also Q2.2 (S); no longer Q2.3 (D)
- net VDD_SEN: now also Q2.3 (D); no longer Q2.2 (S)
Other:
- moved on the sheet: OP1, Q2, R23, R24, R25

Commit message: V1 layout
Parts:
- removed OP1, OP2: OPTO-BJT-1CH, SAMPI:OPTO_SO4_7.6MM, symbol SAMPI:OPTO-BJT-1CH
- removed Q2, Q3: 20V/2.3A, SAMPI:SOT23, symbol SAMPI:FET_P-CH
- removed R23, R26, R29: 1K, SAMPI:RES0603, symbol SAMPI:RES
- removed R24, R25, R28: 10K, SAMPI:RES0603, symbol SAMPI:RES
- removed R27: 5.1K, SAMPI:RES0603, symbol SAMPI:RES
- removed U6, U7: ISO6740, SAMPI:SOIC16-W, symbol SAMPI:ISO6740
- added C23, C28: 10uF, SAMPI:CAP0603, symbol SAMPI:CERCAP
- added R17: 1K, SAMPI:RES0603, symbol SAMPI:RES
- added R18: 100K, SAMPI:RES0603, symbol SAMPI:RES
- added U4, U5, U6: ISO6742, SAMPI:SOIC16-W, symbol SAMPI:ISO6742
- D5: renamed from D4; footprint SAMPI:LED0603 -> SAMPI:LED3MM; MFT Harvatek -> Würth Elektronik; MNP B1911USD-20D000114U1930 -> 151031SS06000
- D6: renamed from D5; footprint SAMPI:LED0603 -> SAMPI:LED3MM; MFT Harvatek -> Würth Elektronik; MNP B1911USD-20D000114U1930 -> 151031SS06000
- J3: MNP PPTC081LGBN-RC -> PBC08SBAN
- J5: footprint SAMPI:IDC-2x5x2MM-TH -> SAMPI:IDC-2x6x2.54MM_TH; MFT Sullins Connector Solutions -> Samtec Inc.; MNP SBH21-NBPN-D05-ST-BK -> TST-106-01-T-D
- renumbered C29 to C24, C26 to C25, C4 to C26, C7 to C27, C28 to C29, C27 to C30, C8 to C31, J2 to J4, R17 to R19, R18 to R20, R15 to R21, R16 to R22, R21 to R23, R22 to R24, U1 to U7
Connections:
- net +3V3: now also C28.2, U4.10 (EN2), U4.16 (VCC2), U5.10 (EN2), U5.16 (VCC2), U6.10 (EN2), U6.16 (VCC2)
- net +3V3_ISO: now also C23.2, U4.1 (VCC1), U4.7 (EN1), U5.1 (VCC1), U5.7 (EN1), U6.1 (VCC1), U6.3 (INA), U6.7 (EN1)
- net DB_TXD: now also U6.13 (OUTB)
- net DV_RTS: now also U5.13 (OUTB)
- net DV_TXD: now also U5.14 (OUTA)
- net GND: now also J3.6, Q1.2 (S), C28.1, R18.1, U4.15 (GND2), U4.9 (GND2), U5.15 (GND2), U5.9 (GND2), U6.15 (GND2), U6.9 (GND2); no longer J3.3
- net GND_ISO: now also C23.1, U4.2 (GND1), U4.8 (GND1), U5.2 (GND1), U5.8 (GND1), U6.2 (GND1), U6.8 (GND1)
- net ISO_DB_TXD: now also U6.4 (INB)
- net ISO_DV_CTS: now also U5.6 (OUTD)
- net ISO_DV_RTS: now also U5.4 (INB)
- net ISO_DV_RXD: now also U5.5 (OUTC)
- net ISO_DV_TXD: now also U5.3 (INA)
- net ISO_PGC: now also U4.3 (INA)
- net ISO_PGD: now also U4.4 (INB)
- net PGC: now also J3.4, U4.14 (OUTA); no longer J3.5
- net PGD: now also U4.12 (INC)
- net VDD_SEN: now also J3.7, U6.14 (OUTA); no longer J3.2
- net ~{ISO_MCLR}: now also U4.6 (OUTD)
- net ~{MCLR}: now also J3.8, Q1.3 (D), U4.11 (IND); no longer J3.1
- net VTG: now reaches C26.+, C27.2, J4.1 (VCC), SW1.5 (COM2), U7.1 (VOUT)
- net at Q1.1 (G): now also R17.1, R18.2
- net at R23.1: now also U4.5 (OUTC)
- net at SW1.1 (NC1): now also J3.5; no longer J3.4
- net at SW1.3 (NO1): now also J3.1; no longer J3.8
- net at R24.2: now also U4.13 (OUTB)
- new net DB_RXD: U6.12 (INC)
- new net DV_CTS: U5.11 (IND)
- new net DV_RXD: U5.12 (INC)
- new net ISO_DB_RXD: J5.11 (DB_RXD), U6.5 (OUTC)
- new net TG_RST: R17.2
- no-connect marks 3 -> 6
Other:
- moved on the sheet: C24, C25, C26, C27, C29, C31, D5, D6, J3, J4, MD1, Q1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
