File: V1/Design/HW.ACIM-DBG/TERMINALS.kicad_sch (KiCad schematic)
At the start: 45 parts, among them J3 SNAP PINOUT, J4 MICRO USB, J5 ISO DBG PORT, Q1 40V/0.2A, SW1 PRG SEL, U4 ISO6742, U5 ISO6742, U6 ISO6742, U7 LOAD SWITCHER

Commit message: V1 layout update 3
Parts:
- added H2: NOISO DBG PORT, Liem:RPDBG, symbol Liem:RPDBG
- H1: value NO ISO DBG PORT -> NOISO DBG EXT PORT
Connections:
- net DBG_RXD: now also H2.3 (DBG_RX)
- net DBG_TXD: now also H2.1 (DBG_TXD)
- net GND: now also H2.6 (GND)
- net PGC: now also H2.10 (PGC/SWCLK)
- net PGD: now also H2.8 (PGD/SWDIO/UPDI)
- net USB_DM: now also H2.7 (USB_DM/ARX)
- net USB_DP: now also H2.5 (USB_DP/ATX)
- net USB_VBUS: now also H2.9 (USB_VBUS)
- net VDD_SEN: now also H2.4 (VDD)
- net ~{MCLR}: now also H2.2 (~{MCLR}/~{RESET})
Other:
- company: TON DUC THANG UNIVERSITY -> KiCad EDA
- moved on the sheet: BT3, H1
