File: V1/Design/HW.ACIM-DBG/TERMINALS.kicad_sch (KiCad schematic)
At the start: 46 parts, among them J3 SNAP PINOUT, J4 MICRO USB, J5 ISO DBG PORT, Q1 40V/0.2A, SW1 PRG SEL, U4 ISO6742, U5 ISO6742, U6 ISO6742, U7 LOAD SWITCHER

Commit message: V1 layout update 5
Parts:
- removed BT2: UCTRL, SAMPI:BUTTON_4P_6x6, symbol SAMPI:BT
- removed C18: 100nF, SAMPI:CAP0603, symbol SAMPI:CERCAP
- removed C23, C24, C25, C28, C29, C30: 10uF, SAMPI:CAP0603, symbol SAMPI:CERCAP
- removed C32, C33: 100pF/2kV, SAMPI:CAP1206, symbol SAMPI:CERCAP
- removed C57: 10pF, SAMPI:CAP0603, symbol SAMPI:CERCAP
- removed C58: 1nF, SAMPI:CAP0603, symbol SAMPI:CERCAP
- removed D11, D12, D13: 0.45VF, SAMPI:SOD-123FL, symbol SAMPI:DIODE-SCH
- removed Q1: 40V/0.2A, SAMPI:SOT23, symbol SAMPI:BJT-NPN
- removed R14: 3.12K, SAMPI:RES0603, symbol SAMPI:RES
- removed R16, R23: 1.1K, SAMPI:RES0603, symbol SAMPI:RES
- removed R17: 84.5R, SAMPI:RES0603, symbol SAMPI:RES
- removed R18: 2.49K, SAMPI:RES0603, symbol SAMPI:RES
- removed R24: 612R, SAMPI:RES0603, symbol SAMPI:RES
- removed R26: 10K, SAMPI:RES0603, symbol SAMPI:RES
- removed U4, U5, U6: ISO6742, SAMPI:SOIC16-W, symbol SAMPI:ISO6742
- D5: value PIC -> ICSP/UPDI
- D6: value ARM -> SWD
- H1: value NOISO DBG EXT PORT -> EXT DBG PORT
- H2: value NOISO DBG PORT -> DBG PORT
- J5: value ISO DBG PORT -> MCDBG PORT
Connections:
- net +3V3_ISO is gone; now on net VDD_SEN: J5.4 (VDD), R13.2
- net GND_ISO is gone; now on net GND: D4.K, J5.6 (GND)
- net ISO_PGC is gone; now on net PGC: J5.10 (PGC/SWDCK)
- net ISO_PGD is gone; now on net PGD: J5.8 (PGD/SWDIO)
- net ~{ISO_MCLR} is gone; now on net ~{MCLR}: J5.2 (~{RESET})
- net SWO: no longer J3.5, SW1.1 (NC1)
- net ISO_DB_RXD: no longer names the net of J5.11 (USB_DM)
- net ISO_DB_TXD: no longer names the net of J5.9 (UDB_DP)
- net ISO_DV_CTS: no longer names the net of J5.7 (DV_RXD)
- net ISO_DV_RTS: no longer names the net of J5.5 (DV_TXD)
- net ISO_DV_RXD: no longer names the net of J5.3 (DB_RXD)
- net ISO_DV_TXD: no longer names the net of J5.1 (DB_TXD)
- net ISO_UCTRL: no longer names the net of J5.12 (VBUS)
- new net: J3.5, SW1.1 (NC1)
Other:
- note removed: "ISOLATED POWER - DANGER-ZONE"
- moved on the sheet: BT3, C26, C27, C31, D4, D5, D6, H1, H2, J3, J4, J5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

Commit message: V1 layout update 6
Parts:
- D4, D5, D6: footprint SAMPI:LED3MM -> SAMPI:LED0603
Other:
- moved on the sheet: H1, H2

Commit message: V1 layout update 8
Parts:
- removed D4: TARGET, SAMPI:LED0603, symbol SAMPI:YLED
- removed R13: 1K, SAMPI:RES0603, symbol SAMPI:RES
- added Q2: MFET N, SAMPI:SOT23, symbol SAMPI:FET_N-CH
- added R3: 100K, SAMPI:RES0603, symbol SAMPI:RES
- BT3: MFT CUI -> SCHUR; MNP TS02-66-170-BK-160-SCR-D -> 1301.9304
- C26: MFT Vishay Sprague -> NCHC; MNP 293D227X96R3C2TE3 -> F930J227KBA
- C27: MFT Samsung -> TAIY; MNP CL10A106MQ8NNNC -> EMK107BBJ106MA-T
- C31: MFT Samsung -> YAGE; MNP CL10B104KB8NNNC -> CC0603ZRY5V9BB104
- D5, D6: MFT Würth Elektronik -> ROHM; MNP 151031SS06000 -> SML-D12V8WT86P
- H1: MFT (none) -> SAMT; MNP (none) -> FTSH-107-01-F-DV; now not fitted; now left out of the parts list
- H2: value DBG PORT -> RPDBG; footprint Liem:RPDBG -> Liem:DIL10-1.27-SMD; MFT (none) -> SAMT; MNP (none) -> FTSH-105-01-F-DV; now not fitted; now left out of the parts list
- J3: MFT Sullins Connector Solutions -> CHINA; MNP PBC08SBAN -> HEADER-1X40-MALE-RIGHT
- J5, MD1: now not fitted; now left out of the parts list
- R19, R20: MFT YAGEO -> NIC; MNP RC0603FR-07100KL -> NRC06F1003TRF
- R21, R22: MFT YAGEO -> ROHM; MNP RC0603FR-071KL -> MCR03PZPZFX1001
Connections:
- net GND: now also Q2.2 (S), R3.1; no longer D5.K, D6.K
- net SWO: now also J3.5, SW1.1 (NC1)
- net VDD_SEN: now also Q2.1 (G), R3.2
- net DBG_TXD2: now reaches J5.1 (DB_TXD)
- net USB2_DM: now reaches J5.11 (USB_DM)
- net USB2_VBUS: now reaches J5.12 (VBUS)
- net DBG_RXD2: now reaches J5.3 (DB_RXD)
- net AUX_TXD2: now reaches J5.5 (DV_TXD)
- net AUX_RXD2: now reaches J5.7 (DV_RXD)
- net USB2_DP: now reaches J5.9 (UDB_DP)
- net AUX_RXD renamed AUX_RXD1
- net AUX_TXD renamed AUX_TXD1
- net DBG_RXD renamed DBG_RXD1
- net DBG_TXD renamed DBG_TXD1
- net USB_DM renamed USB1_DM
- net USB_DP renamed USB1_DP
- net USB_VBUS renamed USB1_VBUS
- new net: D5.K, D6.K, Q2.3 (D)

Commit message: V1 layout update 9
Parts:
- added C1: 100nF, SAMPI:CAP0603, symbol SAMPI:CERCAP
Connections:
- net GND: now also C1.1
- net VTG: now also C1.2
Other:
- moved on the sheet: C31, U7

Commit message: V1 layout update 11
Connections:
- net USB1_DM renamed USB_RP_N
- net USB1_DP renamed USB_RP_P
- net USB1_VBUS renamed USB_RP_VBUS
- net USB2_DM renamed USB_MC_N
- net USB2_DP renamed USB_MC_P
- net USB2_VBUS renamed USB_MC_VBUS
Changed lines of the file:
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@@
 		)
 	)
-	(hierarchical_label "USB2_VBUS"
+	(hierarchical_label "USB_MC_VBUS"
 		(shape input)
 		(at 73.025 43.18 180)
@@
 		)
 	)
-	(hierarchical_label "USB2_DP"
+	(hierarchical_label "USB_MC_P"
 		(shape bidirectional)
 		(at 93.345 40.64 0)
@@
 		)
 	)
-	(hierarchical_label "USB1_VBUS"
+	(hierarchical_label "USB_RP_VBUS"
 		(shape input)
 		(at 68.58 69.85 180)
@@
 		)
 	)
-	(hierarchical_label "USB2_DM"
+	(hierarchical_label "USB_MC_N"
 		(shape bidirectional)
 		(at 93.345 43.18 0)
@@
 		)
 	)
-	(hierarchical_label "USB1_DP"
+	(hierarchical_label "USB_RP_P"
 		(shape bidirectional)
 		(at 69.215 90.805 180)
@@
 		)
 	)
-	(hierarchical_label "USB1_DM"
+	(hierarchical_label "USB_RP_N"
 		(shape bidirectional)
 		(at 69.215 93.345 180)
@@
 		)
 	)
-	(hierarchical_label "USB1_DM"
+	(hierarchical_label "USB_RP_N"
 		(shape bidirectional)
 		(at 68.58 67.31 180)
@@
 		)
 	)
-	(hierarchical_label "USB1_DP"
+	(hierarchical_label "USB_RP_P"
 		(shape bidirectional)
 		(at 68.58 64.77 180)
@@
 		)
 	)
-	(hierarchical_label "USB1_VBUS"
+	(hierarchical_label "USB_RP_VBUS"
 		(shape input)
 		(at 69.215 95.885 180)

Commit message: V1 layout update 12
Connections:
- net VTG: no longer SW1.5 (COM2)
- new net +3V3: SW1.5 (COM2)
Changed lines of the file:
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@@
-	)
-	(symbol
-		(lib_id "SAMPI:VTG")
-		(at 121.92 83.185 90)
-		(unit 1)
-		(exclude_from_sim no)
-		(in_bom yes)
-		(on_board yes)
-		(dnp no)
-		(property "Reference" "#PWR062"
-			(at 125.73 83.185 0)
-			(effects
-				(font
-					(face "Consolas")
-					(size 1.27 1.27)
-					(thickness 0.254)
-					(bold yes)
-				)
-				(hide yes)
-			)
-		)
-		(property "Value" "VTG"
-			(at 116.84 83.185 90)
-			(effects
-				(font
-					(face "Consolas")
-					(size 1.016 1.016)
-					(thickness 0.127)
-				)
-			)
-		)
-		(property "Footprint" ""
-			(at 121.92 83.185 0)
-			(effects
-				(font
-					(face "Consolas")
-					(size 1.016 1.016)
-					(thickness 0.127)
-				)
-				(hide yes)
-			)
-		)
-		(property "Datasheet" ""
-			(at 121.92 83.185 0)
-			(effects
-				(font
-					(face "Consolas")
-					(size 1.016 1.016)
-					(thickness 0.127)
-				)
-				(hide yes)
-			)
-		)
-		(property "Description" "Power symbol creates a global label with name \"VTG\""
-			(at 121.92 83.185 0)
-			(effects
-				(font
-					(face "Consolas")
-					(size 1.016 1.016)
-					(thickness 0.127)
-				)
-				(hide yes)
-			)
-		)
-		(pin "1"
-		)
-		(instances
-			(project "HW.ACIM-DBG"
-				(path "/20f80521-75f2-4ccc-bb34-c9566e70ef5c/41f97a9f-5331-4d01-9d06-5e4a321167bc"
-					(reference "#PWR062")
-					(unit 1)
-				)
-			)
-		)
 	)
 	(symbol
@@
 					(unit 1)
 				)
+			)
+		)
+	)
+	(symbol
+		(lib_id "power:+3V3")
+		(at 121.92 83.185 90)
+		(mirror x)
+		(unit 1)
+		(exclude_from_sim no)
+		(in_bom yes)
+		(on_board yes)
+		(dnp no)
+		(property "Reference" "#PWR045"
+			(at 125.73 83.185 0)
+			(effects
+				(font
+					(face "Consolas")
+					(size 1.27 1.27)
+					(thickness 0.254)
+					(bold yes)
+				)
+				(hide yes)
+			)
+		)
+		(property "Value" "+3V3"
+			(at 117.475 83.185 90)
+			(effects
+				(font
+					(face "Consolas")
+					(size 1.016 1.016)
+				)
+			)
+		)
+		(property "Footprint" ""
+			(at 121.92 83.185 0)
+			(effects
+				(font
+					(face "Consolas")
+					(size 1.016 1.016)
+					(thickness 0.254)
+				)
+				(hide yes)
+			)
+		)
+		(property "Datasheet" ""
+			(at 121.92 83.185 0)
+			(effects
+				(font
+					(face "Consolas")
+					(size 1.016 1.016)
+					(thickness 0.254)
+				)
+				(hide yes)
+			)
+		)
+		(property "Description" ""
+			(at 121.92 83.185 0)
+			(effects
+				(font
+					(face "Consolas")
+					(size 1.016 1.016)
+					(thickness 0.254)
+				)
+				(hide yes)
+			)
+		)
+		(pin "1"
+		)
+		(instances
+			(project "HW.ACIM-DBG"
+				(path "/20f80521-75f2-4ccc-bb34-c9566e70ef5c/41f97a9f-5331-4d01-9d06-5e4a321167bc"
+					(reference "#PWR045")
+					(unit 1)
+				)

Commit message: V1 layout update 13
Parts:
- J5: now fitted; now in the parts list
Changed lines of the file:
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@@
 		(unit 1)
 		(exclude_from_sim no)
-		(in_bom no)
+		(in_bom yes)
 		(on_board yes)
-		(dnp yes)
+		(dnp no)
 		(property "Reference" "J5"
 			(at 83.185 25.4 0)

Commit message: V1 layout update 16
Parts:
- H1: value EXT DBG PORT -> RPDBG EXT; now fitted; now in the parts list
- H2: now fitted; now in the parts list
- J5: value MCDBG PORT -> MCDBG
Changed lines of the file:
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@@
 		(unit 1)
 		(exclude_from_sim no)
-		(in_bom no)
-		(on_board yes)
-		(dnp yes)
+		(in_bom yes)
+		(on_board yes)
+		(dnp no)
 		(property "Reference" "H1"
 			(at 83.185 54.61 0)
@@
 			)
 		)
-		(property "Value" "EXT DBG PORT"
+		(property "Value" "RPDBG EXT"
 			(at 83.185 56.515 0)
 			(effects
@@
 			)
 		)
-		(property "Value" "MCDBG PORT"
+		(property "Value" "MCDBG"
 			(at 83.185 27.305 0)
 			(effects
@@
 		(unit 1)
 		(exclude_from_sim no)
-		(in_bom no)
-		(on_board yes)
-		(dnp yes)
+		(in_bom yes)
+		(on_board yes)
+		(dnp no)
 		(property "Reference" "H2"
 			(at 82.55 80.645 0)
