File: V1/Design/HW.ACIM-DBG/TERMINALS.kicad_sch (KiCad schematic)
At the start: 21 parts, among them J3 SNAP PINOUT, J4 MICRO USB, J5 MCDBG, Q2 MFET N, SW1 PRG SEL, U7 LOAD SWITCHER

Commit message: Production HW.ACIM-DBG_V1.0 update BoM
Parts:
- C26: value 220uF -> 4.7uF; MFT NCHC -> Cal-Chip; MNP F930J227KBA -> GMC31X7R475K10NT
Changed lines of the file:
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@@
 (kicad_sch
-	(version 20231120)
+	(version 20250114)
 	(generator "eeschema")
-	(generator_version "8.0")
+	(generator_version "9.0")
 	(paper "A4")
 	(title_block
@@
 		(dnp no)
 		(property "Reference" "C26"
-			(at 210.185 67.31 90)
+			(at 210.82 67.31 90)
 			(effects
 				(font
@@
 			)
 		)
-		(property "Value" "220uF"
+		(property "Value" "4.7uF"
 			(at 212.09 69.85 90)
 			(effects
@@
 			)
 		)
-		(property "Description" "CAP TANT SMD 1411 220uF 6.3V 10% 1.2OHM WxLxH(2.8x3.5x2.3)"
+		(property "Description" "CAP CER 4.7UF 10V X7R 1206"
 			(at 203.2 67.31 0)
 			(effects
@@
 			)
 		)
-		(property "MNP" "F930J227KBA"
+		(property "MNP" "GMC31X7R475K10NT"
 			(at 203.2 67.31 0)
 			(effects
@@
 			)
 		)
-		(property "MFT" "NCHC"
+		(property "MFT" "Cal-Chip"
 			(at 203.2 67.31 0)
 			(effects
