File: V1/Design/HW.ACIM-DBG/USB_HUB.kicad_sch (KiCad schematic)
At the start: 60 parts, among them J4 USB, U2 USB HUB 2.0 4-CH, U4 24MHz (3225), U9 USB HUB

Commit message: V1 schematic update 1
Parts:
- removed C19, C21, C22: 100nF, SAMPI:CAP0603, symbol SAMPI:CERCAP
- removed C20, C23, C27, C28, C29, C30, C31: 10nF, SAMPI:CAP0603, symbol SAMPI:CERCAP
- removed C24, C25: 22pF, SAMPI:CAP0603, symbol SAMPI:CERCAP
- removed C26: 10uF, SAMPI:CAP0603, symbol SAMPI:CERCAP
- removed C55: 220uF/6.3V, SAMPI:CAP1411, symbol SAMPI:ELECCAP
- removed CB1: JACK USB C, symbol SAMPI:CABLE1
- removed D1: TVS 5.5V 3-CH, SAMPI:SOT143B_NEXT, symbol SAM1:TVS_3CH
- removed D6: VISO, SAMPI:LED0603, symbol SAMPI:WLED
- removed F1: 500mA, SAMPI:FUSE0805, symbol SAM1:FUSE
- removed FT1: 120R@100MHz, SAMPI:FT0603, symbol SAM1:FerriteBead
- removed FT2: 2x 120R@100MHz, SAMPI:IND1210_4P, symbol SAMPI:IND1210_4P
- removed FT4, FT5: 120R@100MHz, SAMPI:FT0603, symbol SAMPI:FerriteBead
- removed J4: USB, SAMPI:HDM-1x4x2.54-TH-RA, symbol SAMPI:SIL04-1
- removed R11, R12, R58, R59, R60, R61: 47K, SAMPI:RES0603, symbol SAMPI:RES
- removed R13, R14: 100K, SAMPI:RES0603, symbol SAMPI:RES
- removed R43, R44, R45, R46, R47, R48, R49, R56, R57: 0R, SAMPI:RES0603, symbol SAMPI:RES
- removed TP1, TP3: 5V, SAMPI:TP1MM, symbol SAMPI:TESTPOINT
- removed TP2: 0V, SAMPI:TP1MM, symbol SAMPI:TESTPOINT
- removed TP4: 3V3, SAMPI:TP1MM, symbol SAMPI:TESTPOINT
- removed TP5: GND, SAMPI:TP1MM, symbol SAMPI:TESTPOINT
- removed U2: USB HUB 2.0 4-CH, SAMPI:SQFN36_6x6_MCHP, symbol SAMPI:USB2514B
- removed U4: 24MHz (3225), SAMPI:CDFN3225-4LD-PL-1, symbol SAMPI:OSC
- removed U9: USB HUB, symbol SAMPI:USB2422
- added C1, C2: 220uF, Liem:CAP2312-6032, symbol SAMPI:ELECCAP
- added C10, C11, C15, C9: 22pF, Liem:CAP0402, symbol SAMPI:CERCAP
- added C12: 1uF, Liem:CAP0402, symbol SAMPI:CERCAP
- added C13, C16, C4: 100nF, Liem:CAP0402, symbol SAMPI:CERCAP
- added C6: 10uF, Liem:CAP0603, symbol SAMPI:CERCAP
- added D1: TVS 5.5V, Liem:SOT143B_NEXT, symbol Liem:PRTR5V0U2X
- added F1: 750mA, tuanlib:FUSE_ 1206, symbol Liem:FUSE
- added J1: USB C, Liem:USB4105, symbol Liem:USB4105
- added R3, R4: 100K, Liem:RES0402, symbol SAMPI:RES
- added TP1: 5V, tuanlib:TestPoint, symbol My_Library:TestPoint
- added TP2: 3V3, tuanlib:TestPoint, symbol My_Library:TestPoint
- added U2: LDO 3.3V, Liem:DFN8_3x3_MCHP, symbol Liem:MCP1727
- added U3: USB HUB, Package_DFN_QFN:QFN-24-1EP_4x4mm_P0.5mm_EP2.8x2.8mm, symbol SAMPI:USB2422
- added Y1: 24MHz, Liem:CDFN3225-4LD-PL-1, symbol TUANLIB:FA-20H
- C14: value 22pF -> 100nF; footprint SAMPI:CAP0603 -> Liem:CAP0402; Checked OK -> (none); MFT Walsin -> Walsin Technology Corporation; MNP 0603N220J500CT -> 0402B104K160CT; Unit Price 0.012 -> (none)
- C17, C3: footprint SAMPI:CAP0603 -> Liem:CAP0402; Checked OK -> (none); MFT Samsung -> Walsin Technology Corporation; MNP CL10B104KB8NNNC -> 0402B104K160CT; Unit Price 0.0146 -> (none)
- C18: value 22pF -> 1uF; footprint SAMPI:CAP0603 -> Liem:CAP0402; Checked OK -> (none); MFT Walsin -> Murata Electronics; MNP 0603N220J500CT -> GRM155R60J105KE19D; Unit Price 0.012 -> (none); now fitted; now in the parts list
- R1: value 1.1K -> 5.1K, 1%; footprint SAMPI:RES0603 -> Liem:RES0402; Checked OK -> (none); MNP AC0603FR-071K1L -> RC0402FR-075K1L; Unit Price 0.021 -> (none)
- R10: footprint SAMPI:RES0603 -> Liem:RES0402; Checked OK -> (none); MFT YAGEO -> Rohm Semiconductor; MNP RC0603FR-0747KL -> MCR01MZPJ473; Unit Price 0.019 -> (none)
- R2: value 0R -> 5.1K, 1%; footprint SAMPI:RES0603 -> Liem:RES0402; Checked OK -> (none); MNP RC0603JR-070RL -> RC0402FR-075K1L; Unit Price 0.015 -> (none)
- R5: value 10K -> 100K; footprint SAMPI:RES0603 -> Liem:RES0402; Checked OK -> (none); MFT YAGEO -> Rohm Semiconductor; MNP RC0603FR-0710KL -> MCR01MRTJ104; Unit Price 0.019 -> (none)
- R6: value 10K -> 12K, 1%; footprint SAMPI:RES0603 -> Liem:RES0402; Checked OK -> (none); MNP RC0603FR-0710KL -> RC0402FR-0712KL; Unit Price 0.019 -> (none)
- R7: value 10K -> 47K; footprint SAMPI:RES0603 -> Liem:RES0402; Checked OK -> (none); MFT YAGEO -> Rohm Semiconductor; MNP RC0603FR-0710KL -> MCR01MZPJ473; Unit Price 0.019 -> (none)
- R8: value 0R -> 47K; footprint SAMPI:RES0603 -> Liem:RES0402; Checked OK -> (none); MFT YAGEO -> Rohm Semiconductor; MNP RC0603JR-070RL -> MCR01MZPJ473; Unit Price 0.015 -> (none)
- R9: value 12K/1% -> 47K; footprint SAMPI:RES0603 -> Liem:RES0402; Checked OK -> (none); MFT YAGEO -> Rohm Semiconductor; MNP RC0603FR-0712KL -> MCR01MZPJ473; Unit Price 0.019 -> (none); now not fitted; now left out of the parts list
Connections:
- net +5V_ISO is gone; now on net +5V: C3.2
- net +3V3: now also C14.2, C17.2, C18.2, R10.1, R5.2, C6.2, TP2.1, U2.7 (SEN/ADJ), U2.8 (VOUT), U3.1 (VDD33), U3.18 (VDD33), U3.9 (VDD33); no longer R5.1
- net +5V: now also C1.+, C2.+, C4.2, D1.4 (VCC), F1.2, R3.2, TP1.1, U2.1 (VIN1), U2.2 (VIN2), U2.3 (~{SHDN}); no longer R6.1
- net GND: now also C3.1, R1.1, R2.1, R6.1, R7.1, R8.1, R9.1, C1.-, C10.1, C11.1, C12.1, C13.1, C15.1, C16.1, C2.-, C4.1, C6.1, C9.1, D1.1 (GND), J1.A1B12 (GND), J1.B1A12 (GND), J1.S1, J1.S2, J1.S3, J1.S4, R4.1, U2.4 (GND), U2.5 (PWRGD), U2.9 (EP), U3.25 (VSS), U3.6 (TEST), Y1.2, Y1.4; no longer R10.2, R7.2, R9.2
- net at R8.2: now also U3.14 (SCL/SMBCLK/CFG_SEL0)
- net GND_ISO: no longer names the net of R1.2
- net GND_ISO: now also J1.B5 (CC2); no longer C3.1
- net PSU_VBUS: no longer names the net of R2.2
- net PSU_VBUS: now also J1.A5 (CC1)
- removed net SYS_CLK: C18.2, R8.1
- new net: C9.2, U3.22 (XTALIN/CLKIN), Y1.1
- new net: C11.2, U3.21 (XTALOUT/CLKIN_EN), Y1.3
- new net: C16.2, R5.1, U3.15 (~{RESET})
- new net: R7.2, U3.13 (SDA/SMBDATA/NON_REM1)
- new net: C13.2, C15.2, U3.23 (PLLFILT)
- new net: F1.1, J1.A4B9 (VBUS), J1.B4A9 (VBUS)
- new net: R10.2, R9.2, U3.17 (SUSP_IND/LOCAL_PWR/NON_REM0)
- new net: C10.2, C12.2, U3.10 (CRFILT)
- new net: R6.2, U3.24 (RBIAS)
- new net HUB_USB_VBUS: R3.1, R4.2, U3.16 (VBUS_DET)
- new net USB1_N: U3.2 (USBDM_DN1)
- new net USB1_P: U3.3 (USBDP_DN1)
- new net USB1_PWR_EN: U3.7 (PRTPWR1/BC_EN1)
- new net USB2_N: U3.4 (USBDM_DN2)
- new net USB2_P: U3.5 (USBDP_DN2)
- new net USB2_PWR_EN: U3.11 (PRTPWR2/BC_EN2)
- new net USB_N: D1.2 (I/O1), J1.A7 (DN1), J1.B7 (DN2), U3.19 (USBDM_UP)
- new net USB_P: D1.3 (I/O2), J1.A6 (DP1), J1.B6 (DP2), U3.20 (USBDP_UP)
- no-connect marks 8 -> 5
Other:
- note removed: "ISOLATED USB"

Commit message: V1 schematic update 2
Parts:
- removed C4: 100nF, Liem:CAP0402, symbol SAMPI:CERCAP
Connections:
- net +3V3: now also C1.+; no longer C6.2
- net +5V: now also C6.2; no longer C1.+
Other:
- moved on the sheet: C1, C10, C12, C13, C14, C15, C16, C17, C18, C2, C3, C6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

Commit message: V1 schematic update 3
Parts:
- C1, C2: footprint Liem:CAP2312-6032 -> SAMPI:CAP1411
- C10, C11, C15, C9: footprint Liem:CAP0402 -> SAMPI:CAP0603; MFT YAGEO -> Walsin; MNP AC0402JRNPO9BN220 -> 0603N220J500CT
- C12, C18: footprint Liem:CAP0402 -> SAMPI:CAP0603; MFT Murata Electronics -> Samsung; MNP GRM155R60J105KE19D -> CL10B105KP8NNNC
- C13, C14, C16, C17, C3: footprint Liem:CAP0402 -> SAMPI:CAP0603; MFT Walsin Technology Corporation -> Samsung; MNP 0402B104K160CT -> CL10B104KB8NNNC
- C6: footprint Liem:CAP0603 -> SAMPI:CAP0603; MFT KEMET -> Samsung; MNP C0603C106M8PACTU -> CL10A106MQ8NNNC
- D1: footprint Liem:SOT143B_NEXT -> SAMPI:SOT143B_NEXT; MFT Nexperia USA Inc. -> Nexperia
- F1: value 750mA -> 500mA; footprint tuanlib:FUSE_ 1206 -> SAMPI:FUSE0805; MFT SCHURTER Inc. -> Littelfuse; MNP 3413.0114.22 -> 0805L050WR
- J1: footprint Liem:USB4105 -> SAMPI:USB4105
- R1, R2: value 5.1K, 1% -> 5.1K; footprint Liem:RES0402 -> SAMPI:RES0603; MNP RC0402FR-075K1L -> RC0603FR-075K1L
- R10, R7, R8: footprint Liem:RES0402 -> SAMPI:RES0603; MFT Rohm Semiconductor -> YAGEO; MNP MCR01MZPJ473 -> RC0603FR-0747KL
- R3, R4, R5: footprint Liem:RES0402 -> SAMPI:RES0603; MFT Rohm Semiconductor -> YAGEO; MNP MCR01MRTJ104 -> RC0603FR-07100KL
- R6: value 12K, 1% -> 12K; footprint Liem:RES0402 -> SAMPI:RES0603; MNP RC0402FR-0712KL -> RC0603FR-0712KL
- TP1, TP2: footprint tuanlib:TestPoint -> SAMPI:TP1MM
- U2: footprint Liem:DFN8_3x3_MCHP -> SAMPI:DFN8_3x3_MCHP
- U3: footprint Package_DFN_QFN:QFN-24-1EP_4x4mm_P0.5mm_EP2.8x2.8mm -> SAMPI:QFN-24-4x4-EP
- Y1: footprint Liem:CDFN3225-4LD-PL-1 -> SAMPI:CDFN3225-4LD-PL-1

Commit message: V1 layout
Parts:
- removed TP1: 5V, SAMPI:TP1MM, symbol My_Library:TestPoint
- removed TP2: 3V3, SAMPI:TP1MM, symbol My_Library:TestPoint
- added C2, C5: 100nF, SAMPI:CAP0603, symbol SAMPI:CERCAP
- renumbered C6 to C1, C12 to C10, C14 to C11, C13 to C12, C17 to C13, C15 to C14, C16 to C15, C18 to C16, C2 to C3, C3 to C4, C1 to C6, C9 to C7, C10 to C8, C11 to C9, R6 to R5, R5 to R6, U2 to U1, U3 to U2
Connections:
- net GND: now also C2.1, C5.1
- net HUB_USB_VBUS: now also C2.2
- net at U1.6 (CDELAY): now also C5.2
- no-connect marks 5 -> 4
Other:
- moved on the sheet: C3, C4, C6

Commit message: V1 layout update 1
Connections:
- net USB_N: now also D1.3 (I/O2); no longer D1.2 (I/O1)
- net USB_P: now also D1.2 (I/O1); no longer D1.3 (I/O2)

Commit message: V1 layout update 2
Parts:
- removed U2: USB HUB, SAMPI:QFN-24-4x4-EP, symbol SAMPI:USB2422
- added BT1: RESET, SAMPI:BUTTON_4P_6x6, symbol SAMPI:BT
- added C17, C38: 100nF, SAMPI:CAP0603, symbol SAMPI:CERCAP
- added C34, C35, C37: 10nF, SAMPI:CAP0603, symbol SAMPI:CERCAP
- added C36: 10uF, SAMPI:CAP0603, symbol SAMPI:CERCAP
- added C39: 22pF, SAMPI:CAP0603, symbol SAMPI:CERCAP
- added D3: POWER, SAMPI:LED3MM, symbol SAMPI:RLED
- added FT1, FT2: 120R@100MHz, SAMPI:FT0603, symbol SAMPI:FerriteBead
- added R11: 1K, SAMPI:RES0603, symbol SAMPI:RES
- added R12, R34, R35: 10K, SAMPI:RES0603, symbol SAMPI:RES
- added R25: 100K, SAMPI:RES0603, symbol SAMPI:RES
- added U2: USB HUB 2.0 4-CH, SAMPI:SQFN36_6x6_MCHP, symbol SAMPI:USB2514B
- C10: value 1uF -> 100nF; MNP CL10B105KP8NNNC -> CL10B104KB8NNNC
- C11, C12: value 100nF -> 10nF; MFT Samsung -> YAGEO; MNP CL10B104KB8NNNC -> CC0603KRX7R9BB103
- C13: value 100nF -> 22pF; MFT Samsung -> Walsin; MNP CL10B104KB8NNNC -> 0603N220J500CT
- C14: value 22pF -> 10nF; MFT Walsin -> YAGEO; MNP 0603N220J500CT -> CC0603KRX7R9BB103
- C16: value 1uF -> 10nF; MFT Samsung -> YAGEO; MNP CL10B105KP8NNNC -> CC0603KRX7R9BB103
- R10: value 47K -> 100K; MNP RC0603FR-0747KL -> RC0603FR-07100KL
- R5: value 12K -> 10K; MNP RC0603FR-0712KL -> RC0603FR-0710KL
- R6: value 100K -> 12K/1%; MNP RC0603FR-07100KL -> RC0603FR-0712KL
- R9: footprint Liem:RES0402 -> SAMPI:RES0603; MFT Rohm Semiconductor -> YAGEO; MNP MCR01MZPJ473 -> RC0603FR-0747KL; now fitted; now in the parts list
Connections:
- net +3V3: now also C8.2, R5.1, R8.2, FT1.1, FT2.1; no longer C11.2, C16.2, R10.1, R6.2
- net +5V: now also R12.2, R34.1; no longer U1.3 (~{SHDN})
- net GND: now also R10.1, R6.2, R7.2, BT1.3, BT1.4, C17.1, C34.1, C35.1, C36.1, C37.1, C38.1, C39.1, D3.K, R25.1, R35.2, U2.11 (TEST), U2.37 (VSS); no longer R5.1, R7.1, R8.1
- net USB1_N: now also U2.1 (USBDM_DN1)
- net USB1_P: now also U2.2 (USBDP_DN1)
- net USB2_N: now also U2.3 (USBDM_DN2)
- net USB2_P: now also U2.4 (USBDP_DN2)
- net USB_N: now also U2.30 (USBDM_UP)
- net USB_P: now also U2.31 (USBDP_UP)
- net XTALIN: now reaches C7.2, Y1.1
- net XTALIN: now also U2.33 (XTALIN/CLKIN)
- net XTALOUT: now reaches C9.2, Y1.3
- net XTALOUT: now also U2.32 (XTALOUT)
- net at C15.2: now also C35.2, U2.34 (PLLFILT); no longer R6.1
- net at C14.2: now also C11.2, C34.2, C37.2, FT1.2, U2.10 (VDDA33), U2.29 (VDDA33), U2.36 (VDDA33), U2.5 (VDDA33); no longer C12.2
- net at R10.2: now also U2.24 (SCL/SMBCLK/CFG_SEL0); no longer R9.2
- net at C10.2: now also C12.2, U2.14 (CRFILT); no longer C8.2
- net at R5.2: now also C38.2, U2.26 (~{RESET})
- new net: C16.2, C36.2, FT2.2, U2.15 (VDD33), U2.23 (VDD33)
- new net: D3.A, R11.1
- new net: R9.2, U2.28 (SUSP_IND/LOCAL_PWR/NON_REM0)
- new net: BT1.1, BT1.2, C17.2, R12.1, U1.3 (~{SHDN})
- new net: R6.1, U2.35 (RBIAS)
- new net: C39.2, R34.2, R35.1, U2.27 (VBUS_DET)
- new net: R7.1, U2.22 (SDA/SMBDATA/NON_REM1)
- new net: R25.2, R8.1, U2.25 (HS_IND/CFG_SEL1)
- new net MODE_SLED: R11.2
- new net USB1_VBUS: U2.12 (PRTPWR1/BC_EN1)
- new net USB2_VBUS: U2.16 (PRTPWR2/BC_EN2)
- new net USB3_N: U2.6 (USBDM_DN3)
- new net USB3_P: U2.7 (USBDP_DN3)
- new net USB3_VBUS: U2.18 (PRTPWR3/BC_EN3)
- new net USB4_N: U2.8 (USBDM_DN4)
- new net USB4_P: U2.9 (USBDP_DN4)
- new net USB4_VBUS: U2.20 (PRTPWR4/BC_EN4)
- no-connect marks 4 -> 8
Other:
- moved on the sheet: C1, C5, C6, C7, C9, U1, Y1

Commit message: V1 layout update 3
Parts:
- removed C2: 100nF, SAMPI:CAP0603, symbol SAMPI:CERCAP
- removed R3, R4: 100K, SAMPI:RES0603, symbol SAMPI:RES
Connections:
- net MODE_SLED is gone; now on net +3V3: R11.2
- net GND: now also C5.2; no longer C5.1, U1.5 (PWRGD)
- net at D3.A, R11.1: now also U1.5 (PWRGD)
- net at U1.6 (CDELAY): now also C5.1; no longer C5.2
- no-connect marks 8 -> 6
Other:
- company: TON DUC THANG UNIVERSITY -> KiCad EDA
- moved on the sheet: BT1, C1, C17, C3, C39, C4, C5, C6, D3, R11, R12, R34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

Commit message: V1 layout update 6
Parts:
- removed F1: 500mA, SAMPI:FUSE0805, symbol Liem:FUSE
- added C2: 100nF, SAMPI:CAP0603, symbol SAMPI:CERCAP
- added Q2: MFET N, SAMPI:SOT23, symbol SAMPI:FET_N-CH
- added R14, R17: 5.1K, SAMPI:RES0603, symbol SAMPI:RES
- added R15, R16: 35.7K, SAMPI:RES0603, symbol SAMPI:RES
- added R18, R23, R24, R26, R3, R4: 10K, SAMPI:RES0603, symbol SAMPI:RES
- added U4: USB PD, SAMPI:QFN16, symbol Liem:UTC2000
- added U5: eFuse, SAMPI:DFN10-EP-3x3, symbol SAMPI:eFUSE
- D3: footprint SAMPI:LED3MM -> SAMPI:LED0603
- R12: value 10K -> 1K; MNP RC0603FR-0710KL -> RC0603FR-071KL
Connections:
- net +5V: now also U1.3 (~{SHDN}), R23.2, U5.10 (VOUT), U5.9 (VOUT); no longer C1.2, D1.4 (VCC), R12.2
- net GND: now also R12.1, C2.1, Q2.2 (S), R14.1, R17.1, U4.13 (VSS), U4.17 (EP), U5.11 (GND), U5.6 (GND)
- net at J1.A5 (CC1), R2.2: now also R3.2
- net at J1.B5 (CC2), R1.2: now also R4.2
- net at BT1.1, BT1.2, C17.2: now also Q2.3 (D), R18.1, U5.4 (EN/UVLO); no longer R12.1, U1.3 (~{SHDN})
- net VBUS: now reaches J1.A4B9 (VBUS), J1.B4A9 (VBUS)
- net VBUS: now also C1.2, D1.4 (VCC), R15.2, R16.2, R18.2, R24.1, R26.1, U4.16 (VDD), U5.1 (VIN), U5.2 (VIN)
- new net: R26.2, U4.2 (CFG_SEL)
- new net: R14.2, R15.1, U4.12 (VMON)
- new net: C2.2, U5.3 (SS)
- new net: R16.1, R17.2, U5.7 (OVP)
- new net: Q2.1 (G), U4.5 (AUDIO_ADAPTER/~{CONNECTED})
- new net: R23.1, U4.1 (~{OCS}), U5.8 (PGD)
- new net: R24.2, U4.3 (ENABLE)
- new net: R12.2, U5.5 (ILIM/IMON)
- new net CC1: R3.1, U4.7 (CC1)
- new net CC2: R4.1, U4.6 (CC2)
- new net FAULT_IND: U4.4 (FAULT_IND)
- no-connect marks 6 -> 7
Other:
- moved on the sheet: BT1, C1, C10, C11, C12, C13, C14, C15, C16, C17, C3, C34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
