File: V1/Design/HW.ACIM-DBG/USB_HUB.kicad_sch (KiCad schematic)
At the start: 58 parts, among them J1 USB C, Q2 MFET N, U1 LDO 3.3V, U2 USB HUB 2.0 4-CH, U4 USB PD, U5 eFuse, Y1 24MHz

Commit message: V1 layout update 7
Parts:
- added R30: 100K, SAMPI:RES0603, symbol SAMPI:RES
- R16: value 35.7K -> 40.2K, 1%
- R17: value 5.1K -> 10K, 1%
Connections:
- net +5V: now also C1.2, R24.1, R26.1, U4.16 (VDD)
- net GND: now also R30.2
- net VBUS: no longer C1.2, R24.1, R26.1, U4.16 (VDD)
- net at Q2.1 (G), U4.5 (AUDIO_ADAPTER/~{CONNECTED}): now also R30.1
Other:
- note added: "Rovpt=(Rovpb*(Vinmax-Vovp))/Vovp Rovpb=10k Vovp=1.2V Vinmax=6V Rovpt=(10k*(6-1.2))/1.2 =40k => Rovpt=40.2k Ilim=20600*Vocp/Rset Vocp=0.6V => Rset=20600*Vocp/Ilim =20600*0.6/3 =4120Ohm"
- moved on the sheet: C38, R5

Commit message: V1 layout update 8
Parts:
- removed C1: 10uF, SAMPI:CAP0603, symbol SAMPI:CERCAP
- removed C2: 100nF, SAMPI:CAP0603, symbol SAMPI:CERCAP
- removed Q2: MFET N, SAMPI:SOT23, symbol SAMPI:FET_N-CH
- removed R12: 1K, SAMPI:RES0603, symbol SAMPI:RES
- removed R14: 5.1K, SAMPI:RES0603, symbol SAMPI:RES
- removed R15: 35.7K, SAMPI:RES0603, symbol SAMPI:RES
- removed R16: 40.2K, 1%, SAMPI:RES0603, symbol SAMPI:RES
- removed R17: 10K, 1%, SAMPI:RES0603, symbol SAMPI:RES
- removed R23, R24, R26, R3, R4: 10K, SAMPI:RES0603, symbol SAMPI:RES
- removed R30: 100K, SAMPI:RES0603, symbol SAMPI:RES
- removed U4: USB PD, SAMPI:QFN16, symbol Liem:UTC2000
- removed U5: eFuse, SAMPI:DFN10-EP-3x3, symbol SAMPI:eFUSE
- added F1: 750mA, Liem:FUSE1812, symbol Liem:FUSE
- BT1: MFT CUI -> SCHUR; MNP TS02-66-170-BK-160-SCR-D -> 1301.9304
- C10, C15, C17, C38, C4, C5: MFT Samsung -> YAGE; MNP CL10B104KB8NNNC -> CC0603ZRY5V9BB104
- C11, C12, C14, C16, C34, C35, C37: MFT YAGEO -> MRTN; MNP CC0603KRX7R9BB103 -> GRM188R71H103KA01D
- C13, C39, C7, C8, C9: MFT Walsin -> YAGE; MNP 0603N220J500CT -> CC0603JRNPO9BN220
- C3, C6: MFT Vishay Sprague -> NCHC; MNP 293D227X96R3C2TE3 -> F930J227KBA
- C36: MFT Samsung -> TAIY; MNP CL10A106MQ8NNNC -> EMK107BBJ106MA-T
- D3: MFT Würth Elektronik -> ROHM; MNP 151031VS06000 -> SML-D12M8WT86
- FT1, FT2: MFT Pulse -> TDK; MNP PE-0603PFB121ST -> MPZ1608S121ATAH0
- R1, R2: MFT YAGEO -> YAGE
- R10, R25: MFT YAGEO -> NIC; MNP RC0603FR-07100KL -> NRC06F1003TRF
- R11: MFT YAGEO -> ROHM; MNP RC0603FR-071KL -> MCR03PZPZFX1001
- R6: value 12K/1% -> 12K
- Y1: footprint SAMPI:CDFN3225-4LD-PL-1 -> SAMPI:CDFN2520-ABM10; MFT Abracon LLC -> CTSF; MNP ABM8AIG-24.000MHZ-12-2Z-T3 -> 425F35B024M0000
Connections:
- net +5V: now also D1.4 (VCC), R18.2, F1.2; no longer U1.3 (~{SHDN})
- net at BT1.1, BT1.2, C17.2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: now also U1.3 (~{SHDN})
- net VBUS: no longer names the net of J1.A4B9 (VBUS), J1.B4A9 (VBUS)
- net VBUS: now also F1.1; no longer D1.4 (VCC), R18.2
- no-connect marks 7 -> 6
Other:
- note removed: "Rovpt=(Rovpb*(Vinmax-Vovp))/Vovp Rovpb=10k Vovp=1.2V Vinmax=6V Rovpt=(10k*(6-1.2))/1.2 =40k => Rovpt=40.2k Ilim=20600*Vocp/Rset Vocp=0.6V => Rset=20600*Vocp/Ilim =20600*0.6/3 =4120Ohm"
- moved on the sheet: BT1, C17, C3, C4, C5, C6, D1, D3, J1, R1, R11, R18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

Commit message: V1 layout update 11
Parts:
- added C2: 100nF, SAMPI:CAP0603, symbol SAMPI:CERCAP
Connections:
- net +3V3: now also C2.2
- net GND: now also C2.1
- net XTALIN: now also C9.2, Y1.3; no longer C7.2, Y1.1
- net XTALOUT: now also C7.2, Y1.1; no longer C9.2, Y1.3
Other:
- moved on the sheet: C6
Changed lines of the file:
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@@
 	)
 	(junction
-		(at 270.51 66.675)
-		(diameter 0)
-		(color 0 0 0 0)
-	)
-	(junction
 		(at 54.61 62.23)
 		(diameter 0)
@@
 	)
 	(junction
+		(at 257.81 66.675)
+		(diameter 0)
+		(color 0 0 0 0)
+	)
+	(junction
 		(at 247.65 89.535)
 		(diameter 0)
@@
 	)
 	(junction
+		(at 270.51 66.675)
+		(diameter 0)
+		(color 0 0 0 0)
+	)
+	(junction
 		(at 54.61 64.77)
 		(diameter 0)
@@
 	)
 	(junction
-		(at 257.81 66.675)
-		(diameter 0)
-		(color 0 0 0 0)
-	)
-	(junction
 		(at 148.59 52.07)
 		(diameter 0)
@@
 	(wire
 		(pts
+			(xy 257.81 66.675) (xy 259.715 66.675)
+		)
+		(stroke
+			(width 0)
+			(type default)
+		)
+	)
+	(wire
+		(pts
 			(xy 199.39 158.75) (xy 205.74 158.75)
 		)
@@
 	(wire
 		(pts
+			(xy 158.75 52.07) (xy 158.75 53.34)
+		)
+		(stroke
+			(width 0)
+			(type default)
+		)
+	)
+	(wire
+		(pts
 			(xy 186.69 59.69) (xy 195.58 59.69)
 		)
@@
 	(wire
 		(pts
+			(xy 256.54 66.675) (xy 257.81 66.675)
+		)
+		(stroke
+			(width 0)
+			(type default)
+		)
+	)
+	(wire
+		(pts
 			(xy 227.33 137.795) (xy 226.06 137.795)
 		)
@@
 	(wire
 		(pts
+			(xy 270.51 66.675) (xy 271.78 66.675)
+		)
+		(stroke
+			(width 0)
+			(type default)
+		)
+	)
+	(wire
+		(pts
 			(xy 227.33 89.535) (xy 237.49 89.535)
 		)
@@
 	(wire
 		(pts
-			(xy 158.75 60.96) (xy 158.75 64.77)
+			(xy 166.37 60.96) (xy 166.37 64.77)
 		)
 		(stroke
@@
 	(wire
 		(pts
-			(xy 237.49 104.775) (xy 227.33 104.775)
+			(xy 158.75 60.96) (xy 158.75 64.77)
 		)
 		(stroke
@@
 	(wire
 		(pts
-			(xy 259.715 66.675) (xy 257.81 66.675)
+			(xy 237.49 104.775) (xy 227.33 104.775)
 		)
 		(stroke
@@
 	(wire
 		(pts
+			(xy 166.37 64.77) (xy 158.75 64.77)
+		)
+		(stroke
+			(width 0)
+			(type default)
+		)
+	)
+	(wire
+		(pts
 			(xy 278.13 103.505) (xy 278.13 104.775)
 		)
@@
 	(wire
 		(pts
-			(xy 257.81 66.675) (xy 256.54 66.675)
-		)
-		(stroke
-			(width 0)
-			(type default)
-		)
-	)
-	(wire
-		(pts
 			(xy 179.07 137.795) (xy 180.34 137.795)
 		)
@@
 	(wire
 		(pts
+			(xy 166.37 52.07) (xy 158.75 52.07)
+		)
+		(stroke
+			(width 0)
+			(type default)
+		)
+	)
+	(wire
+		(pts
 			(xy 226.06 127.635) (xy 252.73 127.635)
 		)
@@
 	(wire
 		(pts
-			(xy 158.75 52.07) (xy 158.75 53.34)
+			(xy 166.37 52.07) (xy 166.37 53.34)
 		)
 		(stroke
@@
 	(wire
 		(pts
-			(xy 271.78 66.675) (xy 270.51 66.675)
-		)
-		(stroke
-			(width 0)
-			(type default)
-		)
-	)
-	(wire
-		(pts
 			(xy 191.77 158.75) (xy 190.5 158.75)
 		)
@@
 	(hierarchical_label "XTALOUT"
 		(shape output)
-		(at 256.54 66.675 180)
+		(at 271.78 66.675 0)
 		(effects
 			(font
@@
 				(thickness 0.254)
 			)
-			(justify right)
+			(justify left)
 		)
 	)
@@
 	(hierarchical_label "XTALIN"
 		(shape input)
-		(at 271.78 66.675 0)
+		(at 256.54 66.675 180)
 		(effects
 			(font
@@
 				(thickness 0.254)
 			)
-			(justify left)
+			(justify right)
 		)
 	)
@@
 	(symbol
 		(lib_id "SAMPI:ELECCAP")
-		(at 156.21 55.88 90)
+		(at 163.83 55.88 90)
 		(mirror x)
 		(unit 1)
@@
 		(dnp no)
 		(property "Reference" "C6"
-			(at 163.195 55.88 90)
+			(at 170.815 55.88 90)
 			(effects
 				(font
@@
 		)
 		(property "Value" "220uF"
-			(at 165.1 58.42 90)
+			(at 172.72 58.42 90)
 			(effects
 				(font
@@
 		)
 		(property "Footprint" "SAMPI:CAP1411"
-			(at 156.21 55.88 0)
+			(at 163.83 55.88 0)
 			(effects
 				(font
@@
 		)
 		(property "Datasheet" ""
-			(at 156.21 55.88 0)
+			(at 163.83 55.88 0)
 			(effects
 				(font
@@
 		)
 		(property "Description" "CAP TANT SMD 1411 220uF 6.3V 10% 1.2OHM WxLxH(2.8x3.5x2.3)"
-			(at 156.21 55.88 0)
+			(at 163.83 55.88 0)
 			(effects
 				(font
@@
 		)
 		(property "MNP" "F930J227KBA"
-			(at 156.21 55.88 0)
+			(at 163.83 55.88 0)
 			(effects
 				(font
@@
 		)
 		(property "MFT" "NCHC"
-			(at 156.21 55.88 0)
+			(at 163.83 55.88 0)
 			(effects
 				(font
@@
 					(unit 1)
 				)
+			)
+		)
+	)
+	(symbol
+		(lib_id "SAMPI:CERCAP")
+		(at 156.21 58.42 90)
+		(unit 1)
+		(exclude_from_sim no)
+		(in_bom yes)
+		(on_board yes)
+		(dnp no)
+		(property "Reference" "C2"
+			(at 160.655 56.515 90)
+			(effects
+				(font
+					(face "Consolas")
+					(size 1.27 1.27)
+					(bold yes)
+				)
+				(justify right)
+			)
+		)
+		(property "Value" "100nF"
+			(at 160.655 59.055 90)
+			(effects
+				(font
+					(face "Consolas")
+					(size 1.016 1.016)
+					(thickness 0.127)
+				)
+				(justify right)
+			)
+		)
+		(property "Footprint" "SAMPI:CAP0603"
+			(at 156.21 58.42 0)
+			(effects
+				(font
+					(face "Consolas")
+					(size 1.016 1.016)
+					(thickness 0.127)
+				)
+				(hide yes)
+			)
+		)
+		(property "Datasheet" ""
+			(at 156.21 58.42 0)
+			(effects
+				(font
+					(face "Consolas")
+					(size 1.016 1.016)
+					(thickness 0.127)
+				)
+				(hide yes)
+			)
+		)
+		(property "Description" "CAP CER SMD 0603 100nF 50V -20%/80% Y5V GENPURPOSE"
+			(at 156.21 58.42 0)
+			(effects
+				(font
+					(face "Consolas")
+					(size 1.016 1.016)
+					(thickness 0.127)
+				)
+				(hide yes)
+			)
+		)
+		(property "MNP" "CC0603ZRY5V9BB104"
+			(at 156.21 58.42 0)
+			(effects
+				(font
+					(face "Consolas")
+					(size 1.016 1.016)
+					(thickness 0.127)
+				)
+				(hide yes)
+			)
+		)
+		(property "MFT" "YAGE"
+			(at 156.21 58.42 0)
+			(effects
+				(font
+					(face "Consolas")
+					(size 1.016 1.016)
+					(thickness 0.127)
+				)
+				(hide yes)
+			)
+		)
+		(pin "2"
+		)
+		(pin "1"
+		)
+		(instances
+			(project "HW.ACIM-DBG"
+				(path "/20f80521-75f2-4ccc-bb34-c9566e70ef5c/34b63420-23a7-4d2d-affc-c07be2bf5f59"
+					(reference "C2")
+					(unit 1)
+				)

Commit message: Production HW.ACIM-DBG_V1.0 update BoM
Parts:
- C6: value 220uF -> 4.7uF; MFT NCHC -> Cal-Chip; MNP F930J227KBA -> GMC31X7R475K10NT
- R8: now not fitted; now left out of the parts list
Changed lines of the file:
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@@
 (kicad_sch
-	(version 20231120)
+	(version 20250114)
 	(generator "eeschema")
-	(generator_version "8.0")
+	(generator_version "9.0")
 	(paper "A4")
 	(title_block
@@
 			)
 		)
-		(property "Value" "220uF"
+		(property "Value" "4.7uF"
 			(at 172.72 58.42 90)
 			(effects
@@
 			)
 		)
-		(property "Description" "CAP TANT SMD 1411 220uF 6.3V 10% 1.2OHM WxLxH(2.8x3.5x2.3)"
+		(property "Description" "CAP CER 4.7UF 10V X7R 1206"
 			(at 163.83 55.88 0)
 			(effects
@@
 			)
 		)
-		(property "MNP" "F930J227KBA"
+		(property "MNP" "GMC31X7R475K10NT"
 			(at 163.83 55.88 0)
 			(effects
@@
 			)
 		)
-		(property "MFT" "NCHC"
+		(property "MFT" "Cal-Chip"
 			(at 163.83 55.88 0)
 			(effects
@@
 		(unit 1)
 		(exclude_from_sim no)
-		(in_bom yes)
+		(in_bom no)
 		(on_board yes)
-		(dnp no)
+		(dnp yes)
 		(property "Reference" "R8"
 			(at 213.36 156.21 0)
