File: V1/Design/HW.ACIM-DBG/VCP.kicad_sch (KiCad schematic)
At the start: 64 parts, among them U5 FT4232H, U6 SPI EEPROM, U7 SHIFT REG 8BIT, U8 12MHz

Commit message: V1 schematic update 1
Parts:
- removed C32, C33, C34, C38, C41, C44, C47: 22pF, SAMPI:CAP0603, symbol SAMPI:CERCAP
- removed C35, C37, C39, C42, C45, C48, C49, C50, C51, C52: 100nF, SAMPI:CAP0603, symbol SAMPI:CERCAP
- removed C36, C40, C43, C46: 10uF, SAMPI:CAP0603, symbol SAMPI:CERCAP
- removed D2: TR1, SAMPI:LED0606_4P, symbol SAMPI:RG_LED
- removed D3: TR2, SAMPI:LED0606_4P, symbol SAMPI:RG_LED
- removed D4: TR3, SAMPI:LED0606_4P, symbol SAMPI:RG_LED
- removed D5: TR4, SAMPI:LED0606_4P, symbol SAMPI:RG_LED
- removed D7: VCP, SAMPI:LED0603, symbol SAMPI:RLED
- removed FT10, FT7, FT8, FT9: 120R@100MHz, SAMPI:FT0603, symbol SAMPI:FerriteBead
- removed FT6: 2x 120R@100MHz, SAMPI:IND1210_4P, symbol SAMPI:IND1210_4P
- removed R21, R22, R23, R24, R25, R26, R27, R28: 0R, SAMPI:RES0603, symbol SAMPI:RES
- removed R29: 12K/1%, SAMPI:RES0603, symbol SAMPI:RES
- removed R3, R35, R36, R37, R38, R39, R40, R41, R42: 1.1K, SAMPI:RES0603, symbol SAMPI:RES
- removed R30, R31, R32, R33, R34: 10K, SAMPI:RES0603, symbol SAMPI:RES
- removed U5: FT4232H, SAMPI:VQFN-56_FTDI, symbol SAMPI:FT4232H
- removed U6: SPI EEPROM, SAMPI:SOT-23-6_MCHP, symbol SAMPI:93LC56
- removed U7: SHIFT REG 8BIT, SAMPI:TSSOP16-SOT403-1, symbol SAMPI:74HC595
- removed U8: 12MHz, SAMPI:CDFN2520-ABM10, symbol SAMPI:XTAL-4P
- added BT1: MODE, Liem:SW_SMD2_6.0x3.5, symbol SAMPI:BT3
- added C19, C20, C21, C24, C25: 100nF, Liem:CAP0402, symbol SAMPI:CERCAP
- added C22, C23: 10uF, Liem:CAP0603, symbol SAMPI:CERCAP
- added D2: DV PORT, Liem:LED0603, symbol Liem:RLED
- added D3: DBG PORT, Liem:LED0603, symbol Liem:RLED
- added D4: PIC, Liem:LED0603, symbol Liem:RLED
- added D5: ARM, Liem:LED0603, symbol Liem:RLED
- added J4: VCP ICSP, symbol SAMPI:SIL06
- added Q1: 60V/265mA, SAMPI:SOT23, symbol SAMPI:FET_N-CH
- added R11: 10K, Liem:RES0402, symbol SAMPI:RES
- added R12, R13, R14: 1K, Liem:RES0402, symbol SAMPI:RES
- added RL1: RELAY2-NL, SAMPI:EA2-5NU, symbol SAMPI:RELAY2-NL
- added U4: MCU, Liem:UQFN28-4x4-EP, symbol TUANLIB:PIC32MM0256GPM028-I_M6
- added U5: I2C EEPROM, symbol SAMPI:24AAxx_SOT23-5
- R15: value 1.1K -> 1K; footprint SAMPI:RES0603 -> Liem:RES0402; Checked OK -> (none); MFT YAGEO -> Rohm Semiconductor; MNP AC0603FR-071K1L -> MCR01MZPJ102; Unit Price 0.021 -> (none); now fitted; now in the parts list
- R16: value 100K -> 1K; footprint SAMPI:RES0603 -> Liem:RES0402; Checked OK -> (none); MFT YAGEO -> Rohm Semiconductor; MNP RC0603FR-07100KL -> MCR01MZPJ102; Unit Price 0.019 -> (none)
- R17: value 0R -> 1K; footprint SAMPI:RES0603 -> Liem:RES0402; Checked OK -> (none); MFT YAGEO -> Rohm Semiconductor; MNP RC0603JR-070RL -> MCR01MZPJ102; Unit Price 0.015 -> (none)
- R18: value 0R -> 47K; footprint SAMPI:RES0603 -> Liem:RES0402; Checked OK -> (none); MFT YAGEO -> Rohm Semiconductor; MNP RC0603JR-070RL -> MCR01MZPJ473; Unit Price 0.015 -> (none)
- R19, R20: value 0R -> 5.1K, 1%; footprint SAMPI:RES0603 -> Liem:RES0402; Checked OK -> (none); MNP RC0603JR-070RL -> RC0402FR-075K1L; Unit Price 0.015 -> (none)
Connections:
- net RXD1 is gone; now on an unnamed net: R18.2
- net RXD2 is gone; now on net +3V3: R20.2
- net TXD2 is gone; now on net +3V3: R19.2
- net +3V3: now also C19.2, C20.2, C22.2, C25.2, J4.2, R11.2, U4.10 (VDD), U4.20 (VUSB3V3), U4.25 (AVDD/VDD), U5.4 (VCC); no longer R15.1
- net GND: now also R18.1, BT1.2, C19.1, C20.1, C21.1, C22.1, C23.1, C24.1, C25.1, D2.K, D3.K, D4.K, D5.K, J4.3, Q1.2 (S), U4.24 (AVSS/VSS), U4.29 (EP), U4.5 (VSS), U5.2 (VSS), U5.5 (WP); no longer R16.2
- net at R15.2: now also RL1.2 (NC1)
- net at R17.1: now also Q1.1 (G)
- net SCL: now reaches R19.1
- net SCL: now also U4.14 (TCK/RP13/SCL1/U1CTS/SCK1/OCM1A/RB8), U5.1 (SCL)
- net SDA: now reaches R20.1
- net SDA: now also U4.15 (TMS/REFCLKI/RP14/SDA1/T1CK/T1G/T2CK/T2G/U1RTS/U1BCLK/SDO1/OCM1B/INT2/RB9), U5.3 (SDA)
- net TXD1 renamed MODE_SEL
- net VCP_VBUS: no longer names the net of R16.1
- net VCP_VBUS: now also D5.A
- new net: BT1.1, C24.2, R12.1
- new net: R16.2, RL1.4 (NO1)
- new net: C23.2, U4.17 (VCAP)
- new net: Q1.3 (D), RL1.10 (COIL-)
- new net: D4.A, R15.1
- new net: D3.A, R14.1
- new net: D2.A, R13.1
- new net +5V: RL1.1 (COIL+)
- new net DBG_RXD: U4.3 (AN4/C1INB/RP8/SDA2/OCM2E/RB2)
- new net DBG_SLED: R14.2
- new net DBG_TXD: U4.4 (TDI/AN11/C1INA/RP9/SCL2/OCM2F/RB3)
- new net DV_SLED: R13.2
- new net MODE_SLED: RL1.3 (COM1)
- new net VCP_PGC: J4.5, U4.2 (PGEC1/AN3/C1INC/C2INA/RP7/OCM2D/RB1)
- new net VCP_PGD: J4.4, U4.1 (PGED1/AN2/C1IND/C2INB/C3INC/RP6/OCM2C/RB0)
- new net VCP_USB_N: U4.18 (D-/RB10)
- new net VCP_USB_P: U4.19 (D+/RB11)
- new net VCP_USB_VBUS: U4.12 (VBUS/RB6)
- new net ~{BT_MODE}: R12.2, U4.7 (OSC2/CLKO/AN6/C3IND/RP4/OCM1D/RA3)
- new net ~{VCP_MCLR}: C21.2, J4.1, R11.1, U4.26 (MCLR)
- no-connect marks 21 -> 2

Commit message: V1 schematic update 2
Parts:
- removed C25: 100nF, Liem:CAP0402, symbol SAMPI:CERCAP
- removed D4: PIC, Liem:LED0603, symbol Liem:RLED
- removed D5: ARM, Liem:LED0603, symbol Liem:RLED
- removed Q1: 60V/265mA, SAMPI:SOT23, symbol SAMPI:FET_N-CH
- removed R15, R16, R17: 1K, Liem:RES0402, symbol SAMPI:RES
- removed R18: 47K, Liem:RES0402, symbol SAMPI:RES
- removed R19, R20: 5.1K, 1%, Liem:RES0402, symbol SAMPI:RES
- removed RL1: RELAY2-NL, SAMPI:EA2-5NU, symbol SAMPI:RELAY2-NL
- removed U5: I2C EEPROM, symbol SAMPI:24AAxx_SOT23-5
- D2: value DV PORT -> HS PORT; symbol Liem:RLED -> SAMPI:BLED
- D3: value DBG PORT -> LS PORT; symbol Liem:RLED -> SAMPI:GLED
- J4: MFT (none) -> <NULL>; MNP (none) -> <NULL>
- U4: value MCU -> PIC32MM0064GPM028
Connections:
- net DBG_RXD renamed LS_RXD
- net DBG_SLED renamed LS_SLED
- net DBG_TXD renamed LS_TXD
- net DV_SLED renamed HS_SLED
- net SCL: no longer names the net of U4.14 (TCK/RP13/SCL1/U1CTS/SCK1/OCM1A/RB8)
- net SDA: no longer names the net of U4.15 (TMS/REFCLKI/RP14/SDA1/T1CK/T1G/T2CK/T2G/U1RTS/U1BCLK/SDO1/OCM1B/INT2/RB9)
- no-connect marks 2 -> 1

Commit message: V1 schematic update 3
Parts:
- removed BT1: MODE, Liem:SW_SMD2_6.0x3.5, symbol SAMPI:BT3
- added BT1: RESET, SAMPI:BUTTON_4P_6x6, symbol SAMPI:BT
- C19, C20, C21, C24: footprint Liem:CAP0402 -> SAMPI:CAP0603; MFT Walsin Technology Corporation -> Samsung; MNP 0402B104K160CT -> CL10B104KB8NNNC
- C22, C23: footprint Liem:CAP0603 -> SAMPI:CAP0603; MFT KEMET -> Samsung; MNP C0603C106M8PACTU -> CL10A106MQ8NNNC
- D2: footprint Liem:LED0603 -> SAMPI:LED0603; MFT Rohm Semiconductor -> Harvatek; MNP SML-D12V8WT86P -> B1931NB--20C007614U1930
- D3: footprint Liem:LED0603 -> SAMPI:LED0603; MFT Rohm Semiconductor -> Harvatek; MNP SML-D12V8WT86P -> B1911NG--20D000214U1930
- J4: footprint (none) -> SAMPI:HD-1x6x1.27MM-TH; MFT <NULL> -> Harwin; MNP <NULL> -> M50-3530642
- R11: footprint Liem:RES0402 -> SAMPI:RES0603; MNP RC0402FR-0710KL -> RC0603FR-0710KL
- R12, R13, R14: footprint Liem:RES0402 -> SAMPI:RES0603; MFT Rohm Semiconductor -> YAGEO; MNP MCR01MZPJ102 -> RC0603FR-071KL
- U4: footprint Liem:UQFN28-4x4-EP -> SAMPI:UQFN28-4x4-EP
Connections:
- net GND: now also BT1.3, BT1.4
- net at C24.2, R12.1: now also BT1.1, BT1.2
Other:
- moved on the sheet: C24, R12

Commit message: V1 layout
Parts:
- added D3: MODE, SAMPI:LED3MM, symbol SAMPI:RLED
- added R15: 1K, SAMPI:RES0603, symbol SAMPI:RES
- added R16: 10K, SAMPI:RES0603, symbol SAMPI:RES
- D2: renamed from D3; footprint SAMPI:LED0603 -> SAMPI:LED3MM; MFT Harvatek -> Würth Elektronik; MNP B1911NG--20D000214U1930 -> 151031VS06000
- D4: renamed from D2; footprint SAMPI:LED0603 -> SAMPI:LED3MM; symbol SAMPI:BLED -> SAMPI:YLED; MFT Harvatek -> Würth Elektronik; MNP B1931NB--20C007614U1930 -> 151031YS06000
- renumbered C19 to C17, C21 to C18, C20 to C19, C22 to C20, C23 to C21, C24 to C22, J4 to J2, U4 to U3
Connections:
- net +3V3: now also R16.2
- net GND: now also D3.K
- net MODE_SLED: now also R15.2
- net ~{BT_MODE}: no longer U3.7 (OSC2/CLKO/AN6/C3IND/RP4/OCM1D/RA3)
- net at BT1.1, BT1.2, C22.2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: now also R16.1
- new net: D3.A, R15.1
Other:
- moved on the sheet: BT1, C18, R11

Commit message: V1 layout update 2
Parts:
- removed BT1: RESET, SAMPI:BUTTON_4P_6x6, symbol SAMPI:BT
- removed C17, C18: 100nF, SAMPI:CAP0603, symbol SAMPI:CERCAP
- removed D3: MODE, SAMPI:LED3MM, symbol SAMPI:RLED
- removed D4: HS PORT, SAMPI:LED3MM, symbol SAMPI:YLED
- removed J2: VCP ICSP, SAMPI:HD-1x6x1.27MM-TH, symbol SAMPI:SIL06
- removed R11, R16: 10K, SAMPI:RES0603, symbol SAMPI:RES
- removed R12, R13, R14: 1K, SAMPI:RES0603, symbol SAMPI:RES
- removed U3: PIC32MM0064GPM028, SAMPI:UQFN28-4x4-EP, symbol TUANLIB:PIC32MM0256GPM028-I_M6
- added C40, C41, C42, C43, C44, C48, C49, C50, C52, C53: 100nF, SAMPI:CAP0603, symbol SAMPI:CERCAP
- added C45, C46, C47, C54: 10uF, SAMPI:CAP0603, symbol SAMPI:CERCAP
- added C51, C55, C56: 22pF, SAMPI:CAP0603, symbol SAMPI:CERCAP
- added D10: TR1, SAMPI:LED0606_4P, symbol SAMPI:RG_LED
- added D7: TR4, SAMPI:LED0606_4P, symbol SAMPI:RG_LED
- added D8: TR3, SAMPI:LED0606_4P, symbol SAMPI:RG_LED
- added D9: TR2, SAMPI:LED0606_4P, symbol SAMPI:RG_LED
- added FT3, FT4, FT5, FT6: 120R@100MHz, SAMPI:FT0603, symbol SAMPI:FerriteBead
- added R27, R49, R50, R51, R52, R53, R54, R55, R56: 1.1K, SAMPI:RES0603, symbol SAMPI:RES
- added R28, R38, R39, R47: 10K, SAMPI:RES0603, symbol SAMPI:RES
- added R29: 2.2K, SAMPI:RES0603, symbol SAMPI:RES
- added R46: 12K/1%, SAMPI:RES0603, symbol SAMPI:RES
- added R48: 100K, SAMPI:RES0603, symbol SAMPI:RES
- added U10: 12MHz, SAMPI:CDFN2520-ABM10, symbol SAMPI:XTAL-4P
- added U3: SPI EEPROM, SAMPI:SOT-23-6_MCHP, symbol SAMPI:93LC56
- added U8: FT4232H, SAMPI:VQFN-56_FTDI, symbol SAMPI:FT4232H
- added U9: SHIFT REG 8BIT, SAMPI:TSSOP16-SOT403-1, symbol SAMPI:74HC595
- C19, C22: value 100nF -> 22pF; MFT Samsung -> Walsin; MNP CL10B104KB8NNNC -> 0603N220J500CT
- C20, C21: value 10uF -> 22pF; MFT Samsung -> Walsin; MNP CL10A106MQ8NNNC -> 0603N220J500CT
- D2: value LS PORT -> VCP
- R15: value 1K -> 1.1K; MNP RC0603FR-071KL -> AC0603FR-071K1L; now not fitted; now left out of the parts list
Connections:
- net +3V3: now also C21.2, C22.2, R15.1, C49.2, C50.2, FT3.1, FT4.1, FT5.1, FT6.1, R28.2, R38.2, R39.2, R47.2, U3.6 (VCC), U9.10 (~{MR}), U9.16 (VCC)
- net GND: now also C40.1, C41.1, C42.1, C43.1, C44.1, C45.1, C46.1, C47.1, C48.1, C49.1, C50.1, C51.1, C52.1, C53.1, C54.1, C55.1, C56.1, D10.1 (GK), D10.4 (RK), D7.1 (GK), D7.4 (RK), D8.1 (GK), D8.4 (RK), D9.1 (GK), D9.4 (RK), R27.2, R46.2, R48.2, U10.2 (GND1), U10.4 (X2), U3.2 (VSS), U8.10 (TEST), U8.21 (GND), U8.41 (GND), U8.45 (GND), U8.57 (TP), U9.8 (GND); no longer D2.K
- net at D2.A: now also U8.30 (~{SUSPEND})
- net MODE_SLED: no longer names the net of R15.2
- net MODE_SLED: now also D2.K, R27.1
- new net: R49.1, U9.6 (Q6)
- new net: D7.3 (RA), R49.2
- new net: D10.2 (GA), R56.2
- new net: D10.3 (RA), R55.2
- new net: R53.1, U9.2 (Q2)
- new net: D9.3 (RA), R53.2
- new net: D7.2 (GA), R50.2
- new net: C52.2, C53.2, C54.2, U8.2 (VCORE), U8.31 (VCORE), U8.43 (VREGOUT)
- new net: C40.2, C44.2, C48.2, FT3.2, U8.16 (VCCIO), U8.36 (VCCIO), U8.50 (VCCIO)
- new net: C41.2, C45.2, FT4.2, U8.44 (VREGIN)
- new net: C43.2, C47.2, FT6.2, U8.5 (VPHY)
- new net: R46.1, U8.6 (REF)
- new net: C42.2, C46.2, FT5.2, U8.9 (VPLL)
- new net: R29.2, R38.1, U3.1 (DO)
- new net: D9.2 (GA), R54.2
- new net: R55.1, U9.15 (Q0)
- new net: R54.1, U9.3 (Q3)
- new net: R51.1, U9.4 (Q4)
- new net: D8.3 (RA), R51.2
- new net: R56.1, U9.1 (Q1)
- new net: R52.1, U9.5 (Q5)
- new net: R50.1, U9.7 (Q7)
- new net: D8.2 (GA), R52.2
- new net CTS2: U8.25 (BDBUS3/~{CTS})
- new net EECLK: R28.1, U3.4 (CLK), U8.56 (EECLK), U9.11 (SHCP)
- new net EECS: R39.1, U3.5 (CS), U8.1 (EECS), U9.12 (STCP)
- new net EEDATA: R29.1, U3.3 (DI), U8.55 (EEDATA), U9.14 (DS)
- new net OSCI: C55.2, U10.1 (X1), U8.3 (OSCI)
- new net OSCO: C56.2, U10.3 (GND2), U8.4 (OSCO)
- new net RTS2: U8.24 (BDBUS2/~{RTS})
- new net RXD1: U8.13 (ADBUS1/RXD)
- new net RXD2: U8.23 (BDBUS1/RXD)
- new net RXD3: U8.33 (CDBUS1/RXD)
- new net RXD4: U8.46 (DDBUS1/RXD)
- new net TXD1: U8.12 (ADBUS0/TXD)
- new net TXD2: U8.22 (BDBUS0/TXD)
- new net TXD3: U8.32 (CDBUS0/TXD)
- new net TXD4: U8.42 (DDBUS0/TXD)
- new net VCP_DM: U8.7 (DM)
- new net VCP_DP: U8.8 (DP)
- new net VCP_VBUS: C51.2, R48.1, U8.11 (~{RESET})
- new net ~{PWREN}: R47.1, U8.54 (~{PWREN}), U9.13 (~{OE})
- no-connect marks 1 -> 23
Other:
- moved on the sheet: D2

Commit message: V1 layout update 3
Other:
- company: TON DUC THANG UNIVERSITY -> KiCad EDA
- moved on the sheet: C51, R48
Changed lines of the file:
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@@
 		(date "2024-12-04")
 		(rev "0.1")
-		(company "TON DUC THANG UNIVERSITY")
+		(company "KiCad EDA")
 		(comment 1 "Schematic Designed by ...")
 		(comment 2 "PCB Designed by ...")
@@
 	)
 	(junction
-		(at 153.035 72.39)
-		(diameter 0)
-		(color 0 0 0 0)
-	)
-	(junction
 		(at 186.69 104.14)
 		(diameter 0)
@@
 	)
 	(junction
+		(at 142.875 72.39)
+		(diameter 0)
+		(color 0 0 0 0)
+	)
+	(junction
 		(at 161.29 35.56)
 		(diameter 0)
@@
 	)
 	(junction
-		(at 161.925 72.39)
+		(at 151.765 72.39)
 		(diameter 0)
 		(color 0 0 0 0)
@@
 	(wire
 		(pts
-			(xy 161.925 72.39) (xy 163.195 72.39)
+			(xy 151.765 72.39) (xy 153.035 72.39)
 		)
 		(stroke
@@
 	(wire
 		(pts
-			(xy 94.615 77.47) (xy 95.885 77.47)
-		)
-		(stroke
-			(width 0)
-			(type default)
-		)
-	)
-	(wire
-		(pts
 			(xy 27.305 128.27) (xy 27.305 129.54)
 		)
@@
 	(wire
 		(pts
-			(xy 161.925 72.39) (xy 161.925 73.66)
+			(xy 151.765 72.39) (xy 151.765 73.66)
 		)
 		(stroke
@@
 	(wire
 		(pts
-			(xy 94.615 72.39) (xy 95.885 72.39)
-		)
-		(stroke
-			(width 0)
-			(type default)
-		)
-	)
-	(wire
-		(pts
 			(xy 90.805 43.18) (xy 92.075 43.18)
 		)
@@
 	(wire
 		(pts
-			(xy 153.035 72.39) (xy 153.035 73.66)
+			(xy 142.875 72.39) (xy 142.875 73.66)
 		)
 		(stroke
@@
 	(wire
 		(pts
-			(xy 94.615 82.55) (xy 95.885 82.55)
+			(xy 163.83 138.43) (xy 163.83 148.59)
 		)
 		(stroke
-			(width 0)
+			(width 0.254)
 			(type default)
 		)
@@
 	(wire
 		(pts
-			(xy 163.83 138.43) (xy 163.83 148.59)
+			(xy 133.985 156.21) (xy 133.985 157.48)
 		)
 		(stroke
-			(width 0.254)
+			(width 0.381)
 			(type default)
 		)
@@
 	(wire
 		(pts
-			(xy 133.985 156.21) (xy 133.985 157.48)
+			(xy 47.625 148.59) (xy 95.885 148.59)
 		)
 		(stroke
@@
 	(wire
 		(pts
-			(xy 47.625 148.59) (xy 95.885 148.59)
+			(xy 132.715 72.39) (xy 142.875 72.39)
 		)
 		(stroke
-			(width 0.381)
+			(width 0)
 			(type default)
 		)
@@
 	(wire
 		(pts
-			(xy 132.715 72.39) (xy 153.035 72.39)
-		)
-		(stroke
-			(width 0)
-			(type default)
-		)
-	)
-	(wire
-		(pts
-			(xy 153.035 72.39) (xy 161.925 72.39)
+			(xy 142.875 72.39) (xy 151.765 72.39)
 		)
 		(stroke
@@
 	(wire
 		(pts
-			(xy 94.615 74.93) (xy 95.885 74.93)
-		)
-		(stroke
-			(width 0)
-			(type default)
-		)
-	)
-	(wire
-		(pts
 			(xy 232.41 78.74) (xy 232.41 80.01)
 		)
@@
 	(hierarchical_label "~{PWREN}"
 		(shape output)
-		(at 94.615 82.55 180)
+		(at 95.885 82.55 180)
 		(fields_autoplaced yes)
 		(effects
@@
 	(hierarchical_label "EECS"
 		(shape output)
-		(at 94.615 72.39 180)
+		(at 95.885 72.39 180)
 		(fields_autoplaced yes)
 		(effects
@@
 	(hierarchical_label "EEDATA"
 		(shape bidirectional)
-		(at 94.615 77.47 180)
+		(at 95.885 77.47 180)
 		(fields_autoplaced yes)
 		(effects
@@
 	(hierarchical_label "EECLK"
 		(shape output)
-		(at 94.615 74.93 180)
+		(at 95.885 74.93 180)
 		(fields_autoplaced yes)
 		(effects
@@
 	(hierarchical_label "VCP_VBUS"
 		(shape input)
-		(at 163.195 72.39 0)
+		(at 153.035 72.39 0)
 		(fields_autoplaced yes)
 		(effects
@@
 	(symbol
 		(lib_id "power:GND")
-		(at 161.925 81.28 0)
+		(at 151.765 81.28 0)
 		(unit 1)
 		(exclude_from_sim no)
@@
 		(dnp no)
 		(property "Reference" "#PWR0128"
-			(at 161.925 87.63 0)
+			(at 151.765 87.63 0)
 			(effects
 				(font
@@
 		)
 		(property "Value" "GND"
-			(at 161.925 85.09 0)
+			(at 151.765 85.09 0)
 			(effects
 				(font
@@
 		)
 		(property "Footprint" ""
-			(at 161.925 81.28 0)
+			(at 151.765 81.28 0)
 			(effects
 				(font
@@
 		)
 		(property "Datasheet" ""
-			(at 161.925 81.28 0)
+			(at 151.765 81.28 0)
 			(effects
 				(font
@@
 		)
 		(property "Description" ""
-			(at 161.925 81.28 0)
+			(at 151.765 81.28 0)
 			(effects
 				(font
@@
 	(symbol
 		(lib_id "SAMPI:CERCAP")
-		(at 150.495 78.74 90)
+		(at 140.335 78.74 90)
 		(unit 1)
 		(exclude_from_sim no)
@@
 		(fields_autoplaced yes)
 		(property "Reference" "C51"
-			(at 155.575 76.1999 90)
+			(at 145.415 76.1999 90)
 			(effects
 				(font
@@
 		)
 		(property "Value" "22pF"
-			(at 155.575 78.7399 90)
+			(at 145.415 78.7399 90)
 			(effects
 				(font
@@
 		)
 		(property "Footprint" "SAMPI:CAP0603"
-			(at 150.495 78.74 0)
+			(at 140.335 78.74 0)
 			(effects
 				(font
@@
 		)
 		(property "Datasheet" ""
-			(at 150.495 78.74 0)
+			(at 140.335 78.74 0)
 			(effects
 				(font
@@
 		)
 		(property "Description" "CAP CER 22PF 50V C0G/NP0 0603"
-			(at 150.495 78.74 0)
+			(at 140.335 78.74 0)
 			(effects
 				(font
@@
 		)
 		(property "MNP" "0603N220J500CT"
-			(at 150.495 78.74 0)
+			(at 140.335 78.74 0)
 			(effects
 				(font
@@
 		)
 		(property "MFT" "Walsin"
-			(at 150.495 78.74 0)
+			(at 140.335 78.74 0)
 			(effects
 				(font
@@
 	(symbol
 		(lib_id "power:GND")
-		(at 153.035 81.28 0)
+		(at 142.875 81.28 0)
 		(unit 1)
 		(exclude_from_sim no)
@@
 		(dnp no)
 		(property "Reference" "#PWR0124"
-			(at 153.035 87.63 0)
+			(at 142.875 87.63 0)
 			(effects
 				(font
@@
 		)
 		(property "Value" "GND"
-			(at 153.035 85.09 0)
+			(at 142.875 85.09 0)
 			(effects
 				(font
@@
 		)
 		(property "Footprint" ""
-			(at 153.035 81.28 0)
+			(at 142.875 81.28 0)
 			(effects
 				(font
@@
 		)
 		(property "Datasheet" ""
-			(at 153.035 81.28 0)
+			(at 142.875 81.28 0)
 			(effects
 				(font
@@
 		)
 		(property "Description" ""
-			(at 153.035 81.28 0)
+			(at 142.875 81.28 0)
 			(effects
 				(font
@@
 	(symbol
 		(lib_id "SAMPI:RES")
-		(at 159.385 76.2 90)
+		(at 149.225 76.2 90)
 		(mirror x)
 		(unit 1)
@@
 		(dnp no)
 		(property "Reference" "R48"
-			(at 165.735 76.2 90)
+			(at 155.575 76.2 90)
 			(effects
 				(font
@@
 		)
 		(property "Value" "100K"
-			(at 165.735 78.74 90)
+			(at 155.575 78.74 90)
 			(effects
 				(font
@@
 		)
 		(property "Footprint" "SAMPI:RES0603"
-			(at 159.385 76.2 0)
+			(at 149.225 76.2 0)
 			(effects
 				(font
@@
 		)
 		(property "Datasheet" ""
-			(at 159.385 76.2 0)
+			(at 149.225 76.2 0)
 			(effects
 				(font
@@
 		)
 		(property "Description" "RES 100K OHM 1% 1/10W 0603"
-			(at 159.385 76.2 0)
+			(at 149.225 76.2 0)
 			(effects
 				(font
@@
 		)
 		(property "MNP" "RC0603FR-07100KL"
-			(at 159.385 76.2 0)
+			(at 149.225 76.2 0)
 			(effects
 				(font
@@
 		)
 		(property "MFT" "YAGEO"
-			(at 159.385 76.2 0)
+			(at 149.225 76.2 0)
 			(effects
 				(font

Commit message: V1 layout update 5
Parts:
- removed R15: 1.1K, SAMPI:RES0603, symbol SAMPI:RES
- added Q1: MFET N, symbol SAMPI:FET_N-CH
Connections:
- net +3V3: now also R27.1
- net GND: now also Q1.2 (S); no longer R27.2
- net at D2.K: now also Q1.3 (D); no longer R27.1
- net at D2.A: now also R27.2; no longer U8.30 (~{SUSPEND})
- net CTS2: no longer names the net of U8.25 (BDBUS3/~{CTS})
- net RTS2: no longer names the net of U8.24 (BDBUS2/~{RTS})
- new net: Q1.1 (G), U8.30 (~{SUSPEND})
- no-connect marks 23 -> 25
Other:
- moved on the sheet: C55, C56, D2, R27, U10

Commit message: V1 layout update 6
Parts:
- D2: footprint SAMPI:LED3MM -> SAMPI:LED0603
- Q1: footprint (none) -> SAMPI:SOT23; MFT (none) -> VISHAY; MNP (none) -> SI2318CDS-T1-GE3
