File: V1/Design/HW.ACIM-DBG/HW.ACIM-DBG.kicad_sch (KiCad schematic)
At the start: 5 parts

Commit message: V1 schematic update 1
Other:
- removed sheet AC-DC ADAPTOR
- removed sheet SIGNAL ANALYZER
- sheet USB HUB ports: added none; removed INV_CTS2, INV_RTS2, INV_RXD1, INV_RXD2, INV_TXD1, INV_TXD2, PSU_CTS2, PSU_RTS2, PSU_RXD1, PSU_RXD2, PSU_TXD1, PSU_TXD2, VCP_DM, VCP_DP, VCP_VBUS
- sheet VCP ports: added none; removed CTS2, CTS4, RTS2, RTS4, RXD1, RXD2, RXD3, RXD4, TXD1, TXD2, TXD3, TXD4, VCP_DM, VCP_DP, VCP_VBUS
- note removed: "ICSP"
- note removed: "USB"
- note removed: "USB, UART"
- note removed: "USB, UART, ICSP"
- moved on the sheet: SH1, SH2, SH3, SH4, SH5

Commit message: V1 schematic update 2
Parts:
- removed SH5: SCREW HOLDER, SAMPI:SCREWHOLE-2.5M, symbol SAMPI:SCREWHOLDER
Connections:
- no-connect marks 0 -> 26
Other:
- sheet ISOLATOR ports: added DB_TXD, DV_CTS, DV_RTS, DV_RXD, DV_TXD, ISO_DB_TXD, ISO_HS_CTS, ISO_HS_RTS, ISO_HS_RXD, ISO_HS_TXD, ISO_PGC, ISO_PGD, PGC, PGD, PRG_USB_N, PRG_USB_P, PRG_VBUS, VDD_SEN, ~{ISO_MCLR}, ~{MCLR}; removed none
- sheet USB HUB ports: added HUB_USB_VBUS, USB1_N, USB1_P, USB1_PWR_EN, USB2_N, USB2_P, USB2_PWR_EN, USB_N, USB_P; removed none
- sheet VCP ports: added HS_CTS, HS_RTS, HS_RXD, HS_SLED, HS_TXD, LS_RXD, LS_SLED, LS_TXD, MODE_SEL, MODE_SLED, SCL, SDA, VCP_PGC, VCP_PGD, VCP_USB_N, VCP_USB_P, VCP_USB_VBUS, ~{BT_MODE}, ~{VCP_MCLR}; removed none
- note added: "ICSP DV UART (3MBIT) DBG UART (115.2KBIT)"
- note added: "INTERCONNECTION"
- moved on the sheet: SH1, SH2, SH3, SH4

Commit message: V1 schematic update 3
Parts:
- SH1, SH2, SH3, SH4: MFT (none) -> Essentra Components; MNP (none) -> 50M020040G005
Changed lines of the file:
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@@
 			)
 		)
-		(property "Description" ""
+		(property "Description" "FILLISTER PHILLIPS SCREW, M2 X ."
 			(at 98.425 111.76 0)
 			(effects
@@
 					(size 1.016 1.016)
 					(thickness 0.1588)
+				)
+				(hide yes)
+			)
+		)
+		(property "MFT" "Essentra Components"
+			(at 98.425 111.76 0)
+			(effects
+				(font
+					(size 1.27 1.27)
+				)
+				(hide yes)
+			)
+		)
+		(property "MNP" "50M020040G005"
+			(at 98.425 111.76 0)
+			(effects
+				(font
+					(size 1.27 1.27)
 				)
 				(hide yes)
@@
 			)
 		)
-		(property "Description" ""
-			(at 79.375 111.76 0)
-			(effects
-				(font
-					(face "Consolas")
-					(size 1.016 1.016)
-					(thickness 0.1588)
+		(property "Description" "FILLISTER PHILLIPS SCREW, M2 X ."
+			(at 79.375 111.76 0)
+			(effects
+				(font
+					(face "Consolas")
+					(size 1.016 1.016)
+					(thickness 0.1588)
+				)
+				(hide yes)
+			)
+		)
+		(property "MFT" "Essentra Components"
+			(at 79.375 111.76 0)
+			(effects
+				(font
+					(size 1.27 1.27)
+				)
+				(hide yes)
+			)
+		)
+		(property "MNP" "50M020040G005"
+			(at 79.375 111.76 0)
+			(effects
+				(font
+					(size 1.27 1.27)
 				)
 				(hide yes)
@@
 			)
 		)
-		(property "Description" ""
-			(at 85.725 111.76 0)
-			(effects
-				(font
-					(face "Consolas")
-					(size 1.016 1.016)
-					(thickness 0.1588)
+		(property "Description" "FILLISTER PHILLIPS SCREW, M2 X ."
+			(at 85.725 111.76 0)
+			(effects
+				(font
+					(face "Consolas")
+					(size 1.016 1.016)
+					(thickness 0.1588)
+				)
+				(hide yes)
+			)
+		)
+		(property "MFT" "Essentra Components"
+			(at 85.725 111.76 0)
+			(effects
+				(font
+					(size 1.27 1.27)
+				)
+				(hide yes)
+			)
+		)
+		(property "MNP" "50M020040G005"
+			(at 85.725 111.76 0)
+			(effects
+				(font
+					(size 1.27 1.27)
 				)
 				(hide yes)
@@
 			)
 		)
-		(property "Description" ""
-			(at 92.075 111.76 0)
-			(effects
-				(font
-					(face "Consolas")
-					(size 1.016 1.016)
-					(thickness 0.1588)
-				)
-				(hide yes)
+		(property "Description" "FILLISTER PHILLIPS SCREW, M2 X ."
+			(at 92.075 111.76 0)
+			(effects
+				(font
+					(face "Consolas")
+					(size 1.016 1.016)
+					(thickness 0.1588)
+				)
+				(hide yes)
+			)
+		)
+		(property "MFT" "Essentra Components"
+			(at 92.075 111.76 0)
+			(effects
+				(font
+					(size 1.27 1.27)
+				)
+				(hide yes)
+			)
+		)
+		(property "MNP" "50M020040G005"
+			(at 92.075 111.76 0)
+			(effects
+				(font
+					(size 1.27 1.27)
+				)
+				(hide yes)

Commit message: V1 layout
Parts:
- added SH5, SH6, SH7, SH8, SH9: SCREW HOLDER, SAMPI:SCREWHOLE-2.5M, symbol SAMPI:SCREWHOLDER
- added TP1: 3V3 ISO, SAMPI:TP1MM, symbol SAMPI:TESTPOINT
- added TP2: GND ISO, SAMPI:TP1MM, symbol SAMPI:TESTPOINT
- added TP3: 5V, SAMPI:TP1MM, symbol SAMPI:TESTPOINT
- added TP4: VTG(5V), SAMPI:TP1MM, symbol SAMPI:TESTPOINT
- added TP5: 3V3, SAMPI:TP1MM, symbol SAMPI:TESTPOINT
- added TP6: GND, SAMPI:TP1MM, symbol SAMPI:TESTPOINT
Connections:
- new net +3V3: TP5.1
- new net +3V3_ISO: TP1.1
- new net +5V: TP3.1
- new net GND: TP6.1
- new net GND_ISO: TP2.1
- new net VTG: TP4.1
- no-connect marks 26 -> 25
Other:
- sheet ISOLATOR ports: added DB_RXD, ISO_DB_RXD, ISO_DV_CTS, ISO_DV_RTS, ISO_DV_RXD, ISO_DV_TXD, TG_RST; removed ISO_HS_CTS, ISO_HS_RTS, ISO_HS_RXD, ISO_HS_TXD
- sheet VCP ports: added TG_RST; removed MODE_SEL

Commit message: V1 layout update 2
Other:
- sheet ISOLATOR renamed TERMINALS
- sheet TERMINALS: file ISOLATOR.kicad_sch -> TERMINALS.kicad_sch
- moved on the sheet: TP1, TP2, TP3, TP4, TP5, TP6

Commit message: V1 layout update 3
Other:
- company: TON DUC THANG UNIVERSITY -> KiCad EDA
Changed lines of the file:
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@@
 		(date "2024-12-04")
 		(rev "0.1")
-		(company "TON DUC THANG UNIVERSITY")
-		(comment 1 "Schematic Designed by ...")
-		(comment 2 "PCB Designed by ...")
-		(comment 3 "Approved by ...")
+		(company "KiCad EDA")
 	)
 	(no_connect

Commit message: V1 layout update 8
Parts:
- removed SH8, SH9: SCREW HOLDER, SAMPI:SCREWHOLE-2.5M, symbol SAMPI:SCREWHOLDER
- removed TP1: 3V3 ISO, SAMPI:TP1MM, symbol SAMPI:TESTPOINT
- removed TP2: GND ISO, SAMPI:TP1MM, symbol SAMPI:TESTPOINT
Connections:
- no-connect marks 25 -> 15
Other:
- sheet TERMINALS ports: added AUX_RXD1, AUX_RXD2, AUX_TXD1, AUX_TXD2, DBG_RXD1, DBG_RXD2, DBG_TXD1, DBG_TXD2, SWO, USB1_DM, USB1_DP, USB1_VBUS, USB2_DM, USB2_DP, USB2_VBUS; removed DB_RXD, DB_TXD, DV_CTS, DV_RTS, DV_RXD, DV_TXD, ISO_DB_RXD, ISO_DB_TXD, ISO_DV_CTS, ISO_DV_RTS, ISO_DV_RXD, ISO_DV_TXD, ISO_PGC, ISO_PGD, TG_RST, ~{ISO_MCLR}
- sheet USB HUB ports: added USB1_VBUS, USB2_VBUS, USB3_N, USB3_P, USB3_VBUS, USB4_N, USB4_P, USB4_VBUS, XTALIN, XTALOUT; removed HUB_USB_VBUS, USB1_PWR_EN, USB2_PWR_EN
- sheet VCP ports: added EECLK, EECS, EEDATA, OSCI, OSCO, RXD1, RXD2, RXD3, RXD4, TXD1, TXD2, TXD3, TXD4, VCP_DM, VCP_DP, VCP_VBUS, ~{PWREN}; removed HS_CTS, HS_RTS, HS_RXD, HS_SLED, HS_TXD, LS_RXD, LS_SLED, LS_TXD, MODE_SLED, SCL, SDA, TG_RST, VCP_PGC, VCP_PGD, VCP_USB_N, VCP_USB_P, VCP_USB_VBUS, ~{BT_MODE}, ~{VCP_MCLR}
