File: V1/Design/HW.ACIM-DBG/HW.ACIM-DBG.kicad_pcb (KiCad board)
At the start: 4 copper layers, 70.1 x 69.8 mm, 85 parts, among them J1 USB C, J2 MICRO USB, J3 SNAP PINOUT, J4 VCP ICSP, J5 MCLS, Q1 20V/2.9A, Q2 20V/2.3A, Q3 20V/2.3A, SW1 PRG SEL, U1 LOAD SWITCHER, U2 LDO 3.3V, U3 USB HUB, U4 PIC32MM0064GPM028, U6 ISO6740, U7 ISO6740, Y1 24MHz

Commit message: V1 layout
Parts:
- removed OP1, OP2: OPTO-BJT-1CH, SAMPI:OPTO_SO4_7.6MM
- removed Q2, Q3: 20V/2.3A, SAMPI:SOT23
- removed R25, R28: 10K, SAMPI:RES0603
- removed R26, R29: 1K, SAMPI:RES0603
- removed R27: 5.1K, SAMPI:RES0603
- added C25: 10uF, SAMPI:CAP0603, F.Cu at (147.7, 124.6)
- added C30: 10uF, SAMPI:CAP0603, F.Cu at (147.7, 110.9)
- added C31: 100nF, SAMPI:CAP0603, F.Cu at (240.6, 79.9)
- added C5: 100nF, SAMPI:CAP0603, F.Cu at (253.7, 56.3)
- added D6: ARM, SAMPI:LED3MM, F.Cu at (244.9, 66.5)
- added G***: HIGH VOLTAGE, LOGO, F.Cu at (149.3, 132.5)
- added R19: 100K, SAMPI:RES0603, F.Cu at (244.3, 77.3)
- added R20: 100K, SAMPI:RES0603, F.Cu at (244.3, 79.9)
- added SH5: SCREW HOLDER, SAMPI:SCREWHOLE-2.5M, F.Cu at (109.5, 50.3)
- added SH6: SCREW HOLDER, SAMPI:SCREWHOLE-2.5M, F.Cu at (154.7, 95.5)
- added SH7: SCREW HOLDER, SAMPI:SCREWHOLE-2.5M, F.Cu at (109.5, 140.7)
- added SH8: SCREW HOLDER, SAMPI:SCREWHOLE-2.5M, F.Cu at (64.2, 116.5)
- added SH9: SCREW HOLDER, SAMPI:SCREWHOLE-2.5M, F.Cu at (102.7, 85.3)
- added TP3: 5V, SAMPI:TP1MM, F.Cu at (262.8, 76.2)
- added TP4: VTG(5V), SAMPI:TP1MM, F.Cu at (262.8, 79.8)
- added TP5: 3V3, SAMPI:TP1MM, F.Cu at (266.4, 76.2)
- added TP6: GND, SAMPI:TP1MM, F.Cu at (266.4, 79.8)
- added U5: ISO6742, SAMPI:SOIC16-W, F.Cu at (129.0, 117.8)
- C1: value 220uF -> 10uF; footprint SAMPI:CAP1411 -> SAMPI:CAP0603
- C10: value 22pF -> 1uF
- C11, C15: value 22pF -> 100nF
- C12, C18: value 1uF -> 100nF
- C14, C8: value 100nF -> 22pF
- C16: value 100nF -> 1uF
- C2, C4: value 220uF -> 100nF; footprint SAMPI:CAP1411 -> SAMPI:CAP0603
- C20, C21, C24: value 100nF -> 10uF
- C22: value 10uF -> 100nF
- C26, C6: value 10uF -> 220uF; footprint SAMPI:CAP0603 -> SAMPI:CAP1411
- C3: value 100nF -> 220uF; footprint SAMPI:CAP0603 -> SAMPI:CAP1411
- C7: value 10uF -> 22pF
- D2: value HS PORT -> LS PORT; footprint SAMPI:LED0603 -> SAMPI:LED3MM
- D3: value LS PORT -> MODE; footprint SAMPI:LED0603 -> SAMPI:LED3MM
- D4: value PIC -> HS PORT; footprint SAMPI:LED0603 -> SAMPI:LED3MM
- D5: value ARM -> PIC; footprint SAMPI:LED0603 -> SAMPI:LED3MM
- J2: value MICRO USB -> VCP ICSP; footprint SAMPI:ZX60-B-5S(31) -> SAMPI:HD-1x6x1.27MM-TH
- J4: value VCP ICSP -> MICRO USB; footprint SAMPI:HD-1x6x1.27MM-TH -> SAMPI:ZX60-B-5S(31)
- J5: footprint SAMPI:IDC-2x5x2MM-TH -> SAMPI:IDC-2x6x2.54MM_TH
- R16: value 1K -> 10K
- R17: value 100K -> 1K
- R21, R22: value 100R -> 1K
- R23: value 1K -> 100R
- R24: value 10K -> 100R
- R5: value 100K -> 12K
- R6: value 12K -> 100K
- TP1: value 5V -> 3V3 ISO
- TP2: value 3V3 -> GND ISO
- U1: value LOAD SWITCHER -> LDO 3.3V; footprint SAMPI:SOT363 -> SAMPI:DFN8_3x3_MCHP
- U2: value LDO 3.3V -> USB HUB; footprint SAMPI:DFN8_3x3_MCHP -> SAMPI:QFN-24-4x4-EP
- U3: value USB HUB -> PIC32MM0064GPM028; footprint SAMPI:QFN-24-4x4-EP -> SAMPI:UQFN28-4x4-EP
- U4: value PIC32MM0064GPM028 -> ISO6742; footprint SAMPI:UQFN28-4x4-EP -> SAMPI:SOIC16-W
- U6: value ISO6740 -> ISO6742
- U7: value ISO6740 -> LOAD SWITCHER; footprint SAMPI:SOIC16-W -> SAMPI:SOT363
- moved SH2 141.2 mm to (64.2, 140.7)
- moved SH1 130.8 mm to (64.2, 52.2)
- moved U1 118.3 mm to (272.2, 65.5)
- moved J3 110.4 mm to (81.2, 121.5)
- moved C4 108.1 mm to (253.7, 53.6)
- moved J4 98.6 mm to (81.2, 52.9), turned to 90 degrees
- moved C7 91.2 mm to (253.7, 58.9)
- moved C8 91.2 mm to (253.7, 61.5)
- moved J5 82.9 mm to (132.1, 138.0)
- moved TP2 82.0 mm to (154.7, 131.3)
- moved R21 81.8 mm to (248.0, 72.0)
- moved R22 81.8 mm to (248.0, 74.7)
- moved TP1 80.9 mm to (154.7, 126.3)
- moved D5 78.5 mm to (244.9, 60.8)
- moved C6 77.8 mm to (269.6, 54.6)
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Connections:
- C10 pad 2: Net-(U3-CRFILT) -> Net-(U2-CRFILT)
- C11 pad 2: Net-(U3-XTALOUT/CLKIN_EN) -> +3V3
- C12 pad 2: Net-(U3-CRFILT) -> Net-(U2-PLLFILT)
- C13 pad 2: Net-(U3-PLLFILT) -> +3V3
- C14 pad 2: +3V3 -> Net-(U2-PLLFILT)
- C15 pad 2: Net-(U3-PLLFILT) -> Net-(U2-~{RESET})
- C16 pad 2: Net-(U3-~{RESET}) -> +3V3
- C18 pad 2: +3V3 -> /VCP/~{VCP_MCLR}
- C21 pad 2: /VCP/~{VCP_MCLR} -> Net-(U3-VCAP)
- C22 pad 2: +3V3 -> Net-(BT1-Pad1)
- C23 pad 1: GND -> GND_ISO
- C23 pad 2: Net-(U4-VCAP) -> +3V3_ISO
- C24 pad 1: GND -> GND_ISO
- C24 pad 2: Net-(BT1-Pad1) -> +3V3_ISO
- C27 pad 2: +3V3 -> VTG
- C29 pad 1: GND_ISO -> GND
- C29 pad 2: +3V3_ISO -> +3V3
- C7 pad 2: Net-(J2-VCC) -> Net-(U2-XTALIN/CLKIN)
- C8 pad 2: +5V -> Net-(U2-CRFILT)
- C9 pad 2: Net-(U3-XTALIN/CLKIN) -> Net-(U2-XTALOUT/CLKIN_EN)
- J2 pad 1: Net-(J2-VCC) -> /VCP/~{VCP_MCLR}
- J2 pad 2: /ISOLATOR/PRG_USB_N -> +3V3
- J2 pad 3: /ISOLATOR/PRG_USB_P -> GND
- J2 pad 4: unconnected-(J2-ID-Pad4) -> /VCP/VCP_PGD
- J2 pad 5: GND -> /VCP/VCP_PGC
- J2 pad 6: GND -> unconnected-(J2-Pad6)
- J3 pad 1: /ISOLATOR/~{MCLR} -> Net-(SW1-NO1)
- J3 pad 2: /ISOLATOR/VDD_SEN -> unconnected-(J3-Pad2)
- J3 pad 3: GND -> unconnected-(J3-Pad3)
- J3 pad 4: Net-(SW1-NC1) -> /ISOLATOR/PGC
- J3 pad 5: /ISOLATOR/PGC -> Net-(SW1-NC1)
- J3 pad 6: unconnected-(J3-Pad6) -> GND
- J3 pad 7: unconnected-(J3-Pad7) -> /ISOLATOR/VDD_SEN
- J3 pad 8: Net-(SW1-NO1) -> /ISOLATOR/~{MCLR}
- J4 pad 1: /VCP/~{VCP_MCLR} -> VTG
- J4 pad 2: +3V3 -> /ISOLATOR/PRG_USB_N
- J4 pad 3: GND -> /ISOLATOR/PRG_USB_P
- J4 pad 4: /VCP/VCP_PGD -> unconnected-(J4-ID-Pad4)
- J4 pad 5: /VCP/VCP_PGC -> GND
- J4 pad 6: unconnected-(J4-Pad6) -> GND
- Q1 pad 1: unconnected-(Q1-G-Pad1) -> Net-(Q1-G)
- Q1 pad 2: unconnected-(Q1-S-Pad2) -> GND
- Q1 pad 3: unconnected-(Q1-D-Pad3) -> /ISOLATOR/~{MCLR}
- R10 pad 2: Net-(U3-SUSP_IND/LOCAL_PWR/NON_REM0) -> Net-(U2-SUSP_IND/LOCAL_PWR/NON_REM0)
- R13 pad 1: Net-(D2-PadA) -> Net-(D4-PadA)
- R14 pad 1: Net-(D3-PadA) -> Net-(D2-PadA)
- R15 pad 1: Net-(D4-PadA) -> Net-(D3-PadA)
- R15 pad 2: Net-(SW1-NC2) -> /VCP/MODE_SLED
- R16 pad 1: Net-(D5-PadA) -> Net-(BT1-Pad1)
- R16 pad 2: Net-(SW1-NO2) -> +3V3
- R17 pad 1: GND -> Net-(Q1-G)
- R17 pad 2: Net-(SW1-NC2) -> /ISOLATOR/TG_RST
- R18 pad 2: Net-(SW1-NO2) -> Net-(Q1-G)
- R21 pad 1: Net-(U7-OUTD) -> Net-(D5-PadA)
- R21 pad 2: /ISOLATOR/ISO_PGD -> Net-(SW1-NC2)
- R22 pad 1: /ISOLATOR/PGD -> Net-(D6-PadA)
- R22 pad 2: Net-(U6-OUTA) -> Net-(SW1-NO2)
- R23 pad 1: Net-(OP1-A) -> Net-(U4-OUTC)
- R23 pad 2: +3V3_ISO -> /ISOLATOR/ISO_PGD
- R24 pad 1: Net-(OP1-C) -> /ISOLATOR/PGD
- R24 pad 2: +3V3 -> Net-(U4-OUTB)
- R5 pad 1: Net-(U3-~{RESET}) -> GND
- R5 pad 2: +3V3 -> Net-(U2-RBIAS)
- R6 pad 1: GND -> Net-(U2-~{RESET})
- R6 pad 2: Net-(U3-RBIAS) -> +3V3
- R7 pad 2: Net-(U3-SDA/SMBDATA/NON_REM1) -> Net-(U2-SDA/SMBDATA/NON_REM1)
- R8 pad 2: Net-(U3-SCL/SMBCLK/CFG_SEL0) -> Net-(U2-SCL/SMBCLK/CFG_SEL0)
- R9 pad 2: Net-(U3-SUSP_IND/LOCAL_PWR/NON_REM0) -> Net-(U2-SUSP_IND/LOCAL_PWR/NON_REM0)
- SW1 pad 5: Net-(J2-VCC) -> VTG
- TP1 pad 1: +5V -> +3V3_ISO
- TP2 pad 1: +3V3 -> GND_ISO
- U1 pad 1: Net-(J2-VCC) -> +5V
- U1 pad 2: GND -> +5V
- U1 pad 3: unconnected-(U1-NC-Pad3) -> +5V
- U1 pad 4: +5V -> GND
- U1 pad 6: /ISOLATOR/PRG_VBUS -> Net-(U1-CDELAY)
- U2 pad 1: +5V -> +3V3
- U2 pad 2: +5V -> /ISOLATOR/PRG_USB_N
- U2 pad 3: +5V -> /ISOLATOR/PRG_USB_P
- U2 pad 4: GND -> /USB HUB/USB2_N
- U2 pad 5: GND -> /USB HUB/USB2_P
- U2 pad 6: unconnected-(U2-CDELAY-Pad6) -> GND
- U2 pad 7: +3V3 -> /ISOLATOR/PRG_VBUS
- U2 pad 8: +3V3 -> unconnected-(U2-~{OCS1}-Pad8)
- U2 pad 9: GND -> +3V3
- U3 pad 1: +3V3 -> /VCP/VCP_PGD
- U3 pad 10: Net-(U3-CRFILT) -> +3V3
- U3 pad 11: /USB HUB/USB2_PWR_EN -> unconnected-(U3-PGED3/RP11/ASDA1/USBID/SS3/FSYNC3/OCM3E/RB5-Pad11)
- U3 pad 12: unconnected-(U3-~{OCS2}-Pad12) -> /USB HUB/USB2_PWR_EN
- U3 pad 13: Net-(U3-SDA/SMBDATA/NON_REM1) -> unconnected-(U3-RP12/SDA3/SDI3/OCM3F/RB7-Pad13)
- U3 pad 14: Net-(U3-SCL/SMBCLK/CFG_SEL0) -> unconnected-(U3-TCK/RP13/SCL1/U1CTS/SCK1/OCM1A/RB8-Pad14)
- U3 pad 15: Net-(U3-~{RESET}) -> unconnected-(U3-TMS/REFCLKI/RP14/SDA1/T1CK/T1G/T2CK/T2G/U1RTS/U1BCLK/SDO1/OCM1B/INT2/RB9-Pad15)
- U3 pad 16: /USB HUB/HUB_USB_VBUS -> unconnected-(U3-PGEC3/TDO/RP18/ASCL1/T3CK/T3G/USBOEN/SDO3/OCM2A/RC9-Pad16)
- U3 pad 17: Net-(U3-SUSP_IND/LOCAL_PWR/NON_REM0) -> Net-(U3-VCAP)
- U3 pad 18: +3V3 -> /USB HUB/USB2_N
- U3 pad 19: /USB HUB/USB_N -> /USB HUB/USB2_P
- U3 pad 2: /ISOLATOR/PRG_USB_N -> /VCP/VCP_PGC
- U3 pad 20: /USB HUB/USB_P -> +3V3
- U3 pad 21: Net-(U3-XTALOUT/CLKIN_EN) -> unconnected-(U3-AN8/LVDIN/RP15/SCL3/SCK3/OCM3A/RB13-Pad21)
- U3 pad 22: Net-(U3-XTALIN/CLKIN) -> unconnected-(U3-CVREF/AN9/C3INB/RP16/RTCC/U1TX/VBUSON/SDI1/OCM3B/INT1/RB14-Pad22)
- U3 pad 23: Net-(U3-PLLFILT) -> unconnected-(U3-AN10/C3INA/REFCLKO/RP17/U1RX/SS1/FSYNC1/OCM2B/INT0/RB15-Pad23)
- U3 pad 24: Net-(U3-RBIAS) -> GND
- U3 pad 25: GND -> +3V3
- U3 pad 3: /ISOLATOR/PRG_USB_P -> /ISOLATOR/DB_TXD
- U3 pad 4: /USB HUB/USB2_N -> /ISOLATOR/DB_RXD
- U3 pad 5: /USB HUB/USB2_P -> GND
- U3 pad 6: GND -> unconnected-(U3-OSC1/CLKI/AN5/RP3/OCM1C/RA2-Pad6)
- U3 pad 7: /ISOLATOR/PRG_VBUS -> unconnected-(U3-OSC2/CLKO/AN6/C3IND/RP4/OCM1D/RA3-Pad7)
- U3 pad 9: +3V3 -> unconnected-(U3-SOSCO/SCLKI/RP5/PWRLCLK/OCM3D/RA4-Pad9)
- U4 pad 1: /VCP/VCP_PGD -> +3V3_ISO
- U4 pad 11: unconnected-(U4-PGED3/RP11/ASDA1/USBID/SS3/FSYNC3/OCM3E/RB5-Pad11) -> /ISOLATOR/~{MCLR}
- U4 pad 12: /USB HUB/USB2_PWR_EN -> /ISOLATOR/PGD
- U4 pad 13: unconnected-(U4-RP12/SDA3/SDI3/OCM3F/RB7-Pad13) -> Net-(U4-OUTB)
- U4 pad 14: unconnected-(U4-TCK/RP13/SCL1/U1CTS/SCK1/OCM1A/RB8-Pad14) -> /ISOLATOR/PGC
- U4 pad 15: unconnected-(U4-TMS/REFCLKI/RP14/SDA1/T1CK/T1G/T2CK/T2G/U1RTS/U1BCLK/SDO1/OCM1B/INT2/RB9-Pad15) -> GND
- U4 pad 16: unconnected-(U4-PGEC3/TDO/RP18/ASCL1/T3CK/T3G/USBOEN/SDO3/OCM2A/RC9-Pad16) -> +3V3
- U4 pad 2: /VCP/VCP_PGC -> GND_ISO
- U4 pad 3: /ISOLATOR/DB_TXD -> /ISOLATOR/ISO_PGC
- U4 pad 4: /VCP/LS_TXD -> /ISOLATOR/ISO_PGD
- U4 pad 5: GND -> Net-(U4-OUTC)
- U4 pad 6: unconnected-(U4-OSC1/CLKI/AN5/RP3/OCM1C/RA2-Pad6) -> /ISOLATOR/~{ISO_MCLR}
- U4 pad 7: /VCP/~{BT_MODE} -> +3V3_ISO
- U4 pad 8: unconnected-(U4-SOSCI/AN7/RP10/OCM3C/RB4-Pad8) -> GND_ISO
- U4 pad 9: unconnected-(U4-SOSCO/SCLKI/RP5/PWRLCLK/OCM3D/RA4-Pad9) -> GND
- U6 pad 11: /ISOLATOR/DB_TXD -> unconnected-(U6-IND-Pad11)
- U6 pad 12: /ISOLATOR/DV_RTS -> /ISOLATOR/DB_RXD
- U6 pad 13: /ISOLATOR/DV_TXD -> /ISOLATOR/DB_TXD
- U6 pad 14: Net-(U6-OUTA) -> /ISOLATOR/VDD_SEN
- U6 pad 3: /ISOLATOR/ISO_PGD -> +3V3_ISO
- U6 pad 4: /ISOLATOR/ISO_DV_TXD -> /ISOLATOR/ISO_DB_TXD
- U6 pad 5: /ISOLATOR/ISO_DV_RTS -> /ISOLATOR/ISO_DB_RXD
- U6 pad 6: /ISOLATOR/ISO_DB_TXD -> unconnected-(U6-OUTD-Pad6)
- U6 pad 7: unconnected-(U6-NC-Pad7) -> +3V3_ISO
- U7 pad 1: +3V3 -> VTG
- U7 pad 3: /ISOLATOR/HS_RXD -> unconnected-(U7-NC-Pad3)
- U7 pad 4: /ISOLATOR/HS_CTS -> +5V
- U7 pad 5: /ISOLATOR/PGC -> GND
- U7 pad 6: /ISOLATOR/PGD -> /ISOLATOR/PRG_VBUS
- Y1 pad 1: Net-(U3-XTALIN/CLKIN) -> Net-(U2-XTALIN/CLKIN)
- Y1 pad 3: Net-(U3-XTALOUT/CLKIN_EN) -> Net-(U2-XTALOUT/CLKIN_EN)
Routing:
- net +3V3_ISO: track 0.00 -> 86.3 mm, vias 0 -> 6
- net /ISOLATOR/~{ISO_MCLR}: track 0.00 -> 25.3 mm, vias 0 -> 1
- net /ISOLATOR/ISO_DB_TXD: track 0.00 -> 24.4 mm
- net /ISOLATOR/ISO_DB_RXD: track 0.00 -> 22.3 mm
- net /ISOLATOR/ISO_DV_RTS: track 0.00 -> 17.6 mm
- net /ISOLATOR/ISO_DV_CTS: track 0.00 -> 17.6 mm
- net /ISOLATOR/ISO_DV_TXD: track 0.00 -> 17.3 mm
- net /ISOLATOR/ISO_DV_RXD: track 0.00 -> 17.2 mm, vias 0 -> 1
- net /ISOLATOR/ISO_PGD: track 0.00 -> 16.7 mm
- net /ISOLATOR/ISO_PGC: track 0.00 -> 15.1 mm, vias 0 -> 1
- net Net-(U4-OUTC): track 0.00 -> 2.03 mm
- net GND_ISO: track 0.00 -> 0.38 mm, vias 0 -> 6
- added copper zone on B.Cu, net GND_ISO
- added copper zone on F.Cu, net GND_ISO
- added copper zone on In1.Cu, net GND_ISO
- added copper zone on In2.Cu, net GND_ISO
Other:
- board size 70.1 x 69.8 mm -> 95 x 95 mm
- board text added: "3V3 DVRXD"
- board text added: "GND DVRTS"
- board text added: "N.C DBRXD"
- board text added: "PGC DBTXD"
- board text added: "PGD DVCTS"
- board text added: "RST DVTXD"

Commit message: V1 layout update 1
Parts:
- moved D5 185.4 mm to (72.4, 129.0)
- moved D6 185.4 mm to (72.4, 134.6)
- moved SW1 157.4 mm to (89.0, 130.2)
- moved R5 140.3 mm to (125.3, 63.7), turned to 90 degrees
- moved Y1 139.5 mm to (129.6, 61.0)
- moved U2 134.1 mm to (132.5, 66.2)
- moved C12 132.2 mm to (125.3, 61.0), turned to -90 degrees
- moved C14 130.5 mm to (126.9, 63.7), turned to 90 degrees
- moved F1 128.5 mm to (138.4, 54.3), turned to -90 degrees
- moved C7 126.8 mm to (126.9, 61.0), turned to -90 degrees
- moved D1 126.3 mm to (146.6, 57.7), turned to -90 degrees
- moved C9 125.8 mm to (132.2, 61.0), turned to 90 degrees
- moved BT1 117.6 mm to (101.5, 130.2)
- moved R2 112.2 mm to (149.0, 57.7), turned to 90 degrees
- moved R1 110.6 mm to (150.6, 57.7), turned to 90 degrees
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Connections:
- D1 pad 2: /USB HUB/USB_N -> /USB HUB/USB_P
- D1 pad 3: /USB HUB/USB_P -> /USB HUB/USB_N
Routing:
- net Net-(F1-Pad1): track 0.00 -> 10.8 mm, vias 0 -> 4
- net Net-(U2-XTALOUT/CLKIN_EN): track 0.00 -> 8.63 mm
- net Net-(U2-PLLFILT): track 0.00 -> 7.65 mm
- net Net-(U2-RBIAS): track 0.00 -> 6.65 mm
- net Net-(U2-XTALIN/CLKIN): track 0.00 -> 6.52 mm
- net /USB HUB/USB_P: track 0.00 -> 5.97 mm
- net Net-(J1-CC2): track 0.00 -> 5.08 mm, vias 0 -> 1
- net GND: track 0.00 -> 2.76 mm
- net /USB HUB/USB_N: track 0.00 -> 2.36 mm

Commit message: V1 layout update 6
Parts:
- removed C18: 100nF, SAMPI:CAP0603
- removed C23, C24, C25, C28, C29, C30: 10uF, SAMPI:CAP0603
- removed F1: 500mA, SAMPI:FUSE0805
- removed G***: HIGH VOLTAGE, LOGO
- removed J2: VCP ICSP, SAMPI:HD-1x6x1.27MM-TH
- removed U6: ISO6742, SAMPI:SOIC16-W
- added BT3: TG RESET, SAMPI:BUTTON_4P_6x6, F.Cu at (175.4, 95.6)
- added C34: 10nF, SAMPI:CAP0603, F.Cu at (192.5, 85.5)
- added C35: 10nF, SAMPI:CAP0603, F.Cu at (192.5, 88.1)
- added C36: 10uF, SAMPI:CAP0603, F.Cu at (192.5, 90.7)
- added C37: 10nF, SAMPI:CAP0603, F.Cu at (192.5, 93.3)
- added C38: 100nF, SAMPI:CAP0603, F.Cu at (196.2, 85.5)
- added C39: 22pF, SAMPI:CAP0603, F.Cu at (196.2, 88.1)
- added C40: 100nF, SAMPI:CAP0603, F.Cu at (172.3, 55.8)
- added C41: 100nF, SAMPI:CAP0603, F.Cu at (172.3, 58.4)
- added C42: 100nF, SAMPI:CAP0603, F.Cu at (172.3, 61.0)
- added C43: 100nF, SAMPI:CAP0603, F.Cu at (172.3, 63.6)
- added C44: 100nF, SAMPI:CAP0603, F.Cu at (172.3, 66.2)
- added C45: 10uF, SAMPI:CAP0603, F.Cu at (172.3, 68.8)
- added C46: 10uF, SAMPI:CAP0603, F.Cu at (172.3, 71.4)
- added C47: 10uF, SAMPI:CAP0603, F.Cu at (172.3, 74.0)
- added C48: 100nF, SAMPI:CAP0603, F.Cu at (176.0, 55.8)
- added C49: 100nF, SAMPI:CAP0603, F.Cu at (176.0, 58.4)
- added C50: 100nF, SAMPI:CAP0603, F.Cu at (176.0, 61.0)
- added C51: 22pF, SAMPI:CAP0603, F.Cu at (176.0, 63.6)
- added C52: 100nF, SAMPI:CAP0603, F.Cu at (176.0, 66.2)
- added C53: 100nF, SAMPI:CAP0603, F.Cu at (176.0, 68.8)
- added C54: 10uF, SAMPI:CAP0603, F.Cu at (176.0, 71.4)
- added C55: 22pF, SAMPI:CAP0603, F.Cu at (176.0, 74.0)
- added C56: 22pF, SAMPI:CAP0603, F.Cu at (179.7, 55.8)
- added D10: TR1, SAMPI:LED0606_4P, F.Cu at (191.0, 65.0)
- added D7: TR4, SAMPI:LED0606_4P, F.Cu at (191.0, 56.0)
- added D8: TR3, SAMPI:LED0606_4P, F.Cu at (191.0, 59.0)
- added D9: TR2, SAMPI:LED0606_4P, F.Cu at (191.0, 62.0)
- added FT1: 120R@100MHz, SAMPI:FT0603, F.Cu at (196.2, 90.7)
- added FT2: 120R@100MHz, SAMPI:FT0603, F.Cu at (196.2, 93.3)
- added FT3: 120R@100MHz, SAMPI:FT0603, F.Cu at (179.7, 58.4)
- added FT4: 120R@100MHz, SAMPI:FT0603, F.Cu at (179.7, 61.0)
- added FT5: 120R@100MHz, SAMPI:FT0603, F.Cu at (179.7, 63.6)
- added FT6: 120R@100MHz, SAMPI:FT0603, F.Cu at (179.7, 66.2)
- added H1: EXT DBG PORT, Liem:DIL14-1.27-SMD, F.Cu at (175.8, 87.9)
- added H2: DBG PORT, Liem:RPDBG, F.Cu at (184.5, 94.2)
- added Q2: MFET N, SAMPI:SOT23, F.Cu at (193.0, 97.0)
- added R25: 100K, SAMPI:RES0603, F.Cu at (199.9, 85.5)
- added R26: 10K, SAMPI:RES0603, F.Cu at (199.9, 88.1)
- added R27: 1.1K, SAMPI:RES0603, F.Cu at (179.7, 68.8)
- added R28: 10K, SAMPI:RES0603, F.Cu at (179.7, 71.4)
- added R29: 2.2K, SAMPI:RES0603, F.Cu at (179.7, 74.0)
- added R34: 10K, SAMPI:RES0603, F.Cu at (199.9, 90.7)
- added R35: 10K, SAMPI:RES0603, F.Cu at (199.9, 93.3)
- added R38: 10K, SAMPI:RES0603, F.Cu at (183.4, 55.8)
- added R39: 10K, SAMPI:RES0603, F.Cu at (183.4, 58.4)
- added R46: 12K/1%, SAMPI:RES0603, F.Cu at (183.4, 61.0)
- added R47: 10K, SAMPI:RES0603, F.Cu at (183.4, 63.6)
- added R48: 100K, SAMPI:RES0603, F.Cu at (183.4, 66.2)
- added R49: 1.1K, SAMPI:RES0603, F.Cu at (183.4, 68.8)
- added R50: 1.1K, SAMPI:RES0603, F.Cu at (183.4, 71.4)
- added R51: 1.1K, SAMPI:RES0603, F.Cu at (183.4, 74.0)
- added R52: 1.1K, SAMPI:RES0603, F.Cu at (187.1, 55.8)
- added R53: 1.1K, SAMPI:RES0603, F.Cu at (187.1, 58.4)
- added R54: 1.1K, SAMPI:RES0603, F.Cu at (187.1, 61.0)
- added R55: 1.1K, SAMPI:RES0603, F.Cu at (187.1, 63.6)
- added R56: 1.1K, SAMPI:RES0603, F.Cu at (187.1, 66.2)
- added U10: 12MHz, SAMPI:CDFN2520-ABM10, F.Cu at (181.5, 77.6)
- added U8: FT4232H, SAMPI:VQFN-56_FTDI, F.Cu at (194.0, 71.5)
- added U9: SHIFT REG 8BIT, SAMPI:TSSOP16-SOT403-1, F.Cu at (174.8, 78.8)
- C10: value 1uF -> 100nF
- C11, C12: value 100nF -> 10nF
- C13, C19, C22: value 100nF -> 22pF
- C14: value 22pF -> 10nF
- C16: value 1uF -> 10nF
- C20, C21: value 10uF -> 22pF
- D2: value LS PORT -> VCP; footprint SAMPI:LED3MM -> SAMPI:LED0603
- D3: value MODE -> POWER; footprint SAMPI:LED3MM -> SAMPI:LED0603
- D4: value HS PORT -> TARGET; footprint SAMPI:LED3MM -> SAMPI:LED0603
- D5: value PIC -> ICSP/UPDI; footprint SAMPI:LED3MM -> SAMPI:LED0603
- D6: value ARM -> SWD; footprint SAMPI:LED3MM -> SAMPI:LED0603
- J5: value MCLS -> MCDBG PORT
- Q1: value 20V/2.9A -> MFET N
- R10: value 47K -> 100K
- R11: value 10K -> 1K
- R14, R17: value 1K -> 5.1K
- R15: value 1K -> 35.7K
- R16: value 10K -> 35.7K
- R18, R3, R4: value 100K -> 10K
- R23, R24: value 100R -> 10K
- R5: value 12K -> 10K
- R6: value 100K -> 12K/1%
- R9: footprint Liem:RES0402 -> SAMPI:RES0603
- U2: value USB HUB -> USB HUB 2.0 4-CH; footprint SAMPI:QFN-24-4x4-EP -> SAMPI:SQFN36_6x6_MCHP
- U3: value PIC32MM0064GPM028 -> SPI EEPROM; footprint SAMPI:UQFN28-4x4-EP -> SAMPI:SOT-23-6_MCHP
- U4: value ISO6742 -> USB PD; footprint SAMPI:SOIC16-W -> SAMPI:QFN16
- U5: value ISO6742 -> eFuse; footprint SAMPI:SOIC16-W -> SAMPI:DFN10-EP-3x3
- moved U5 47.1 mm to (176.1, 118.7), turned to 0 degrees
- moved R24 41.0 mm to (180.3, 119.9), turned to 0 degrees
- moved R23 40.7 mm to (180.3, 117.2), turned to 0 degrees
- moved U4 36.4 mm to (176.4, 113.3), turned to 0 degrees
- moved TP2 34.8 mm to (186.0, 116.0)
- moved TP1 34.2 mm to (186.0, 112.4)
Connections:
- BT1 pad 1: Net-(BT1-Pad1) -> Net-(Q2-D)
- BT1 pad 2: Net-(BT1-Pad1) -> Net-(Q2-D)
- C1 pad 2: +5V -> VBUS
- C11 pad 2: +3V3 -> Net-(C11-Pad2)
- C12 pad 2: Net-(U2-PLLFILT) -> Net-(U2-CRFILT)
- C14 pad 2: Net-(U2-PLLFILT) -> Net-(C11-Pad2)
- C15 pad 2: Net-(U2-~{RESET}) -> Net-(U2-PLLFILT)
- C16 pad 2: +3V3 -> Net-(C16-Pad2)
- C17 pad 2: +3V3 -> Net-(Q2-D)
- C2 pad 2: /USB HUB/HUB_USB_VBUS -> Net-(U5-SS)
- C21 pad 2: Net-(U3-VCAP) -> +3V3
- C22 pad 2: Net-(BT1-Pad1) -> +3V3
- C5 pad 1: GND -> Net-(U1-CDELAY)
- C5 pad 2: Net-(U1-CDELAY) -> GND
- C7 pad 2: Net-(U2-XTALIN/CLKIN) -> /USB HUB/XTALIN
- C8 pad 2: Net-(U2-CRFILT) -> +3V3
- C9 pad 2: Net-(U2-XTALOUT/CLKIN_EN) -> /USB HUB/XTALOUT
- D1 pad 4: +5V -> VBUS
- D2 pad K: GND -> Net-(Q1-D)
- D3 pad A: Net-(D3-PadA) -> Net-(U1-PWRGD)
- J1 pad A4B9: Net-(F1-Pad1) -> VBUS
- J1 pad B4A9: Net-(F1-Pad1) -> VBUS
- J3 pad 4: /ISOLATOR/PGC -> /TERMINALS/PGC
- J3 pad 7: /ISOLATOR/VDD_SEN -> /TERMINALS/VDD_SEN
- J3 pad 8: /ISOLATOR/~{MCLR} -> /TERMINALS/~{MCLR}
- J4 pad 2: /ISOLATOR/PRG_USB_N -> /TERMINALS/PRG_USB_N
- J4 pad 3: /ISOLATOR/PRG_USB_P -> /TERMINALS/PRG_USB_P
- J5 pad 1: /ISOLATOR/ISO_DV_TXD -> unconnected-(J5-DB_TXD-Pad1)
- J5 pad 10: /ISOLATOR/ISO_PGC -> /TERMINALS/PGC
- J5 pad 11: /ISOLATOR/ISO_DB_RXD -> unconnected-(J5-USB_DM-Pad11)
- J5 pad 2: /ISOLATOR/~{ISO_MCLR} -> /TERMINALS/~{MCLR}
- J5 pad 3: /ISOLATOR/ISO_DV_RXD -> unconnected-(J5-DB_RXD-Pad3)
- J5 pad 4: +3V3_ISO -> /TERMINALS/VDD_SEN
- J5 pad 5: /ISOLATOR/ISO_DV_RTS -> unconnected-(J5-DV_TXD-Pad5)
- J5 pad 6: GND_ISO -> GND
- J5 pad 7: /ISOLATOR/ISO_DV_CTS -> unconnected-(J5-DV_RXD-Pad7)
- J5 pad 8: /ISOLATOR/ISO_PGD -> /TERMINALS/PGD
- J5 pad 9: /ISOLATOR/ISO_DB_TXD -> unconnected-(J5-UDB_DP-Pad9)
- Q1 pad 3: /ISOLATOR/~{MCLR} -> Net-(Q1-D)
- R10 pad 1: +3V3 -> GND
- R10 pad 2: Net-(U2-SUSP_IND/LOCAL_PWR/NON_REM0) -> Net-(U2-SCL/SMBCLK/CFG_SEL0)
- R11 pad 1: /VCP/~{VCP_MCLR} -> Net-(U1-PWRGD)
- R12 pad 1: Net-(BT1-Pad1) -> GND
- R12 pad 2: /VCP/~{BT_MODE} -> Net-(U5-ILIM/IMON)
- R13 pad 2: /VCP/HS_SLED -> /TERMINALS/VDD_SEN
- R14 pad 1: Net-(D2-PadA) -> GND
- R14 pad 2: /VCP/LS_SLED -> Net-(U4-VMON)
- R15 pad 1: Net-(D3-PadA) -> Net-(U4-VMON)
- R15 pad 2: /VCP/MODE_SLED -> VBUS
- R16 pad 1: Net-(BT1-Pad1) -> Net-(U5-OVP)
- R16 pad 2: +3V3 -> VBUS
- R17 pad 1: Net-(Q1-G) -> GND
- R17 pad 2: /ISOLATOR/TG_RST -> Net-(U5-OVP)
- R18 pad 1: GND -> Net-(Q2-D)
- R18 pad 2: Net-(Q1-G) -> VBUS
- R23 pad 1: Net-(U4-OUTC) -> Net-(U4-~{OCS})
- R23 pad 2: /ISOLATOR/ISO_PGD -> +5V
- R24 pad 1: /ISOLATOR/PGD -> VBUS
- R24 pad 2: Net-(U4-OUTB) -> Net-(U4-ENABLE)
- R3 pad 1: /USB HUB/HUB_USB_VBUS -> /USB HUB/CC1
- R3 pad 2: +5V -> Net-(J1-CC1)
- R4 pad 1: GND -> /USB HUB/CC2
- R4 pad 2: /USB HUB/HUB_USB_VBUS -> Net-(J1-CC2)
- R5 pad 1: GND -> +3V3
- R5 pad 2: Net-(U2-RBIAS) -> Net-(U2-~{RESET})
- R6 pad 1: Net-(U2-~{RESET}) -> Net-(U2-RBIAS)
- R6 pad 2: +3V3 -> GND
- R7 pad 1: GND -> Net-(U2-SDA/SMBDATA/NON_REM1)
- R7 pad 2: Net-(U2-SDA/SMBDATA/NON_REM1) -> GND
- R8 pad 1: GND -> Net-(U2-HS_IND/CFG_SEL1)
- R8 pad 2: Net-(U2-SCL/SMBCLK/CFG_SEL0) -> +3V3
- SW1 pad 2: /ISOLATOR/PGD -> /TERMINALS/PGD
- U1 pad 5: GND -> Net-(U1-PWRGD)
- U2 pad 1: +3V3 -> /TERMINALS/PRG_USB_N
- U2 pad 10: Net-(U2-CRFILT) -> Net-(C11-Pad2)
- U2 pad 11: /USB HUB/USB2_PWR_EN -> GND
- U2 pad 12: unconnected-(U2-~{OCS2}-Pad12) -> /USB HUB/USB1_VBUS
- U2 pad 13: Net-(U2-SDA/SMBDATA/NON_REM1) -> unconnected-(U2-~{OCS1}-Pad13)
- U2 pad 14: Net-(U2-SCL/SMBCLK/CFG_SEL0) -> Net-(U2-CRFILT)
- U2 pad 15: Net-(U2-~{RESET}) -> Net-(C16-Pad2)
- U2 pad 16: /USB HUB/HUB_USB_VBUS -> /USB HUB/USB2_VBUS
- U2 pad 17: Net-(U2-SUSP_IND/LOCAL_PWR/NON_REM0) -> unconnected-(U2-~{OCS2}-Pad17)
- U2 pad 18: +3V3 -> /USB HUB/USB3_VBUS
- U2 pad 19: /USB HUB/USB_N -> unconnected-(U2-~{OCS3}-Pad19)
- U2 pad 2: /ISOLATOR/PRG_USB_N -> /TERMINALS/PRG_USB_P
- U2 pad 20: /USB HUB/USB_P -> /USB HUB/USB4_VBUS
- U2 pad 21: Net-(U2-XTALOUT/CLKIN_EN) -> unconnected-(U2-~{OCS4}-Pad21)
- U2 pad 22: Net-(U2-XTALIN/CLKIN) -> Net-(U2-SDA/SMBDATA/NON_REM1)
- U2 pad 23: Net-(U2-PLLFILT) -> Net-(C16-Pad2)
- U2 pad 24: Net-(U2-RBIAS) -> Net-(U2-SCL/SMBCLK/CFG_SEL0)
- U2 pad 25: GND -> Net-(U2-HS_IND/CFG_SEL1)
- U2 pad 3: /ISOLATOR/PRG_USB_P -> /USB HUB/USB2_N
- U2 pad 4: /USB HUB/USB2_N -> /USB HUB/USB2_P
- U2 pad 5: /USB HUB/USB2_P -> Net-(C11-Pad2)
- U2 pad 6: GND -> /USB HUB/USB3_N
- U2 pad 7: /ISOLATOR/PRG_VBUS -> /USB HUB/USB3_P
- U2 pad 8: unconnected-(U2-~{OCS1}-Pad8) -> /USB HUB/USB4_N
- U2 pad 9: +3V3 -> /USB HUB/USB4_P
- U3 pad 1: /VCP/VCP_PGD -> Net-(U3-DO)
- U3 pad 2: /VCP/VCP_PGC -> GND
- U3 pad 3: /ISOLATOR/DB_TXD -> /VCP/EEDATA
- U3 pad 4: /ISOLATOR/DB_RXD -> /VCP/EECLK
- U3 pad 5: GND -> /VCP/EECS
- U3 pad 6: unconnected-(U3-OSC1/CLKI/AN5/RP3/OCM1C/RA2-Pad6) -> +3V3
- U4 pad 1: +3V3_ISO -> Net-(U4-~{OCS})
- U4 pad 10: +3V3 -> unconnected-(U4-PPC_EN/~{3.0A_IND}-Pad10)
- U4 pad 11: /ISOLATOR/~{MCLR} -> unconnected-(U4-~{PLUG_ORIENTATION}-Pad11)
- U4 pad 12: /ISOLATOR/PGD -> Net-(U4-VMON)
- U4 pad 13: Net-(U4-OUTB) -> GND
- U4 pad 14: /ISOLATOR/PGC -> unconnected-(U4-NC-Pad14)
- U4 pad 15: GND -> unconnected-(U4-NC-Pad15)
- U4 pad 16: +3V3 -> VBUS
- U4 pad 2: GND_ISO -> Net-(U4-CFG_SEL)
- U4 pad 3: /ISOLATOR/ISO_PGC -> Net-(U4-ENABLE)
- U4 pad 4: /ISOLATOR/ISO_PGD -> /USB HUB/FAULT_IND
- U4 pad 5: Net-(U4-OUTC) -> Net-(Q2-G)
- U4 pad 6: /ISOLATOR/~{ISO_MCLR} -> /USB HUB/CC2
- U4 pad 7: +3V3_ISO -> /USB HUB/CC1
- U4 pad 8: GND_ISO -> unconnected-(U4-~{VCONN2_OUT}/~{LEGACY_IND}-Pad8)
- U4 pad 9: GND -> unconnected-(U4-~{VCONN1_OUT}/~{1.5A_IND}-Pad9)
- U5 pad 1: +3V3_ISO -> VBUS
- U5 pad 10: +3V3 -> +5V
- U5 pad 11: /ISOLATOR/DV_CTS -> GND
- U5 pad 2: GND_ISO -> VBUS
- U5 pad 3: /ISOLATOR/ISO_DV_TXD -> Net-(U5-SS)
- U5 pad 4: /ISOLATOR/ISO_DV_RTS -> Net-(Q2-D)
- U5 pad 5: /ISOLATOR/ISO_DV_RXD -> Net-(U5-ILIM/IMON)
- U5 pad 6: /ISOLATOR/ISO_DV_CTS -> GND
- U5 pad 7: +3V3_ISO -> Net-(U5-OVP)
- U5 pad 8: GND_ISO -> Net-(U4-~{OCS})
- U5 pad 9: GND -> +5V
- U7 pad 6: /ISOLATOR/PRG_VBUS -> /TERMINALS/PRG_VBUS
- Y1 pad 1: Net-(U2-XTALIN/CLKIN) -> /USB HUB/XTALIN
- Y1 pad 3: Net-(U2-XTALOUT/CLKIN_EN) -> /USB HUB/XTALOUT
Routing:
- net +3V3_ISO: track 86.3 -> 0.00 mm, vias 6 -> 0
- net /ISOLATOR/~{ISO_MCLR}: track 25.3 -> 0.00 mm, vias 1 -> 0
- net /ISOLATOR/ISO_DB_TXD: track 24.4 -> 0.00 mm
- net /ISOLATOR/ISO_DB_RXD: track 22.3 -> 0.00 mm
- net /ISOLATOR/ISO_DV_RTS: track 17.6 -> 0.00 mm
- net /ISOLATOR/ISO_DV_CTS: track 17.6 -> 0.00 mm
- net /ISOLATOR/ISO_DV_TXD: track 17.3 -> 0.00 mm
- net /ISOLATOR/ISO_DV_RXD: track 17.2 -> 0.00 mm, vias 1 -> 0
- net /ISOLATOR/ISO_PGD: track 16.7 -> 0.00 mm
- net (no net): track 0.00 -> 15.1 mm
- net /ISOLATOR/ISO_PGC: track 15.1 -> 0.00 mm, vias 1 -> 0
- net VBUS: track 0.00 -> 10.8 mm, vias 0 -> 4
- net Net-(F1-Pad1): track 10.8 -> 0.00 mm, vias 4 -> 0
- net Net-(U2-XTALOUT/CLKIN_EN): track 8.63 -> 0.00 mm
- net Net-(U2-XTALIN/CLKIN): track 6.52 -> 0.00 mm
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- removed copper zone on B.Cu, net GND_ISO
- removed copper zone on F.Cu, net GND_ISO
- removed copper zone on In1.Cu, net GND_ISO
- removed copper zone on In2.Cu, net GND_ISO
Other:
- board text removed: "3V3 DVRXD"
- board text removed: "GND DVRTS"
- board text removed: "N.C DBRXD"
- board text removed: "PGC DBTXD"
- board text removed: "PGD DVCTS"
- board text removed: "RST DVTXD"

Commit message: V1 layout update 7
Parts:
- added R30: 100K, SAMPI:RES0603, F.Cu at (177.0, 109.8)
- moved U10 16.9 mm to (196.3, 69.2)
- moved U8 12.9 mm to (206.9, 72.2)
- moved C31 7.68 mm to (248.2, 80.8)
- moved C27 7.68 mm to (244.5, 80.8)
- moved R20 7.68 mm to (251.9, 80.8)
Connections:
- C1 pad 2: VBUS -> +5V
- R24 pad 1: VBUS -> +5V
- R26 pad 1: VBUS -> +5V
- U4 pad 16: VBUS -> +5V
Routing:
- net (no net): track 15.1 -> 0.00 mm
- net Net-(U2-PLLFILT): track 7.65 -> 0.00 mm
- net Net-(U2-RBIAS): track 6.65 -> 0.00 mm
- net /USB HUB/XTALOUT: track 0.00 -> 1.58 mm

Commit message: V1 layout update 8
Parts:
- removed C1: 10uF, SAMPI:CAP0603
- removed C2: 100nF, SAMPI:CAP0603
- removed D4: TARGET, SAMPI:LED0603
- removed R12, R13: 1K, SAMPI:RES0603
- removed R14, R17: 5.1K, SAMPI:RES0603
- removed R15, R16: 35.7K, SAMPI:RES0603
- removed R23, R24, R26, R4: 10K, SAMPI:RES0603
- removed R30: 100K, SAMPI:RES0603
- removed SH8, SH9: SCREW HOLDER, SAMPI:SCREWHOLE-2.5M
- removed TP1: 3V3 ISO, SAMPI:TP1MM
- removed TP2: GND ISO, SAMPI:TP1MM
- removed U4: USB PD, SAMPI:QFN16
- removed U5: eFuse, SAMPI:DFN10-EP-3x3
- added F1: 750mA, Liem:FUSE1812, F.Cu at (102.1, 51.8)
- H2: value DBG PORT -> RPDBG; footprint Liem:RPDBG -> Liem:DIL10-1.27-SMD
- R27, R49, R50, R51, R52, R53, R54, R55, R56: value 1.1K -> 1K
- R3: value 10K -> 100K
- R46, R6: value 12K/1% -> 12K
- Y1: footprint SAMPI:CDFN3225-4LD-PL-1 -> SAMPI:CDFN2520-ABM10
- moved R3 211.2 mm to (64.7, 136.6)
- moved R9 202.9 mm to (70.7, 75.1)
- moved R6 201.3 mm to (67.0, 88.1)
- moved R7 201.3 mm to (67.0, 90.7)
- moved C10 200.8 mm to (59.6, 85.5)
- moved C15 200.0 mm to (63.3, 77.7)
- moved C4 195.0 mm to (59.6, 72.5)
- moved C5 195.0 mm to (59.6, 75.1)
- moved C8 195.0 mm to (59.6, 80.3)
- moved R10 195.0 mm to (70.7, 77.7)
- moved R8 194.8 mm to (70.7, 72.5)
- moved R20 190.5 mm to (68.1, 130.9)
- moved R22 188.1 mm to (67.9, 128.9)
- moved R21 187.4 mm to (68.0, 124.3)
- moved TP5 187.0 mm to (81.3, 103.1)
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Connections:
- BT1 pad 1: Net-(Q2-D) -> Net-(U1-~{SHDN})
- BT1 pad 2: Net-(Q2-D) -> Net-(U1-~{SHDN})
- C17 pad 2: Net-(Q2-D) -> Net-(U1-~{SHDN})
- C51 pad 2: /VCP/VCP_VBUS -> /USB HUB/USB1_VBUS
- D1 pad 4: VBUS -> +5V
- D5 pad K: GND -> Net-(Q2-D)
- D6 pad K: GND -> Net-(Q2-D)
- H1 pad 1: /TERMINALS/DBG_TXD -> /TERMINALS/DBG_TXD1
- H1 pad 11: /TERMINALS/AUX_TXD -> /TERMINALS/AUX_TXD1
- H1 pad 13: /TERMINALS/AUX_RXD -> /TERMINALS/AUX_RXD1
- H1 pad 3: /TERMINALS/DBG_RXD -> /TERMINALS/DBG_RXD1
- H1 pad 5: /TERMINALS/USB_DP -> /TERMINALS/USB1_DP
- H1 pad 7: /TERMINALS/USB_DM -> /TERMINALS/USB1_DM
- H1 pad 9: /TERMINALS/USB_VBUS -> /TERMINALS/USB1_VBUS
- H2 pad 1: /TERMINALS/DBG_TXD -> /TERMINALS/DBG_TXD1
- H2 pad 3: /TERMINALS/DBG_RXD -> /TERMINALS/DBG_RXD1
- H2 pad 5: /TERMINALS/USB_DP -> /TERMINALS/USB1_DP
- H2 pad 7: /TERMINALS/USB_DM -> /TERMINALS/USB1_DM
- H2 pad 9: /TERMINALS/USB_VBUS -> /TERMINALS/USB1_VBUS
- J1 pad A4B9: VBUS -> Net-(F1-Pad1)
- J1 pad B4A9: VBUS -> Net-(F1-Pad1)
- J3 pad 5: Net-(SW1-NC1) -> /TERMINALS/SWO
- J5 pad 1: unconnected-(J5-DB_TXD-Pad1) -> /TERMINALS/DBG_TXD2
- J5 pad 11: unconnected-(J5-USB_DM-Pad11) -> /TERMINALS/USB2_DM
- J5 pad 12: unconnected-(J5-VBUS-Pad12) -> /TERMINALS/USB2_VBUS
- J5 pad 3: unconnected-(J5-DB_RXD-Pad3) -> /TERMINALS/DBG_RXD2
- J5 pad 5: unconnected-(J5-DV_TXD-Pad5) -> /TERMINALS/AUX_TXD2
- J5 pad 7: unconnected-(J5-DV_RXD-Pad7) -> /TERMINALS/AUX_RXD2
- J5 pad 9: unconnected-(J5-UDB_DP-Pad9) -> /TERMINALS/USB2_DP
- Q2 pad 1: Net-(Q2-G) -> /TERMINALS/VDD_SEN
- R18 pad 1: Net-(Q2-D) -> Net-(U1-~{SHDN})
- R18 pad 2: VBUS -> +5V
- R3 pad 1: /USB HUB/CC1 -> GND
- R3 pad 2: Net-(J1-CC1) -> /TERMINALS/VDD_SEN
- R48 pad 1: /VCP/VCP_VBUS -> /USB HUB/USB1_VBUS
- SW1 pad 1: Net-(SW1-NC1) -> /TERMINALS/SWO
- U1 pad 3: +5V -> Net-(U1-~{SHDN})
- U2 pad 1: /TERMINALS/PRG_USB_N -> /USB HUB/USB1_N
- U2 pad 16: /USB HUB/USB2_VBUS -> /TERMINALS/USB1_VBUS
- U2 pad 18: /USB HUB/USB3_VBUS -> /TERMINALS/USB2_VBUS
- U2 pad 2: /TERMINALS/PRG_USB_P -> /USB HUB/USB1_P
- U2 pad 20: /USB HUB/USB4_VBUS -> /TERMINALS/PRG_VBUS
- U2 pad 3: /USB HUB/USB2_N -> /TERMINALS/USB1_DM
- U2 pad 4: /USB HUB/USB2_P -> /TERMINALS/USB1_DP
- U2 pad 6: /USB HUB/USB3_N -> /TERMINALS/USB2_DM
- U2 pad 7: /USB HUB/USB3_P -> /TERMINALS/USB2_DP
- U2 pad 8: /USB HUB/USB4_N -> /TERMINALS/PRG_USB_N
- U2 pad 9: /USB HUB/USB4_P -> /TERMINALS/PRG_USB_P
- U8 pad 11: /VCP/VCP_VBUS -> /USB HUB/USB1_VBUS
- U8 pad 12: /VCP/TXD1 -> /TERMINALS/DBG_RXD1
- U8 pad 13: /VCP/RXD1 -> /TERMINALS/DBG_TXD1
- U8 pad 22: /VCP/TXD2 -> /TERMINALS/AUX_RXD1
- U8 pad 23: /VCP/RXD2 -> /TERMINALS/AUX_TXD1
- U8 pad 32: /VCP/TXD3 -> /TERMINALS/DBG_RXD2
- U8 pad 33: /VCP/RXD3 -> /TERMINALS/DBG_TXD2
- U8 pad 42: /VCP/TXD4 -> /TERMINALS/AUX_RXD2
- U8 pad 46: /VCP/RXD4 -> /TERMINALS/AUX_TXD2
- U8 pad 7: /VCP/VCP_DM -> /USB HUB/USB1_N
- U8 pad 8: /VCP/VCP_DP -> /USB HUB/USB1_P
Routing:
- net VBUS: track 10.8 -> 0.00 mm, vias 4 -> 0
- net Net-(F1-Pad1): track 0.00 -> 10.8 mm, vias 0 -> 4
- net /USB HUB/XTALOUT: track 1.58 -> 0.00 mm
Other:
- board size 95 x 95 mm -> 60 x 95 mm

Commit message: V1 layout update 9
Parts:
- added C1: 100nF, SAMPI:CAP0603, F.Cu at (88.0, 50.8)
- moved C17 48.7 mm to (109.0, 66.2)
- moved C4 48.2 mm to (106.9, 63.1)
- moved TP4 45.6 mm to (88.7, 54.5)
- moved TP6 41.8 mm to (39.5, 104.3)
- moved R18 41.3 mm to (107.1, 60.6)
- moved U7 5.59 mm to (94.8, 50.0), turned to 180 degrees
- moved C31 2.44 mm to (94.8, 52.4), turned to 180 degrees
- moved C26 2.32 mm to (91.4, 50.8)
- moved C27 2.32 mm to (88.0, 52.4)
- moved R22 2.20 mm to (65.8, 129.7), turned to -90 degrees
- moved R21 2.19 mm to (65.8, 124.7), turned to -90 degrees
- moved R19 1.76 mm to (67.4, 124.7), turned to -90 degrees
- moved R20 1.43 mm to (67.4, 129.7), turned to -90 degrees
- moved R3 1.10 mm to (65.0, 135.5), turned to 180 degrees
- moved D1 1.01 mm to (110.5, 57.7)
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Routing:
- net GND: track 2.76 -> 49.1 mm
- net /TERMINALS/PGC: track 0.00 -> 27.0 mm
- net /TERMINALS/VDD_SEN: track 0.00 -> 22.8 mm
- net VTG: track 0.00 -> 21.8 mm
- net /TERMINALS/PGD: track 0.00 -> 17.7 mm
- net Net-(SW1-NC2): track 0.00 -> 13.5 mm
- net /TERMINALS/~{MCLR}: track 0.00 -> 13.4 mm
- net +5V: track 0.00 -> 11.0 mm
- net Net-(F1-Pad1): track 10.8 -> 19.8 mm
- net Net-(Q2-D): track 0.00 -> 7.21 mm
- net Net-(SW1-NO2): track 0.00 -> 6.68 mm
- net Net-(U1-~{SHDN}): track 0.00 -> 6.50 mm
- net /TERMINALS/SWO: track 0.00 -> 6.42 mm
- net /USB HUB/USB_N: track 2.36 -> 6.93 mm
- net /USB HUB/USB_P: track 5.97 -> 10.1 mm
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