File: V1/Design/HW.ACIM-DBG/HW.ACIM-DBG.kicad_pcb (KiCad board)
At the start: 4 copper layers, 60 x 95 mm, 126 parts, among them J1 USB C, J3 SNAP PINOUT, J4 MICRO USB, J5 MCDBG PORT, Q1 MFET N, Q2 MFET N, SW1 PRG SEL, U1 LDO 3.3V, U10 12MHz, U2 USB HUB 2.0 4-CH, U3 SPI EEPROM, U7 LOAD SWITCHER, U8 FT4232H, U9 SHIFT REG 8BIT, Y1 24MHz

Commit message: V1 layout update 10
Parts:
- added C101: 22pF, SAMPI:CAP0402, F.Cu at (76.4, 60.2)
- added C110: 100nF, SAMPI:CAP0402, B.Cu at (85.0, 76.0)
- added C112: 100nF, SAMPI:CAP0402, F.Cu at (74.1, 72.3)
- added C113: 10uF, SAMPI:CAP0402, F.Cu at (73.2, 71.5)
- added C119: 22pF, SAMPI:CAP0402, F.Cu at (85.1, 76.1)
- added C120: 22pF, SAMPI:CAP0402, F.Cu at (88.9, 72.4)
- added C121: 100nF, SAMPI:CAP0402, F.Cu at (76.6, 74.8)
- added C122: 10uF, SAMPI:CAP0402, F.Cu at (75.7, 74.0)
- added C123: 100nF, SAMPI:CAP0402, B.Cu at (86.7, 74.3)
- added C124: 10uF, SAMPI:CAP0402, B.Cu at (85.8, 75.1)
- added C125: 100nF, SAMPI:CAP0402, F.Cu at (86.2, 60.3)
- added C126: 10uF, SAMPI:CAP0402, F.Cu at (87.1, 61.2)
- added C127: 100nF, SAMPI:CAP0402, F.Cu at (74.7, 61.9)
- added C128: 10uF, SAMPI:CAP0402, F.Cu at (73.8, 62.7)
- added D101: SLED, SAMPI:LED0603, F.Cu at (95.4, 76.3)
- added D102: PWR, SAMPI:LED0603, F.Cu at (67.1, 76.3)
- added J101: HEADER 2x15POS, SAMPI:HD-2x15x1.27-SMD, B.Cu at (69.2, 67.4)
- added J102: HEADER 2x15POS, SAMPI:HD-2x15x1.27-SMD, B.Cu at (93.2, 67.4)
- added R101: 1K, SAMPI:RES0402, F.Cu at (92.9, 76.3)
- added R102: 1K, SAMPI:RES0402, F.Cu at (77.4, 75.7)
- added R103: 10K, SAMPI:RES0402, F.Cu at (75.5, 61.0)
- added TP101: GND, SAMPI:TP1MM, F.Cu at (95.4, 69.9)
- added TP102: 3V3, SAMPI:TP1MM, F.Cu at (95.4, 59.8)
- added TP103: AGND, SAMPI:TP1MM, F.Cu at (73.8, 75.0)
- added TP104: AVDD, SAMPI:TP1MM, F.Cu at (71.4, 75.0)
- added U101: MIPS 32-bit DSC, SAMPI:TQFP64_10x10_MCHP, F.Cu at (81.2, 67.4)
- added U102: 12MHz, SAMPI:SMD4-2520, F.Cu at (87.2, 74.5)
- moved C10 106.4 mm to (165.9, 89.2)
- moved C11 106.4 mm to (165.9, 91.8)
- moved C12 106.4 mm to (165.9, 94.5)
- moved C13 106.4 mm to (169.6, 76.2)
- moved C14 106.4 mm to (169.6, 78.8)
- moved C15 106.4 mm to (169.6, 81.4)
- moved C16 106.4 mm to (169.6, 84.0)
- moved C34 106.4 mm to (169.6, 89.2)
- moved C35 106.4 mm to (169.6, 91.8)
- moved C36 106.4 mm to (169.6, 94.5)
- moved C37 106.4 mm to (173.3, 76.2)
- moved C38 106.4 mm to (173.3, 78.8)
- moved C39 106.4 mm to (173.3, 81.4)
- moved C44 106.4 mm to (191.3, 76.2)
- moved C45 106.4 mm to (191.3, 78.8)
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Routing:
- net +3V3_ISO: track 0.00 -> 65.4 mm, vias 0 -> 5
- net /PIM/MC_VR_DIV: track 0.00 -> 28.6 mm, vias 0 -> 2
- net /PIM/~{MCLR}: track 0.00 -> 25.8 mm, vias 0 -> 2
- net /PIM/MC_IU_SEN: track 0.00 -> 24.3 mm, vias 0 -> 2
- net /PIM/PWR_RELAY: track 0.00 -> 23.1 mm, vias 0 -> 1
- net /PIM/DV_CTS: track 0.00 -> 22.7 mm, vias 0 -> 1
- net /PIM/SCK: track 0.00 -> 22.1 mm, vias 0 -> 2
- net /PIM/MC_IV_SEN: track 0.00 -> 21.9 mm, vias 0 -> 2
- net /PIM/SDO: track 0.00 -> 20.4 mm, vias 0 -> 2
- net /PIM/MC_VV_DIV: track 0.00 -> 19.9 mm, vias 0 -> 2
- net /PIM/~{CS}: track 0.00 -> 19.8 mm, vias 0 -> 1
- net /PIM/MC_VU_DIV: track 0.00 -> 18.8 mm, vias 0 -> 2
- net /PIM/SDI: track 0.00 -> 18.6 mm, vias 0 -> 2
- net AVDD_ISO: track 0.00 -> 17.8 mm, vias 0 -> 2
- net /PIM/SCL: track 0.00 -> 17.7 mm, vias 0 -> 2
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- added copper zone on B.Cu, net +3V3_ISO
- added copper zone on B.Cu, net AGND_ISO
- added copper zone on F.Cu, net AGND_ISO
- added copper zone on B.Cu, net AVDD_ISO
- added copper zone on F.Cu, net AVDD_ISO
- added copper zone on B.Cu, net GND_ISO
- added copper zone on F.Cu, net GND_ISO
- added copper zone on In1.Cu, net GND_ISO
- added copper zone on In2.Cu, net GND_ISO
Other:
- outline, holes or cut-outs redrawn
- board text added: "2-1"
- board text added: "30-29"
- board text added: "HW.ACIM-MCU-32MK"
- board text added: "PCB V0.0"
