File: V1/Design/HW.ACIM-DBG/HW.ACIM-DBG.kicad_pcb (KiCad board)
At the start: 4 copper layers, 60 x 95 mm, 153 parts, among them J1 USB C, J101 HEADER 2x15POS, J102 HEADER 2x15POS, J3 SNAP PINOUT, J4 MICRO USB, J5 MCDBG PORT, Q1 MFET N, Q2 MFET N, SW1 PRG SEL, U1 LDO 3.3V, U10 12MHz, U101 MIPS 32-bit DSC, U102 12MHz, U2 USB HUB 2.0 4-CH, U3 SPI EEPROM, U7 LOAD SWITCHER, U8 FT4232H, U9 SHIFT REG 8BIT, Y1 24MHz

Commit message: V1 layout update 11
Parts:
- removed C51: 22pF, SAMPI:CAP0603
- removed R48: 100K, SAMPI:RES0603
- added C2: 100nF, SAMPI:CAP0603, F.Cu at (104.1, 64.8)
- moved TP3 99.5 mm to (98.8, 54.5)
- moved R28 97.8 mm to (101.6, 90.0), turned to -90 degrees
- moved FT5 96.9 mm to (98.4, 101.3)
- moved R39 95.2 mm to (103.8, 94.3), turned to -90 degrees
- moved C46 94.6 mm to (98.0, 97.1)
- moved C21 94.6 mm to (94.3, 97.1)
- moved C42 94.2 mm to (93.8, 100.0)
- moved R38 93.9 mm to (105.4, 94.3), turned to -90 degrees
- moved C52 93.2 mm to (109.4, 112.8), turned to 90 degrees
- moved R29 92.6 mm to (107.0, 94.3), turned to -90 degrees
- moved FT6 91.0 mm to (110.2, 97.2), turned to -90 degrees
- moved U10 90.0 mm to (115.4, 97.2), turned to 90 degrees
- moved C49 89.3 mm to (102.2, 94.3), turned to 90 degrees
- moved R47 88.6 mm to (110.2, 94.3), turned to -90 degrees
- moved R46 86.5 mm to (112.9, 99.9), turned to 90 degrees
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Connections:
- C110 pad 2: (no net) -> +3V3_ISO
- C112 pad 1: (no net) -> AGND_ISO
- C112 pad 2: (no net) -> AVDD_ISO
- C113 pad 1: (no net) -> AGND_ISO
- C113 pad 2: (no net) -> AVDD_ISO
- C121 pad 2: (no net) -> +3V3_ISO
- C122 pad 2: (no net) -> +3V3_ISO
- C123 pad 2: (no net) -> +3V3_ISO
- C124 pad 2: (no net) -> +3V3_ISO
- C125 pad 2: (no net) -> +3V3_ISO
- C126 pad 2: (no net) -> +3V3_ISO
- C127 pad 2: (no net) -> +3V3_ISO
- C128 pad 2: (no net) -> +3V3_ISO
- C7 pad 2: /USB HUB/XTALIN -> /USB HUB/XTALOUT
- C9 pad 2: /USB HUB/XTALOUT -> /USB HUB/XTALIN
- H1 pad 5: /TERMINALS/USB1_DP -> /TERMINALS/USB_RP_P
- H1 pad 7: /TERMINALS/USB1_DM -> /TERMINALS/USB_RP_N
- H1 pad 9: /TERMINALS/USB1_VBUS -> /TERMINALS/USB_RP_VBUS
- H2 pad 5: /TERMINALS/USB1_DP -> /TERMINALS/USB_RP_P
- H2 pad 7: /TERMINALS/USB1_DM -> /TERMINALS/USB_RP_N
- H2 pad 9: /TERMINALS/USB1_VBUS -> /TERMINALS/USB_RP_VBUS
- J101 pad 1: (no net) -> AGND_ISO
- J101 pad 11: (no net) -> /PIM/SCL
- J101 pad 12: (no net) -> /PIM/SDA
- J101 pad 13: (no net) -> /PIM/~{CS}
- J101 pad 14: (no net) -> /PIM/SDO
- J101 pad 15: (no net) -> /PIM/SCK
- J101 pad 16: (no net) -> /PIM/SDI
- J101 pad 17: (no net) -> /PIM/PFC_PWM_ENB
- J101 pad 19: (no net) -> /PIM/PFC_PWM_ENA
- J101 pad 2: (no net) -> AGND_ISO
- J101 pad 27: (no net) -> /PIM/ENC_HOME
- J101 pad 28: (no net) -> /PIM/ENC_A
- J101 pad 29: (no net) -> /PIM/ENC_IDX
- J101 pad 3: (no net) -> AVDD_ISO
- J101 pad 30: (no net) -> /PIM/ENC_B
- J101 pad 4: (no net) -> AVDD_ISO
- J101 pad 7: (no net) -> /PIM/IO1
- J101 pad 8: (no net) -> /PIM/IO2
- J101 pad 9: (no net) -> /PIM/PWR_RELAY
- J102 pad 1: (no net) -> /PIM/VBUS
- J102 pad 10: (no net) -> /PIM/DV_TXD
- J102 pad 11: (no net) -> /PIM/DV_RTS
- J102 pad 12: (no net) -> /PIM/DV_CTS
- J102 pad 13: (no net) -> /PIM/~{INV_FLT}
- J102 pad 2: (no net) -> /PIM/PGD
- J102 pad 21: (no net) -> /PIM/MC_TEMP_SEN
- J102 pad 22: (no net) -> /PIM/MC_VR_DIV
- J102 pad 23: (no net) -> /PIM/MC_VU_DIV
- J102 pad 24: (no net) -> /PIM/MC_IU_SEN
- J102 pad 25: (no net) -> /PIM/MC_VV_DIV
- J102 pad 26: (no net) -> /PIM/MC_IV_SEN
- J102 pad 27: (no net) -> +3V3_ISO
- J102 pad 28: (no net) -> +3V3_ISO
- J102 pad 3: (no net) -> /PIM/USB_N
- J102 pad 5: (no net) -> /PIM/USB_P
- J5 pad 11: /TERMINALS/USB2_DM -> /TERMINALS/USB_MC_N
- J5 pad 12: /TERMINALS/USB2_VBUS -> /TERMINALS/USB_MC_VBUS
- J5 pad 9: /TERMINALS/USB2_DP -> /TERMINALS/USB_MC_P
- R102 pad 2: (no net) -> +3V3_ISO
- R103 pad 2: (no net) -> +3V3_ISO
- TP102 pad 1: (no net) -> +3V3_ISO
- TP103 pad 1: (no net) -> AGND_ISO
- TP104 pad 1: (no net) -> AVDD_ISO
- U101 pad 10: (no net) -> +3V3_ISO
- U101 pad 11: (no net) -> /PIM/PFC_PWM_ENA
- U101 pad 12: (no net) -> /PIM/PFC_PWM_ENB
- U101 pad 16: (no net) -> /PIM/MC_VU_DIV
- U101 pad 19: (no net) -> AVDD_ISO
- U101 pad 20: (no net) -> AGND_ISO
- U101 pad 22: (no net) -> /PIM/IO2
- U101 pad 23: (no net) -> /PIM/MC_VV_DIV
- U101 pad 24: (no net) -> /PIM/IO1
- U101 pad 26: (no net) -> +3V3_ISO
- U101 pad 27: (no net) -> /PIM/SDA
- U101 pad 28: (no net) -> /PIM/SCL
- U101 pad 29: (no net) -> /PIM/DV_CTS
- U101 pad 30: (no net) -> /PIM/MC_VR_DIV
- U101 pad 31: (no net) -> /PIM/MC_IV_SEN
- U101 pad 32: (no net) -> /PIM/DV_RTS
- U101 pad 33: (no net) -> /PIM/MC_IU_SEN
- U101 pad 34: (no net) -> /PIM/VBUS
- U101 pad 35: (no net) -> +3V3_ISO
- U101 pad 36: (no net) -> /PIM/USB_N
- U101 pad 37: (no net) -> /PIM/USB_P
- U101 pad 38: (no net) -> +3V3_ISO
- U101 pad 4: (no net) -> /PIM/ENC_A
- U101 pad 43: (no net) -> /PIM/PGD
- U101 pad 45: (no net) -> /PIM/DV_TXD
- U101 pad 49: (no net) -> /PIM/MC_TEMP_SEN
- U101 pad 5: (no net) -> /PIM/ENC_B
- U101 pad 57: (no net) -> +3V3_ISO
- U101 pad 59: (no net) -> /PIM/~{INV_FLT}
- U101 pad 6: (no net) -> /PIM/ENC_IDX
- U101 pad 60: (no net) -> /PIM/SDI
- U101 pad 61: (no net) -> /PIM/SCK
- U101 pad 62: (no net) -> /PIM/PWR_RELAY
- U101 pad 63: (no net) -> /PIM/SDO
- U101 pad 64: (no net) -> /PIM/~{CS}
- U101 pad 8: (no net) -> /PIM/ENC_HOME
- U2 pad 1: /USB HUB/USB1_N -> /TERMINALS/PRG_USB_N
- U2 pad 12: /USB HUB/USB1_VBUS -> /TERMINALS/PRG_VBUS
- U2 pad 16: /TERMINALS/USB1_VBUS -> /TERMINALS/USB_MC_VBUS
- U2 pad 18: /TERMINALS/USB2_VBUS -> /TERMINALS/USB_RP_VBUS
- U2 pad 2: /USB HUB/USB1_P -> /TERMINALS/PRG_USB_P
- U2 pad 20: /TERMINALS/PRG_VBUS -> /USB HUB/USB4_VBUS
- U2 pad 3: /TERMINALS/USB1_DM -> /TERMINALS/USB_MC_N
- U2 pad 4: /TERMINALS/USB1_DP -> /TERMINALS/USB_MC_P
- U2 pad 6: /TERMINALS/USB2_DM -> /TERMINALS/USB_RP_N
- U2 pad 7: /TERMINALS/USB2_DP -> /TERMINALS/USB_RP_P
- U2 pad 8: /TERMINALS/PRG_USB_N -> /USB HUB/USB4_N
- U2 pad 9: /TERMINALS/PRG_USB_P -> /USB HUB/USB4_P
- U8 pad 11: /USB HUB/USB1_VBUS -> /USB HUB/USB4_VBUS
- U8 pad 7: /USB HUB/USB1_N -> /USB HUB/USB4_N
- U8 pad 8: /USB HUB/USB1_P -> /USB HUB/USB4_P
- Y1 pad 1: /USB HUB/XTALIN -> /USB HUB/XTALOUT
- Y1 pad 3: /USB HUB/XTALOUT -> /USB HUB/XTALIN
Routing:
- net +3V3: track 0.00 -> 107.0 mm, vias 0 -> 6
- net /TERMINALS/USB_MC_N: track 0.00 -> 90.3 mm, vias 0 -> 1
- net /TERMINALS/USB_MC_P: track 0.00 -> 89.7 mm, vias 0 -> 1
- net /TERMINALS/USB_RP_N: track 0.00 -> 85.5 mm, vias 0 -> 3
- net /TERMINALS/USB_RP_P: track 0.00 -> 84.7 mm, vias 0 -> 3
- net /TERMINALS/PRG_USB_P: track 2.35 -> 46.5 mm, vias 1 -> 2
- net /TERMINALS/PRG_USB_N: track 2.35 -> 44.9 mm, vias 1 -> 2
- net /TERMINALS/PRG_VBUS: track 0.65 -> 37.5 mm, vias 1 -> 2
- net /VCP/EEDATA: track 0.00 -> 35.3 mm, vias 0 -> 2
- net Net-(U1-~{SHDN}): track 6.50 -> 39.2 mm
- net /VCP/EECS: track 0.00 -> 32.0 mm, vias 0 -> 2
- net /USB HUB/USB4_N: track 0.00 -> 31.6 mm, vias 0 -> 2
- net /USB HUB/USB4_P: track 0.00 -> 31.0 mm
- net GND: track 49.1 -> 79.4 mm
- net /VCP/EECLK: track 0.00 -> 30.2 mm, vias 0 -> 2
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Other:
- outline, holes or cut-outs redrawn
- board text added: "RED: TX YEL: RX"

Commit message: V1 layout update 12
Parts:
- moved FT3 28.2 mm to (104.8, 105.5)
- moved C40 24.3 mm to (104.8, 103.9)
- moved C48 21.2 mm to (118.4, 106.4), turned to 180 degrees
- moved C19 15.9 mm to (102.1, 103.9)
- moved C42 13.2 mm to (107.0, 99.9), turned to -90 degrees
- moved C21 11.4 mm to (105.4, 99.9), turned to 90 degrees
- moved FT4 10.3 mm to (118.4, 111.2), turned to 180 degrees
- moved C45 10.3 mm to (118.4, 109.6), turned to 180 degrees
- moved C46 8.99 mm to (107.0, 97.2), turned to -90 degrees
- moved C20 8.94 mm to (118.4, 112.8)
- moved FT5 8.18 mm to (105.4, 97.2), turned to 90 degrees
- moved C41 6.99 mm to (118.4, 108.0), turned to 180 degrees
- moved C44 4.71 mm to (111.9, 113.5), turned to 90 degrees
- moved C54 4.47 mm to (115.5, 113.5), turned to 90 degrees
- moved C52 0.62 mm to (109.4, 113.5)
Connections:
- SW1 pad 5: VTG -> +3V3
- U8 pad 12: /TERMINALS/DBG_RXD1 -> /TERMINALS/AUX_RXD2
- U8 pad 13: /TERMINALS/DBG_TXD1 -> /TERMINALS/AUX_TXD2
- U8 pad 42: /TERMINALS/AUX_RXD2 -> /TERMINALS/DBG_RXD1
- U8 pad 46: /TERMINALS/AUX_TXD2 -> /TERMINALS/DBG_TXD1
Routing:
- net GND: track 79.4 -> 264.5 mm, vias 0 -> 29
- net +3V3: track 107.0 -> 255.7 mm, vias 6 -> 8
- net /TERMINALS/USB_MC_VBUS: track 1.00 -> 107.7 mm
- net /TERMINALS/USB_RP_VBUS: track 1.00 -> 85.5 mm, vias 1 -> 2
- net Net-(Q1-G): track 1.00 -> 59.5 mm, vias 1 -> 2
- net /TERMINALS/AUX_RXD2: track 0.00 -> 56.5 mm, vias 0 -> 1
- net /TERMINALS/AUX_TXD2: track 0.00 -> 52.8 mm, vias 0 -> 1
- net /TERMINALS/DBG_TXD1: track 0.00 -> 49.3 mm, vias 0 -> 2
- net /TERMINALS/DBG_RXD1: track 0.00 -> 45.8 mm, vias 0 -> 2
- net /TERMINALS/~{MCLR}: track 13.4 -> 55.4 mm
- net /TERMINALS/DBG_RXD2: track 0.00 -> 41.1 mm, vias 0 -> 1
- net /TERMINALS/PGD: track 17.7 -> 58.7 mm, vias 0 -> 1
- net /TERMINALS/PGC: track 27.0 -> 66.7 mm, vias 0 -> 1
- net /TERMINALS/DBG_TXD2: track 0.00 -> 39.2 mm, vias 0 -> 1
- net /TERMINALS/VDD_SEN: track 44.7 -> 82.8 mm, vias 0 -> 1
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- added copper zone on B.Cu, net GND
- added copper zone on F.Cu, net GND
- added copper zone on In1.Cu, net GND
- added copper zone on In2.Cu, net GND

Commit message: V1 layout update 13
Parts:
- added C18: 10uF, SAMPI:CAP0402, F.Cu at (90.4, 99.9)
- added C23: 100nF, SAMPI:CAP0402, F.Cu at (87.0, 96.4)
- added C24: 22pF, SAMPI:CAP0402, F.Cu at (73.4, 107.9)
- added C25: 100nF, SAMPI:CAP0402, F.Cu at (75.5, 110.1)
- added C28: 10uF, SAMPI:CAP0402, F.Cu at (87.9, 97.4)
- added C29: 100nF, SAMPI:CAP0402, B.Cu at (85.4, 108.8)
- added C30: 100nF, SAMPI:CAP0402, F.Cu at (88.7, 98.2)
- added C32: 100nF, SAMPI:CAP0402, F.Cu at (92.5, 105.2)
- added C33: 100nF, SAMPI:CAP0402, F.Cu at (86.2, 111.5)
- added C51: 100nF, SAMPI:CAP0402, F.Cu at (87.1, 110.7)
- added C57: 2.2uF, SAMPI:CAP0402, F.Cu at (85.9, 95.4)
- added C58: 100nF, SAMPI:CAP0402, F.Cu at (75.2, 96.7)
- added C59: 100nF, SAMPI:CAP0402, B.Cu at (87.0, 110.8)
- added C60: 100nF, SAMPI:CAP0402, F.Cu at (91.3, 100.8)
- added C61: 22pF, SAMPI:CAP0402, F.Cu at (91.7, 106.1)
- added C62: 22pF, SAMPI:CAP0402, F.Cu at (87.9, 109.8)
- added D11: SLED, SAMPI:LED0603, F.Cu at (95.4, 112.1)
- added D4: PWR, SAMPI:LED0603, F.Cu at (67.1, 112.1)
- added FT7: 1K@100MHz, SAMPI:IND0402, F.Cu at (89.6, 99.1)
- added FT8: 1K@100MHz, SAMPI:IND0402, B.Cu at (86.1, 111.6)
- added J2: HEADER 2x15POS, SAMPI:HD-2x15x1.27-SMD, B.Cu at (69.2, 103.2)
- added J6: HEADER 2x15POS, SAMPI:HD-2x15x1.27-SMD, B.Cu at (93.2, 103.2)
- added R12: 10K, SAMPI:RES0402, F.Cu at (76.3, 110.9)
- added R13: 1K, SAMPI:RES0402, F.Cu at (69.5, 112.1)
- added R14: 1K, SAMPI:RES0402, F.Cu at (92.9, 112.1)
- added R4: 10K, SAMPI:RES0402, F.Cu at (74.2, 108.8)
- added TP1: GND, SAMPI:TP1MM, F.Cu at (69.2, 109.6)
- added TP10: ERASE, SAMPI:TP1MM, F.Cu at (77.6, 112.3)
- added TP2: 3V3, SAMPI:TP1MM, F.Cu at (95.4, 95.6)
- added TP7: AGND, SAMPI:TP1MM, F.Cu at (89.5, 95.7)
- added TP8: AVDD, SAMPI:TP1MM, F.Cu at (71.4, 110.9)
- added TP9: VCORE, SAMPI:TP1MM, F.Cu at (88.7, 112.2)
- added U4: ATSAME70J20B, SAMPI:TQFP64_10x10_MCHP, F.Cu at (81.2, 103.3)
- added U5: 12MHz, SAMPI:SMD4-2520, F.Cu at (90.0, 108.1)
Connections:
- net /PIM/DB_RXD renamed /PIM-PIC32MK/DB_RXD
- net /PIM/DB_TXD renamed /PIM-PIC32MK/DB_TXD
- net /PIM/DEV_RELAY renamed /PIM-PIC32MK/DEV_RELAY
- net /PIM/DV_CTS renamed /PIM-PIC32MK/DV_CTS
- net /PIM/DV_RTS renamed /PIM-PIC32MK/DV_RTS
- net /PIM/DV_RXD renamed /PIM-PIC32MK/DV_RXD
- net /PIM/DV_TXD renamed /PIM-PIC32MK/DV_TXD
- net /PIM/ENC_A renamed /PIM-PIC32MK/ENC_A
- net /PIM/ENC_B renamed /PIM-PIC32MK/ENC_B
- net /PIM/ENC_HOME renamed /PIM-PIC32MK/ENC_HOME
- net /PIM/ENC_IDX renamed /PIM-PIC32MK/ENC_IDX
- net /PIM/IDC_SEN renamed /PIM-PIC32MK/IDC_SEN
- net /PIM/IO1 renamed /PIM-PIC32MK/IO1
- net /PIM/IO2 renamed /PIM-PIC32MK/IO2
- net /PIM/MC_IU_SEN renamed /PIM-PIC32MK/MC_IU_SEN
- net /PIM/MC_IV_SEN renamed /PIM-PIC32MK/MC_IV_SEN
- net /PIM/MC_PWM_UH renamed /PIM-PIC32MK/MC_PWM_UH
- net /PIM/MC_PWM_UL renamed /PIM-PIC32MK/MC_PWM_UL
- net /PIM/MC_PWM_VH renamed /PIM-PIC32MK/MC_PWM_VH
- net /PIM/MC_PWM_WH renamed /PIM-PIC32MK/MC_PWM_WH
- net /PIM/MC_TEMP_SEN renamed /PIM-PIC32MK/MC_TEMP_SEN
- net /PIM/MC_VR_DIV renamed /PIM-PIC32MK/MC_VR_DIV
- net /PIM/MC_VU_DIV renamed /PIM-PIC32MK/MC_VU_DIV
- net /PIM/MC_VV_DIV renamed /PIM-PIC32MK/MC_VV_DIV
- net /PIM/PFC_IA_SEN renamed /PIM-PIC32MK/PFC_IA_SEN
- net /PIM/PFC_IB_SEN renamed /PIM-PIC32MK/PFC_IB_SEN
- net /PIM/PFC_PWM_A renamed /PIM-PIC32MK/PFC_PWM_A
- net /PIM/PFC_PWM_B renamed /PIM-PIC32MK/PFC_PWM_B
- net /PIM/PFC_PWM_ENA renamed /PIM-PIC32MK/PFC_PWM_ENA
- net /PIM/PFC_PWM_ENB renamed /PIM-PIC32MK/PFC_PWM_ENB
- net /PIM/PGC renamed /PIM-PIC32MK/PGC
- net /PIM/PGD renamed /PIM-PIC32MK/PGD
- net /PIM/PWR_RELAY renamed /PIM-PIC32MK/PWR_RELAY
- net /PIM/SCK renamed /PIM-PIC32MK/SCK
- net /PIM/SCL renamed /PIM-PIC32MK/SCL
- net /PIM/SDA renamed /PIM-PIC32MK/SDA
- net /PIM/SDI renamed /PIM-PIC32MK/SDI
- net /PIM/SDO renamed /PIM-PIC32MK/SDO
- net /PIM/SLED renamed /PIM-PIC32MK/SLED
- net /PIM/USB_N renamed /PIM-PIC32MK/USB_N
- net /PIM/USB_P renamed /PIM-PIC32MK/USB_P
- net /PIM/VAC_DIV renamed /PIM-PIC32MK/VAC_DIV
- net /PIM/VBUS renamed /PIM-PIC32MK/VBUS
- net /PIM/VDC_DIV renamed /PIM-PIC32MK/VDC_DIV
- net /PIM/~{BUTTON} renamed /PIM-PIC32MK/~{BUTTON}
- net /PIM/~{CS} renamed /PIM-PIC32MK/~{CS}
- net /PIM/~{INV_FLT} renamed /PIM-PIC32MK/~{INV_FLT}
- net /PIM/~{MCLR} renamed /PIM-PIC32MK/~{MCLR}
- net /PIM/~{PFC_FLT} renamed /PIM-PIC32MK/~{PFC_FLT}
- J102 pad 16: /PIM/MC_PWM_WL -> /PIM-PIC32MK/MC_PWM_VL
- J102 pad 18: /PIM/MC_PWM_VL -> /PIM-PIC32MK/MC_PWM_WL
- U101 pad 51: /PIM/MC_PWM_WL -> /PIM-PIC32MK/MC_PWM_WL
- U101 pad 55: /PIM/MC_PWM_VL -> /PIM-PIC32MK/MC_PWM_VL
Routing:
- net VDD: track 0.00 -> 60.6 mm, vias 0 -> 7
- net /PIM-SAME70/MC_IU_SEN: track 0.00 -> 24.7 mm, vias 0 -> 1
- net /PIM-SAME70/MC_PWM_UL: track 0.00 -> 21.7 mm, vias 0 -> 2
- net Net-(U4-VDDOUT): track 0.00 -> 21.5 mm, vias 0 -> 1
- net /PIM-SAME70/MC_IV_SEN: track 0.00 -> 19.6 mm, vias 0 -> 1
- net /PIM-SAME70/MC_PWM_VL: track 0.00 -> 19.4 mm, vias 0 -> 1
- net /PIM-SAME70/MC_PWM_WL: track 0.00 -> 18.6 mm, vias 0 -> 2
- net GND1: track 0.00 -> 15.5 mm, vias 0 -> 2
- net /PIM-SAME70/~{INV_FLT}: track 0.00 -> 14.7 mm, vias 0 -> 1
- net /PIM-SAME70/MC_PWM_WH: track 0.00 -> 14.2 mm, vias 0 -> 1
- net /PIM-PIC32MK/MC_PWM_VL: track 0.00 -> 13.9 mm, vias 0 -> 1
- net AGND1: track 0.00 -> 12.9 mm
- net /PIM/MC_PWM_VL: track 12.6 -> 0.00 mm, vias 1 -> 0
- net /PIM-SAME70/USB_N: track 0.00 -> 11.0 mm, vias 0 -> 1
- net /PIM-SAME70/USB_P: track 0.00 -> 10.7 mm, vias 0 -> 1
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- added copper zone on B.Cu, net GND1
- added copper zone on F.Cu, net GND1
- added copper zone on In1.Cu, net GND1
- added copper zone on In2.Cu, net GND1
Other:
- outline, holes or cut-outs redrawn
- board text added: "HW.ACIM-MCU-E70"
