File: V1/Design/HW.ACIM-DBG/HW.ACIM-DBG.kicad_pcb (KiCad board)
At the start: 4 copper layers, 60 x 95 mm, 186 parts, among them J1 USB C, J101 HEADER 2x15POS, J102 HEADER 2x15POS, J2 HEADER 2x15POS, J3 SNAP PINOUT, J4 MICRO USB, J5 MCDBG PORT, J6 HEADER 2x15POS, Q1 MFET N, Q2 MFET N, SW1 PRG SEL, U1 LDO 3.3V, U10 12MHz, U101 MIPS 32-bit DSC, U102 12MHz, U2 USB HUB 2.0 4-CH, U3 SPI EEPROM, U4 ATSAME70J20B, U5 12MHz, U7 LOAD SWITCHER, U8 FT4232H, U9 SHIFT REG 8BIT, Y1 24MHz

Commit message: V1 layout update 15
Routing:
- net GND: track 264.5 -> 37.6 mm, vias 29 -> 31
- net +3V3: track 255.7 -> 301.0 mm, vias 8 -> 14
- net Net-(F1-Pad1): track 19.8 -> 61.2 mm, vias 4 -> 5
- net /PIM-SAME70/DB_TXD: track 0.00 -> 34.2 mm, vias 1 -> 2
- net /PIM-SAME70/DV_TXD: track 1.77 -> 32.9 mm
- net /PIM-SAME70/SWDCLK: track 1.27 -> 32.2 mm
- net /PIM-SAME70/~{MCLR}: track 3.93 -> 32.3 mm
- net /PIM-SAME70/SWDIO: track 3.59 -> 26.7 mm
- net /PIM-SAME70/DV_RXD: track 2.00 -> 24.9 mm, vias 1 -> 2
- net /PIM-SAME70/DB_RXD: track 3.27 -> 25.5 mm
- net /PIM-SAME70/MC_PWM_VH: track 0.00 -> 19.4 mm, vias 1 -> 2
- net /PIM-SAME70/VDC_DIV: track 0.00 -> 19.0 mm, vias 1 -> 2
- net /PIM-SAME70/IDC_SEN: track 0.00 -> 18.8 mm, vias 1 -> 2
- net /PIM-SAME70/MC_PWM_UH: track 3.20 -> 19.2 mm
- net GND1: track 17.8 -> 4.00 mm, vias 3 -> 8
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- added copper zone on B.Cu, net +3V3
- added copper zone on F.Cu, net +3V3
- added copper zone on In1.Cu, net +3V3
- added copper zone on In2.Cu, net +3V3
- added copper zone on F.Cu, net +5V
- added copper zone on F.Cu, net Net-(C11-Pad2)
- added copper zone on F.Cu, net Net-(F1-Pad1)
- added copper zone on In1.Cu, net Net-(F1-Pad1)
- added copper zone on F.Cu, net VTG
