File: V1/Design/HW.ACIM-DBG/PIM-PIC32MK.kicad_sch (KiCad schematic)
At the start: 27 parts, among them J101 HEADER 2x15POS, J102 HEADER 2x15POS, U101 MIPS 32-bit DSC, U102 12MHz

Commit message: V1 layout update 13
Connections:
- net MC_PWM_VL: now also J102.16; no longer J102.18
- net MC_PWM_WL: now also J102.18; no longer J102.16
Changed lines of the file:
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@@
 	(hierarchical_label "MC_PWM_VL"
 		(shape output)
-		(at 101.6 170.18 0)
+		(at 101.6 172.72 0)
 		(effects
 			(font
@@
 		)
 		(property "Netclass" "PWM5L"
-			(at 115.57 170.18 0)
+			(at 115.57 172.72 0)
 			(effects
 				(font
@@
 	(hierarchical_label "MC_PWM_WL"
 		(shape output)
-		(at 101.6 172.72 0)
+		(at 101.6 170.18 0)
 		(effects
 			(font
@@
 		)
 		(property "Netclass" "PWM6L"
-			(at 120.015 172.72 0)
-			(effects
-				(font
+			(at 120.015 170.18 0)
+			(effects
+				(font
