File: V1/Design/HW.ACIM-DBG/PIM-SAME70.kicad_sch (KiCad schematic)
At the start: 34 parts

Commit message: V1 layout update 14
Connections:
- net DEV_RELAY: now also U?.40 (PA3/SDA0/USLONCOL1); no longer U?.44 (PD10/PWM0.L0)
- net IO1: now also U?.43 (PD11/PWM0.H0); no longer U?.46 (PB4/PWM0.H2/SDA1/USTXD1)
- net IO2: now also U?.41 (PD12); no longer U?.47 (PB5/PWM0.L0/SCL1)
- net PWR_RELAY: now also U?.44 (PD10/PWM0.L0); no longer U?.43 (PD11/PWM0.H0)
- net SLED: now also U?.50 (PD7/PWM1.H3); no longer U?.16 (PA8/PWM1.H3/XOUT32)
- net USB_VBUS: now also U?.51 (PD6/PWM1.L3); no longer U?.15 (PA7/PWM0.H3/XIN32)
- no-connect marks 41 -> 42
Changed lines of the file:
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@@
+	)
+	(no_connect
+		(at 158.75 35.56)
+	)
+	(no_connect
+		(at 158.75 33.02)
+	)
+	(no_connect
+		(at 101.6 177.8)
+	)
+	(no_connect
+		(at 31.115 172.72)
+	)
+	(no_connect
+		(at 99.06 71.12)
+	)
+	(no_connect
+		(at 31.115 175.26)
+	)
+	(no_connect
+		(at 158.75 78.74)
+	)
+	(no_connect
+		(at 92.71 162.56)
+	)
+	(no_connect
+		(at 40.005 172.72)
+	)
+	(no_connect
+		(at 92.71 160.02)
+	)
+	(no_connect
+		(at 99.06 86.36)
+	)
+	(no_connect
+		(at 92.71 165.1)
+	)
+	(no_connect
+		(at 101.6 165.1)
+	)
+	(no_connect
+		(at 40.005 160.02)
+	)
+	(no_connect
+		(at 31.115 154.94)
+	)
+	(no_connect
+		(at 101.6 175.26)
+	)
+	(no_connect
+		(at 158.75 55.88)
+	)
+	(no_connect
+		(at 31.115 165.1)
+	)
+	(no_connect
+		(at 31.115 177.8)
+	)
+	(no_connect
+		(at 40.005 165.1)
+	)
+	(no_connect
+		(at 158.75 68.58)
+	)
+	(no_connect
+		(at 158.75 58.42)
+	)
+	(no_connect
+		(at 40.005 170.18)
+	)
+	(no_connect
+		(at 99.06 30.48)
+	)
+	(no_connect
+		(at 31.115 167.64)
 	)
 	(no_connect
@@
 	)
 	(no_connect
-		(at 101.6 177.8)
-	)
-	(no_connect
-		(at 31.115 172.72)
-	)
-	(no_connect
-		(at 99.06 71.12)
-	)
-	(no_connect
-		(at 99.06 55.88)
-	)
-	(no_connect
-		(at 31.115 175.26)
-	)
-	(no_connect
-		(at 92.71 162.56)
-	)
-	(no_connect
-		(at 40.005 172.72)
-	)
-	(no_connect
-		(at 92.71 160.02)
-	)
-	(no_connect
-		(at 99.06 86.36)
-	)
-	(no_connect
-		(at 92.71 165.1)
-	)
-	(no_connect
-		(at 99.06 43.18)
-	)
-	(no_connect
-		(at 101.6 165.1)
-	)
-	(no_connect
-		(at 40.005 160.02)
-	)
-	(no_connect
-		(at 31.115 154.94)
-	)
-	(no_connect
-		(at 101.6 175.26)
-	)
-	(no_connect
-		(at 158.75 55.88)
-	)
-	(no_connect
-		(at 31.115 165.1)
-	)
-	(no_connect
-		(at 31.115 177.8)
-	)
-	(no_connect
-		(at 40.005 165.1)
-	)
-	(no_connect
-		(at 158.75 68.58)
-	)
-	(no_connect
-		(at 158.75 58.42)
-	)
-	(no_connect
-		(at 40.005 170.18)
-	)
-	(no_connect
-		(at 99.06 30.48)
-	)
-	(no_connect
-		(at 31.115 167.64)
-	)
-	(no_connect
 		(at 40.005 167.64)
 	)
 	(no_connect
-		(at 99.06 40.64)
-	)
-	(no_connect
 		(at 99.06 27.94)
 	)
@@
 	(no_connect
 		(at 92.71 177.8)
+	)
+	(no_connect
+		(at 158.75 76.2)
 	)
 	(no_connect
@@
 		)
 	)
-	(hierarchical_label "USB_VBUS"
-		(shape input)
-		(at 158.75 33.02 0)
-		(effects
-			(font
-				(size 1.27 1.27)
-			)
-			(justify left)
-		)
-		(property "Netclass" ""
-			(at 172.72 33.02 0)
-			(effects
-				(font
-					(size 1.27 1.27)
-					(italic yes)
-				)
-				(justify left)
-			)
-		)
-	)
-	(hierarchical_label "PWR_RELAY"
-		(shape output)
-		(at 99.06 53.34 180)
-		(effects
-			(font
-				(size 1.27 1.27)
-			)
-			(justify right)
-		)
-	)
 	(hierarchical_label "MC_PWM_VL"
 		(shape output)
@@
 				(justify left)
 			)
-		)
-	)
-	(hierarchical_label "SLED"
-		(shape output)
-		(at 158.75 35.56 0)
-		(effects
-			(font
-				(size 1.27 1.27)
-			)
-			(justify left)
 		)
 	)
@@
 		)
 	)
+	(hierarchical_label "IO1"
+		(shape bidirectional)
+		(at 99.06 53.34 180)
+		(effects
+			(font
+				(size 1.27 1.27)
+			)
+			(justify right)
+		)
+	)
+	(hierarchical_label "IO2"
+		(shape bidirectional)
+		(at 99.06 55.88 180)
+		(effects
+			(font
+				(size 1.27 1.27)
+			)
+			(justify right)
+		)
+	)
 	(hierarchical_label "VDC_DIV"
 		(shape input)
@@
 				(justify left)
 			)
+		)
+	)
+	(hierarchical_label "SLED"
+		(shape output)
+		(at 99.06 43.18 180)
+		(effects
+			(font
+				(size 1.27 1.27)
+			)
+			(justify right)
 		)
 	)
@@
 		)
 	)
-	(hierarchical_label "IO2"
-		(shape bidirectional)
-		(at 158.75 78.74 0)
-		(effects
-			(font
-				(size 1.27 1.27)
-			)
-			(justify left)
-		)
-	)
 	(hierarchical_label "DEV_RELAY"
 		(shape output)
-		(at 99.06 50.8 180)
-		(effects
-			(font
-				(size 1.27 1.27)
-			)
-			(justify right)
+		(at 158.75 25.4 0)
+		(effects
+			(font
+				(size 1.27 1.27)
+			)
+			(justify left)
 		)
 	)
@@
 		)
 	)
+	(hierarchical_label "USB_VBUS"
+		(shape input)
+		(at 99.06 40.64 180)
+		(effects
+			(font
+				(size 1.27 1.27)
+			)
+			(justify right)
+		)
+		(property "Netclass" ""
+			(at 85.09 40.64 0)
+			(effects
+				(font
+					(size 1.27 1.27)
+					(italic yes)
+				)
+				(justify right)
+			)
+		)
+	)
 	(hierarchical_label "~{INV_FLT}"
 		(shape input)
@@
 				(justify left)
 			)
+		)
+	)
+	(hierarchical_label "PWR_RELAY"
+		(shape output)
+		(at 99.06 50.8 180)
+		(effects
+			(font
+				(size 1.27 1.27)
+			)
+			(justify right)
 		)
 	)
@@
 		)
 	)
-	(hierarchical_label "IO1"
-		(shape bidirectional)
-		(at 158.75 76.2 0)
-		(effects
-			(font
-				(size 1.27 1.27)
-			)
-			(justify left)
-		)
-	)

Commit message: Production HW.ACIM-DBG_V1.0 update BoM
Parts:
- gave numbers to parts that had none: 34
